Commit message: add acone camera

File: arx_lift2s_description/xacro/components/ac_one.xacro (robot description, xacro)
@@ -25,4 +25,16 @@
 			</collision>
 		</link>
+		<link name="head_camera">
+			<visual>
+				<geometry>
+					<mesh filename="file://$(find sensor_models)/meshes/d405/d405.obj"/>
+				</geometry>
+			</visual>
+		</link>
+		<joint name="head_camera_joint" type="fixed">
+			<origin xyz="0.090415 0.002 0.2285" rpy="0 1.0472 0"/>
+			<parent link="body_link"/>
+			<child link="head_camera"/>
+		</joint>
 	</xacro:macro>
 </robot>
