Commit message: update chassis config

File: arx_lift2s_description/xacro/component.xacro (robot description, xacro)
@@ -4,5 +4,5 @@
 <!-- |    This file includes the base robot structure and both arms                    | -->
 <!-- =================================================================================== -->
-<robot name="ARX_Lift2S" xmlns:xacro="http://www.ros.org/wiki/xacro">
+<robot name="AC One" xmlns:xacro="http://www.ros.org/wiki/xacro">
 	<xacro:property name="PI" value="3.1415926535897931"/>
 	<xacro:arg name="type" default="chassis"/>
@@ -10,5 +10,5 @@
 		<!-- Include Chassis -->
 		<xacro:include filename="$(find arx_lift2s_description)/xacro/components/chassis.xacro"/>
-		<xacro:chassis/>
+		<xacro:chassis enable_wheel_joints="true"/>
 	</xacro:if>
 	<xacro:if value="${'$(arg type)' == 'ac_one'}">

File: arx_lift2s_description/xacro/components/chassis.xacro (robot description, xacro)
@@ -2,5 +2,4 @@
 <robot xmlns:xacro="http://www.ros.org/wiki/xacro" name="arx_lift2s_base">
 	<xacro:arg name="robot_name" default="arx_lift2s_base"/>
-	<xacro:include filename="$(find arx_lift2s_description)/xacro/components/wheel.xacro"/>
 	<xacro:macro name="chassis" params="enable_wheel_joints:='false'">
 		<link name="base_link">
@@ -47,8 +46,20 @@
 			<limit lower="0" upper="0.46" effort="400" velocity="0.15"/>
 		</joint>
-		<xacro:wheel wheel_name="wheel_1" enable_passive_wheels="false"/>
-		<xacro:wheel wheel_name="wheel_2" enable_passive_wheels="false"/>
-		<xacro:wheel wheel_name="wheel_3" enable_passive_wheels="false"/>
-		<joint name="wheel1_joint" type="fixed">
+		<xacro:property name="wheel_joint_type" value="fixed"/>
+		<xacro:if value="${enable_wheel_joints}">
+			<xacro:property name="wheel_joint_type" value="continuous"/>
+		</xacro:if>
+		<xacro:if value="${enable_wheel_joints}">
+			<link name="wheel_1"/>
+			<link name="wheel_2"/>
+			<link name="wheel_3"/>
+		</xacro:if>
+		<xacro:unless value="${enable_wheel_joints}">
+			<xacro:include filename="$(find arx_lift2s_description)/xacro/components/wheel.xacro"/>
+			<xacro:wheel wheel_name="wheel_1" enable_passive_wheels="false"/>
+			<xacro:wheel wheel_name="wheel_2" enable_passive_wheels="false"/>
+			<xacro:wheel wheel_name="wheel_3" enable_passive_wheels="false"/>
+		</xacro:unless>
+		<joint name="wheel1_joint" type="${wheel_joint_type}">
 			<origin xyz="0.15361 0.29246 -0.093" rpy="0.0 0.0 1.0472"/>
 			<parent link="base_link"/>
@@ -58,5 +69,5 @@
 			</xacro:if>
 		</joint>
-		<joint name="wheel2_joint" type="fixed">
+		<joint name="wheel2_joint" type="${wheel_joint_type}">
 			<origin xyz="0.15361 -0.29245 -0.093" rpy="0.0 0.0 -1.0472"/>
 			<parent link="base_link"/>
@@ -66,5 +77,5 @@
 			</xacro:if>
 		</joint>
-		<joint name="wheel3_joint" type="fixed">
+		<joint name="wheel3_joint" type="${wheel_joint_type}">
 			<origin xyz="-0.35293 0 -0.093" rpy="0.0 0.0 3.1415"/>
 			<parent link="base_link"/>

File: arx_lift2s_description/xacro/robot.xacro (robot description, xacro)
@@ -1,5 +1,5 @@
 <robot name="arx_lift2s" xmlns:xacro="http://www.ros.org/wiki/xacro">
 	<xacro:arg name="type" default="x5"/>
-	<xacro:arg name="enable_wheel_joints" default="true"/>
+	<xacro:arg name="enable_wheel_joints" default="false"/>
 	<xacro:arg name="ros2_control_hardware_type" default="mock_components"/>
 	<xacro:property name="type_arg" value="$(arg type)"/>
