Commit message: add self-collision for lift body

File: arx_lift2s_description/xacro/component.xacro (robot description, xacro)
@@ -9,5 +9,5 @@
 	<xacro:if value="${'$(arg type)' == 'chassis'}">
 		<xacro:include filename="$(find arx_lift2s_description)/xacro/components/chassis.xacro"/>
-		<xacro:chassis enable_wheel_joints="true"/>
+		<xacro:chassis enable_wheel_joints="true" collider="$(arg collider)"/>
 	</xacro:if>
 	<xacro:if value="${'$(arg type)' == 'wheel'}">

File: arx_lift2s_description/xacro/components/chassis.xacro (robot description, xacro)
@@ -2,5 +2,5 @@
 <robot xmlns:xacro="http://www.ros.org/wiki/xacro" name="arx_lift2s_base">
 	<xacro:arg name="robot_name" default="arx_lift2s_base"/>
-	<xacro:macro name="chassis" params="enable_wheel_joints:='false'">
+	<xacro:macro name="chassis" params="enable_wheel_joints:='false' collider:='simple'">
 		<link name="base_link">
 			<inertial>
@@ -15,10 +15,59 @@
 				</geometry>
 			</visual>
-			<collision>
-				<geometry>
-					<mesh filename="file://$(find arx_lift2s_description)/meshes/chassis/base_link.glb"/>
-				</geometry>
-			</collision>
+			<xacro:if value="${collider == 'convex'}">
+				<collision>
+					<geometry>
+						<mesh filename="file://$(find arx_lift2s_description)/meshes/chassis/base_link.glb"/>
+					</geometry>
+				</collision>
+			</xacro:if>
+			<xacro:if value="${collider == 'simple'}">
+				<!-- Main chassis deck (not used in OCS2 arm self-collision pairs) -->
+				<collision name="simple_base_platform">
+					<origin xyz="-0.09 0 0.0" rpy="0 0 0"/>
+					<geometry>
+						<box size="0.52 0.36 0.22"/>
+					</geometry>
+				</collision>
+				<!-- Left / right side skirts -->
+				<collision name="simple_base_left">
+					<origin xyz="0.0 0.24 -0.066" rpy="0 0 0"/>
+					<geometry>
+						<box size="0.44 0.18 0.13"/>
+					</geometry>
+				</collision>
+				<collision name="simple_base_right">
+					<origin xyz="0.0 -0.24 -0.066" rpy="0 0 0"/>
+					<geometry>
+						<box size="0.43 0.18 0.13"/>
+					</geometry>
+				</collision>
+			</xacro:if>
 		</link>
+		<!-- Dedicated mast link so OCS2 pairs hit the lift column, not deck/skirts/rear panel -->
+		<link name="lift_mast_link">
+			<xacro:if value="${collider == 'simple'}">
+				<collision name="simple_lift_mast">
+					<origin xyz="0 0 0" rpy="0 0 0"/>
+					<geometry>
+						<box size="0.13 0.13 0.60"/>
+					</geometry>
+				</collision>
+			</xacro:if>
+			<xacro:if value="${collider == 'convex'}">
+				<!-- approximate mast volume when convex meshes are used on base/lift -->
+				<collision name="simple_lift_mast">
+					<origin xyz="0 0 0" rpy="0 0 0"/>
+					<geometry>
+						<box size="0.13 0.13 0.60"/>
+					</geometry>
+				</collision>
+			</xacro:if>
+		</link>
+		<joint name="lift_mast_joint" type="fixed">
+			<origin xyz="0.01 0 0.50" rpy="0 0 0"/>
+			<parent link="base_link"/>
+			<child link="lift_mast_link"/>
+		</joint>
 		<link name="lift_link">
 			<inertial>
@@ -33,9 +82,20 @@
 				</geometry>
 			</visual>
-			<collision>
-				<geometry>
-					<mesh filename="file://$(find arx_lift2s_description)/meshes/chassis/lift.glb"/>
-				</geometry>
-			</collision>
+			<xacro:if value="${collider == 'convex'}">
+				<collision>
+					<geometry>
+						<mesh filename="file://$(find arx_lift2s_description)/meshes/chassis/lift.glb"/>
+					</geometry>
+				</collision>
+			</xacro:if>
+			<xacro:if value="${collider == 'simple'}">
+				<!-- Carriage plate only; rear upright removed (was registering as back screen) -->
+				<collision name="simple_lift_carriage">
+					<origin xyz="-0.015 0 -0.01" rpy="0 0 0"/>
+					<geometry>
+						<box size="0.24 0.16 0.12"/>
+					</geometry>
+				</collision>
+			</xacro:if>
 		</link>
 		<joint name="lift_joint" type="prismatic">

File: arx_lift2s_description/xacro/robot.xacro (robot description, xacro)
@@ -11,5 +11,5 @@
 	<!-- Lift chassis + prismatic lift_joint -->
 	<xacro:include filename="$(find arx_lift2s_description)/xacro/components/chassis.xacro"/>
-	<xacro:chassis enable_wheel_joints="$(arg enable_wheel_joints)"/>
+	<xacro:chassis enable_wheel_joints="$(arg enable_wheel_joints)" collider="$(arg collider)"/>
 	<joint name="body_joint" type="fixed">
 		<origin xyz="0.13 0.001801 0.0529"/>
