Commit message: :construction: migrate hardware interface,need to fixed the bug of missing gripper and lift_body joint

File: arx_lift2s_description/xacro/robot.xacro (robot description, xacro)
@@ -10,10 +10,7 @@
 		<xacro:property name="selected_arm_type" value="r5"/>
 	</xacro:if>
-	<xacro:if value="${type_arg == 'acone_x5'}">
-		<xacro:property name="selected_base_type" value="acone"/>
-	</xacro:if>
+	<!-- acone_x5 / acone_r5: arm config variant only; keep lift2s chassis (lift_joint) for body bridge -->
 	<xacro:if value="${type_arg == 'acone_r5'}">
 		<xacro:property name="selected_arm_type" value="r5"/>
-		<xacro:property name="selected_base_type" value="acone"/>
 	</xacro:if>
 	<xacro:if value="${selected_base_type == 'lift2s'}">

File: arx_lift2s_description/xacro/ros2_control/interfaces.xacro (robot description, xacro)
@@ -1,5 +1,5 @@
 <?xml version="1.0"?>
 <robot xmlns:xacro="http://www.ros.org/wiki/xacro">
-    <!-- ARX LIFT 2S 基座关节接口宏定义 -->
+    <!-- ARX LIFT 2S 基座关节接口宏定义（仿真用） -->
     <xacro:macro name="arx_lift2s_base_interfaces">
         <!-- 升降关节接口定义 (仅 lift2s 底盘需要) -->
@@ -13,3 +13,72 @@
         </xacro:if>
     </xacro:macro>
+    <!-- Lift column: ArxLiftHardware setHeight (meters). -->
+    <xacro:macro name="arx_lift2s_lift_interfaces">
+        <joint name="lift_joint">
+            <command_interface name="position"/>
+            <state_interface name="position"/>
+            <state_interface name="velocity"/>
+            <state_interface name="effort"/>
+        </joint>
+    </xacro:macro>
+    <!-- Single X5 arm (+ gripper): used by ArxX5Hardware or mock/gz/isaac. -->
+    <xacro:macro name="arx_lift2s_arm_interfaces" params="name">
+        <xacro:property name="prefix" value="${name + '_' if name else ''}"/>
+        <xacro:arg name="gazebo" default="false"/>
+        <joint name="${prefix}joint1">
+            <command_interface name="position"/>
+            <state_interface name="position"/>
+            <state_interface name="velocity"/>
+            <state_interface name="effort"/>
+        </joint>
+        <joint name="${prefix}joint2">
+            <command_interface name="position"/>
+            <state_interface name="position">
+                <param name="initial_value">0.4</param>
+            </state_interface>
+            <state_interface name="velocity"/>
+            <state_interface name="effort"/>
+        </joint>
+        <joint name="${prefix}joint3">
+            <command_interface name="position"/>
+            <state_interface name="position">
+                <param name="initial_value">0.12</param>
+            </state_interface>
+            <state_interface name="velocity"/>
+            <state_interface name="effort"/>
+        </joint>
+        <joint name="${prefix}joint4">
+            <command_interface name="position"/>
+            <state_interface name="position">
+                <param name="initial_value">0.26</param>
+            </state_interface>
+            <state_interface name="velocity"/>
+            <state_interface name="effort"/>
+        </joint>
+        <joint name="${prefix}joint5">
+            <command_interface name="position"/>
+            <state_interface name="position"/>
+            <state_interface name="velocity"/>
+            <state_interface name="effort"/>
+        </joint>
+        <joint name="${prefix}joint6">
+            <command_interface name="position"/>
+            <state_interface name="position"/>
+            <state_interface name="velocity"/>
+            <state_interface name="effort"/>
+        </joint>
+        <joint name="${prefix}gripper_joint">
+            <command_interface name="position"/>
+            <state_interface name="position"/>
+            <state_interface name="velocity"/>
+            <state_interface name="effort"/>
+        </joint>
+        <xacro:if value="$(arg gazebo)">
+            <joint name="${prefix}joint8">
+                <state_interface name="position"/>
+                <state_interface name="velocity"/>
+                <state_interface name="effort"/>
+            </joint>
+        </xacro:if>
+    </xacro:macro>
 </robot>

File: arx_lift2s_description/xacro/ros2_control/robot.xacro (robot description, xacro)
@@ -1,3 +1,8 @@
 <?xml version="1.0"?>
+<!--
+  LIFT2S ros2_control wiring.
+  - mock_components / gz / isaac: single system (arx5_interfaces + base lift)
+  - real: left can1, right can3, lift can5 via arxlift2s_ros2_control
+-->
 <robot xmlns:xacro="http://www.ros.org/wiki/xacro" name="arx_lift2s">
     <xacro:arg name="ros2_control_hardware_type" default="mock_components"/>
@@ -7,29 +12,32 @@
     <xacro:include filename="$(find arx_lift2s_description)/xacro/ros2_control/interfaces.xacro"/>
     <xacro:if value="${'$(arg ros2_control_hardware_type)' == 'real'}">
+        <!-- Left arm -->
         <ros2_control name="arx_lift2s_left_system" type="system">
             <hardware>
-                <plugin>arx_ros2_control/ArxX5Hardware</plugin>
-                <param name="robot_model">X5</param>
-                <param name="can_interface">can1</param>
-                <param name="joint_k_gains">[80.0, 70.0, 70.0, 30.0, 30.0, 20.0]</param>
-                <param name="joint_d_gains">[2.0, 2.0, 2.0, 1.0, 1.0, 0.7]</param>
-                <!-- 可选：夹爪增益，不写则用默认 -->
-                <!-- <param name="gripper_kp">5.0</param> -->
-                <!-- <param name="gripper_kd">0.2</param> -->
+                <plugin>arxlift2s_ros2_control/ArxX5Hardware</plugin>
+                <param name="can_name">can1</param>
+                <param name="urdf_path">$(find arx_lift2s_description)/urdf/x5_sdk.urdf</param>
+                <param name="end_type">2</param>
             </hardware>
-            <xacro:arx5_interfaces name="left"/>
+            <xacro:arx_lift2s_arm_interfaces name="left"/>
         </ros2_control>
+        <!-- Right arm -->
         <ros2_control name="arx_lift2s_right_system" type="system">
             <hardware>
-                <plugin>arx_ros2_control/ArxX5Hardware</plugin>
-                <param name="robot_model">X5</param>
-                <param name="can_interface">can3</param>
-                <param name="joint_k_gains">[80.0, 70.0, 70.0, 30.0, 30.0, 20.0]</param>
-                <param name="joint_d_gains">[2.0, 2.0, 2.0, 1.0, 1.0, 0.7]</param>
-                <!-- 可选：夹爪增益，不写则用默认 -->
-                <!-- <param name="gripper_kp">5.0</param> -->
-                <!-- <param name="gripper_kd">0.2</param> -->
+                <plugin>arxlift2s_ros2_control/ArxX5Hardware</plugin>
+                <param name="can_name">can3</param>
+                <param name="urdf_path">$(find arx_lift2s_description)/urdf/x5_sdk.urdf</param>
+                <param name="end_type">2</param>
             </hardware>
-            <xacro:arx5_interfaces name="right"/>
+            <xacro:arx_lift2s_arm_interfaces name="right"/>
+        </ros2_control>
+        <!-- Lift column only (ArxLiftHardware; robot_type 2 = LIFTS) -->
+        <ros2_control name="arx_lift2s_lift_system" type="system">
+            <hardware>
+                <plugin>arxlift2s_ros2_control/ArxLiftHardware</plugin>
+                <param name="can_name">can5</param>
+                <param name="robot_type">2</param>
+            </hardware>
+            <xacro:arx_lift2s_lift_interfaces/>
         </ros2_control>
     </xacro:if>
