Commit message: CLEAN UP arx mesh

File: arx5_description/urdf/arx5_ac1.urdf (robot description, URDF)
Before this commit: robot ARX 5, 14 links, 13 joints
Links:
- link camera: geometry visual mesh filename=package://sensor_models/meshes/d405.glb
- link link3: mass 0.54534 -> 0.54316
- link link4: mass 0.11714 -> 0.11827
- link link5: mass 0.63488 -> 0.67398; geometry collision mesh filename=package://arx5_description/meshes/ac1/link5.glb; visual mesh filename=package://arx5_description/meshes/ac1/link5.glb
- link link6: mass 0.44089 -> 0.34667
- link link7: mass 0.064798 -> 0.08924
- link link8: mass 0.064798 -> 0.089402
Joints:
- joint gripper_center_fixed: origin xyz=0.145 0 0.006376 -> xyz=0.1424 0 0.0001057
- joint gripper_joint: origin xyz=0.08657 0.024896 -0.0002436 -> xyz=0.08397 0.02721 -0.0062702
- joint joint1: limit lower=-2.094 upper=3.1416 effort=27 velocity=5.5 -> lower=-2.094 upper=3.141592653589793 effort=27 velocity=5.5
- joint joint2: limit lower=0 upper=3.66 effort=100 velocity=5 -> lower=0 upper=3.665 effort=27 velocity=5.5
- joint joint3: axis 0 1 0 -> 0 -1 0; limit lower=0 upper=3.14 effort=100 velocity=5 -> lower=0 upper=3.24 effort=27 velocity=5.5; origin xyz=-0.264 0 0 rpy=3.1416 0 0 -> xyz=-0.264 0 0 rpy=0 0 0
- joint joint4: axis 0 1 0 -> 0 -1 0; limit lower=-1.57 upper=1.57 effort=100 velocity=5 -> lower=-1.671 upper=1.671 effort=7 velocity=20; origin xyz=0.245 0 -0.056 -> xyz=0.245 0 0.056
- joint joint5: axis 0 0 1 -> 0 0 -1; limit lower=-1.57 upper=1.57 effort=100 velocity=5 -> lower=-1.671 upper=1.671 effort=7 velocity=20; origin xyz=0.06775 0.0005 -0.0865 -> xyz=0.06775 0 0.0845
- joint joint6: limit lower=-1.57 upper=1.57 effort=100 velocity=5 -> lower=-2.094 upper=2.094 effort=7 velocity=20; origin xyz=0.02895 0 0.0865 rpy=-3.1416 0 0 -> xyz=0.02895 0 -0.0845
- joint joint8: origin xyz=0.08657 -0.0249 -0.00024366 -> xyz=0.08397 -0.023638 -0.0062703

File: arx5_description/xacro/X5_ac1.xacro (robot description, xacro)
@@ -1,341 +1,345 @@
 <?xml version="1.0"?>
 <robot xmlns:xacro="http://www.ros.org/wiki/xacro">
-  <xacro:macro name="X5" params="name camera:=d405">
-    <xacro:property name="prefix" value="${name + '_' if name else ''}"/>
-    <link name="${prefix}base_link">
-      <inertial>
-        <origin xyz="-3.0001E-05 3.0589E-05 0.027324"/>
-        <mass value="0.43995"/>
-        <inertia
-            ixx="0.00017"
-            ixy="0.00000"
-            ixz="0.00000"
-            iyy="0.00017"
-            iyz="0.00000"
-            izz="0.00016"/>
-      </inertial>
-      <visual>
-        <geometry>
-          <mesh filename="file://$(find arx5_description)/meshes/x5/base_link.glb"/>
-        </geometry>
-      </visual>
-      <collision>
-        <geometry>
-          <mesh filename="file://$(find arx5_description)/meshes/x5/base_link.glb"/>
-        </geometry>
-      </collision>
-    </link>
-    <link name="${prefix}link1">
-      <inertial>
-        <origin xyz="0.0054231 -0.0080289 0.017086"/>
-        <mass value="0.066982" />
-        <inertia
-            ixx="0.00008086"
-            ixy="0.00000207"
-            ixz="-0.00000876"
-            iyy="0.00003211"
-            iyz="0.00000440"
-            izz="0.00007702" />
-      </inertial>
-      <visual>
-        <geometry>
-          <mesh filename="file://$(find arx5_description)/meshes/x5/link1.glb"/>
-        </geometry>
-      </visual>
-      <collision>
-        <geometry>
-          <mesh filename="file://$(find arx5_description)/meshes/x5/link1.glb"/>
-        </geometry>
-      </collision>
-    </link>
-    <joint name="${prefix}joint1" type="revolute">
-      <origin xyz="0 0 0.0605"/>
-      <parent link="${prefix}base_link"/>
-      <child link="${prefix}link1"/>
-      <axis xyz="0 0 1"/>
-      <limit lower="-2.094" upper="3.1416" effort="27" velocity="5.5" />
-    </joint>
-    <link name="${prefix}link2">
-      <inertial>
-        <origin xyz="-0.13234 -0.0040166 0.00010941" />
-        <mass value="1.1068" />
-        <inertia
-            ixx="0.00054299"
-            ixy="-0.00000184"
-            ixz="0.00003884"
-            iyy="0.01652639"
-            iyz="-0.00000035"
-            izz="0.01654931" />
-      </inertial>
-      <visual>
-        <geometry>
-          <mesh filename="file://$(find arx5_description)/meshes/x5/link2.glb"/>
-        </geometry>
-      </visual>
-      <collision>
-        <geometry>
-          <mesh filename="file://$(find arx5_description)/meshes/x5/link2.glb"/>
-        </geometry>
-      </collision>
-    </link>
-    <joint name="${prefix}joint2" type="revolute">
-      <origin xyz="0.02 0 0.04"/>
-      <parent link="${prefix}link1"/>
-      <child link="${prefix}link2"/>
-      <axis xyz="0 1 0"/>
-      <limit lower="0" upper="3.66" effort="100" velocity="5"/>
-    </joint>
-    <link name="${prefix}link3">
-      <inertial>
-        <origin xyz="0.18531 0.00068376 -0.051638"/>
-        <mass value="0.54534"/>
-        <inertia
-            ixx="0.00036"
-            ixy="-0.00003"
-            ixz="-0.00039"
-            iyy="0.00423"
-            iyz="0.00001"
-            izz="0.00420"/>
-      </inertial>
-      <visual>
-        <geometry>
-          <mesh filename="file://$(find arx5_description)/meshes/x5/link3.glb"/>
-        </geometry>
-      </visual>
-      <collision>
-        <geometry>
-          <mesh filename="file://$(find arx5_description)/meshes/x5/link3.glb"/>
-        </geometry>
-      </collision>
-    </link>
-    <joint name="${prefix}joint3" type="revolute">
-      <origin xyz="-0.264 0 0" rpy="3.1416 0 0"/>
-      <parent link="${prefix}link2"/>
-      <child link="${prefix}link3"/>
-      <axis xyz="0 1 0"/>
-      <limit lower="0" upper="3.14" effort="100" velocity="5"/>
-    </joint>
-    <link name="${prefix}link4">
-      <inertial>
-        <origin xyz="0.040231 0.0044807 -0.035335"/>
-        <mass value="0.11714"/>
-        <inertia
-            ixx="0.00019"
-            ixy="-0.00002"
-            ixz="-0.00009"
-            iyy="0.00023"
-            iyz="0.00002"
-            izz="0.00014"/>
-      </inertial>
-      <visual>
-        <geometry>
-          <mesh filename="file://$(find arx5_description)/meshes/x5/link4.glb"/>
-        </geometry>
-      </visual>
-      <collision>
-        <geometry>
-          <mesh filename="file://$(find arx5_description)/meshes/x5/link4.glb"/>
-        </geometry>
-      </collision>
-    </link>
-    <joint name="${prefix}joint4" type="revolute">
-      <origin xyz="0.245 0 -0.056"/>
-      <parent link="${prefix}link3"/>
-      <child link="${prefix}link4"/>
-      <axis xyz="0 1 0"/>
-      <limit lower="-1.57" upper="1.57" effort="100" velocity="5"/>
-    </joint>
-    <link name="${prefix}link5">
-      <inertial>
-        <origin xyz="0.003612 -1.5455E-05 0.055214"/>
-        <mass value="0.63488"/>
-        <inertia
-            ixx="0.00083"
-            ixy="0.00000"
-            ixz="0.00007"
-            iyy="0.00082"
-            iyz="0.00000"
-            izz="0.00026"/>
-      </inertial>
-      <visual>
-        <origin xyz="0.0037 0 0"/>
-        <geometry>
-          <mesh filename="file://$(find arx5_description)/meshes/x5/link5.glb"/>
-        </geometry>
-      </visual>
-      <collision>
-        <geometry>
-          <mesh filename="file://$(find arx5_description)/meshes/x5/link5.glb"/>
-        </geometry>
-      </collision>
-    </link>
-    <joint name="${prefix}joint5" type="revolute">
-      <origin xyz="0.06775 0.0005 -0.0865"/>
-      <parent link="${prefix}link4"/>
-      <child link="${prefix}link5"/>
-      <axis xyz="0 0 1"/>
-      <limit lower="-1.57" upper="1.57" effort="100" velocity="5"/>
-    </joint>
-    <link name="${prefix}link6">
-      <inertial>
-        <origin xyz="0.041697 2.4368E-05 0.00014464"/>
-        <mass value="0.44089"/>
-        <inertia
-            ixx="0.00038"
-            ixy="0.00000"
-            ixz="0.00000"
-            iyy="0.00028"
-            iyz="0.00000"
-            izz="0.00050"/>
-      </inertial>
-      <visual>
-        <geometry>
-          <mesh filename="file://$(find arx5_description)/meshes/ac1/link6.glb"/>
-        </geometry>
-      </visual>
-      <collision>
-        <geometry>
-          <mesh filename="file://$(find arx5_description)/meshes/ac1/link6.glb"/>
-        </geometry>
-      </collision>
-    </link>
-    <joint name="${prefix}joint6" type="revolute">
-      <origin xyz="0.02895 0 0.0865" rpy="-3.1416 0 0"/>
-      <parent link="${prefix}link5"/>
-      <child link="${prefix}link6"/>
-      <axis xyz="1 0 0"/>
-      <limit lower="-1.57" upper="1.57" effort="100" velocity="5"/>
-    </joint>
-    <link name="${prefix}link7">
-      <inertial>
-        <origin xyz="-0.00035522 -0.007827 -0.0029883"/>
-        <mass value="0.064798"/>
-        <inertia
-            ixx="0.00002"
-            ixy="0.00000"
-            ixz="0.00000"
-            iyy="0.00003"
-            iyz="0.00000"
-            izz="0.00003"/>
-      </inertial>
-      <visual>
-        <geometry>
-          <mesh filename="file://$(find arx5_description)/meshes/ac1/link7.glb"/>
-        </geometry>
-      </visual>
-      <collision>
-        <geometry>
-          <mesh filename="file://$(find arx5_description)/meshes/ac1/link7.glb"/>
-        </geometry>
-      </collision>
-    </link>
-    <joint name="${prefix}gripper_joint" type="prismatic">
-      <origin xyz="0.08657 0.024896 -0.0002436"/>
-      <parent link="${prefix}link6"/>
-      <child link="${prefix}link7"/>
-      <axis xyz="0 1 0"/>
-      <limit lower="0" upper="0.044" effort="100" velocity="5"/>
-    </joint>
-    <link name="${prefix}link8">
-      <inertial>
-        <origin xyz="-0.00035522 0.0078277 0.0024201"/>
-        <mass value="0.064798"/>
-        <inertia
-            ixx="0.00002"
-            ixy="0.00000"
-            ixz="0.00000"
-            iyy="0.00003"
-            iyz="0.00000"
-            izz="0.00003"/>
-      </inertial>
-      <visual>
-        <geometry>
-          <mesh filename="file://$(find arx5_description)/meshes/ac1/link8.glb"/>
-        </geometry>
-      </visual>
-      <collision>
-        <geometry>
-          <mesh filename="file://$(find arx5_description)/meshes/ac1/link8.glb"/>
-        </geometry>
-      </collision>
-    </link>
-    <joint name="${prefix}joint8" type="prismatic">
-      <origin xyz="0.08657 -0.0249 -0.00024366"/>
-      <parent link="${prefix}link6"/>
-      <child link="${prefix}link8"/>
-      <axis xyz="0 -1 0"/>
-      <limit lower="0" upper="0.044" effort="100" velocity="5"/>
-      <mimic joint="${prefix}gripper_joint" multiplier="1" offset="0"/>
-    </joint>
-    <link name="${prefix}gripper_center"/>
-    <joint name="${prefix}gripper_center_fixed" type="fixed">
-      <parent link="${prefix}link6"/>
-      <child link="${prefix}gripper_center"/>
-      <origin xyz="0.145 0 0.006376" />
-    </joint>
-    <link name="${prefix}left_pad"/>
-    <joint name="${prefix}left_pad_joint" type="fixed">
-      <parent link="${prefix}link7"/>
-      <child link="${prefix}left_pad"/>
-      <origin xyz="0.05843 -0.0249 0.006376" />
-    </joint>
-    <link name="${prefix}right_pad"/>
-    <joint name="${prefix}right_pad_joint" type="fixed">
-      <parent link="${prefix}link8"/>
-      <child link="${prefix}right_pad"/>
-      <origin xyz="0.05843 0.0249 0.006376" />
-    </joint>
-    <xacro:if value="${camera == 'd405'}">
-      <link name="${prefix}camera_support">
-        <visual>
-          <geometry>
-            <mesh filename="file://$(find arx5_description)/meshes/camera_stand/stand_d405.glb"/>
-          </geometry>
-        </visual>
-      </link>
-      <joint name="${prefix}camera_support_fixed" type="fixed">
-        <parent link="${prefix}link6"/>
-        <child link="${prefix}camera_support"/>
-        <origin xyz="0.045 0 0.021"/>
-      </joint>
-      <link name="${prefix}camera">
-        <visual>
-          <geometry>
-            <mesh filename="file://$(find sensor_models)/meshes/d405.glb"/>
-          </geometry>
-        </visual>
-      </link>
-      <joint name="${prefix}camera_fixed" type="fixed">
-        <origin xyz="0.0385 0 0.0475" rpy="0 0.523 0"/>
-        <parent link="${prefix}camera_support"/>
-        <child link="${prefix}camera"/>
-      </joint>
-    </xacro:if>
-    <xacro:if value="${camera == 'd435'}">
-      <link name="${prefix}camera_support">
-        <visual>
-          <geometry>
-            <mesh filename="file://$(find arx5_description)/meshes/camera_stand/stand_d435.glb"/>
-          </geometry>
-        </visual>
-      </link>
-      <joint name="${prefix}camera_support_fixed" type="fixed">
-        <parent link="${prefix}link6"/>
-        <child link="${prefix}camera_support"/>
-        <origin xyz="0.045 0 0.021"/>
-      </joint>
-      <link name="${prefix}camera">
-        <visual>
-          <geometry>
-            <mesh filename="file://$(find sensor_models)/meshes/d435.glb"/>
-          </geometry>
-        </visual>
-      </link>
-      <joint name="${prefix}camera_fixed" type="fixed">
-        <origin xyz="0.03 0 0.034113" />
-        <parent link="${prefix}camera_support"/>
-        <child link="${prefix}camera"/>
-      </joint>
-    </xacro:if>
-  </xacro:macro>
+	<xacro:property name="PI" value="3.1415926535897931"/>
+	<xacro:macro name="X5" params="name camera:=d405">
+		<xacro:property name="prefix" value="${name + '_' if name else ''}"/>
+		<link name="${prefix}base_link">
+			<inertial>
+				<origin xyz="-3.0001E-05 3.0589E-05 0.027324"/>
+				<mass value="0.43995"/>
+				<inertia
+						ixx="0.00017"
+						ixy="0.00000"
+						ixz="0.00000"
+						iyy="0.00017"
+						iyz="0.00000"
+						izz="0.00016"/>
+			</inertial>
+			<visual>
+				<geometry>
+					<mesh filename="file://$(find arx5_description)/meshes/x5/base_link.glb"/>
+				</geometry>
+			</visual>
+			<collision>
+				<geometry>
+					<mesh filename="file://$(find arx5_description)/meshes/x5/base_link.glb"/>
+				</geometry>
+			</collision>
+		</link>
+		<link name="${prefix}link1">
+			<inertial>
+				<origin xyz="0.0054231 -0.0080289 0.017086"/>
+				<mass value="0.066982"/>
+				<inertia
+						ixx="0.00008086"
+						ixy="0.00000207"
+						ixz="-0.00000876"
+						iyy="0.00003211"
+						iyz="0.00000440"
+						izz="0.00007702"/>
+			</inertial>
+			<visual>
+				<geometry>
+					<mesh filename="file://$(find arx5_description)/meshes/x5/link1.glb"/>
+				</geometry>
+			</visual>
+			<collision>
+				<geometry>
+					<mesh filename="file://$(find arx5_description)/meshes/x5/link1.glb"/>
+				</geometry>
+			</collision>
+		</link>
+		<joint name="${prefix}joint1" type="revolute">
+			<origin xyz="0 0 0.0605"/>
+			<parent link="${prefix}base_link"/>
+			<child link="${prefix}link1"/>
+			<axis xyz="0 0 1"/>
+			<limit lower="-2.094" upper="${PI}" effort="27" velocity="5.5"/>
+		</joint>
+		<link name="${prefix}link2">
+			<inertial>
+				<origin xyz="-0.13234 -0.0040166 0.00010941"/>
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