Commit message: update arx5 to glb mesh

File: arx5_description/urdf/arx5.urdf (robot description, URDF)
Before this commit: robot ARX 5, 14 links, 13 joints
Links:
- link base_link: geometry collision mesh filename=package://arx5_description/meshes/x5/base_link.glb; visual mesh filename=package://arx5_description/meshes/x5/base_link.glb
- link camera: geometry visual mesh filename=file:///home/fiveages/ros2_ws/install/sensor_models/share/s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
- link camera_support: geometry visual mesh filename=package://arx5_description/meshes/camera_stand/stand_d405.g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
- link link1: geometry collision mesh filename=package://arx5_description/meshes/x5/link1.glb; visual mesh filename=package://arx5_description/meshes/x5/link1.glb
- link link2: geometry collision mesh filename=package://arx5_description/meshes/x5/link2.glb; visual mesh filename=package://arx5_description/meshes/x5/link2.glb
- link link3: geometry collision mesh filename=package://arx5_description/meshes/x5/link3.glb; visual mesh filename=package://arx5_description/meshes/x5/link3.glb
- link link4: geometry collision mesh filename=package://arx5_description/meshes/x5/link4.glb; visual mesh filename=package://arx5_description/meshes/x5/link4.glb
- link link5: geometry collision mesh filename=package://arx5_description/meshes/x5/link5.glb; visual mesh filename=package://arx5_description/meshes/x5/link5.glb
- link link6: geometry collision mesh filename=package://arx5_description/meshes/r5/link6.glb; visual mesh filename=package://arx5_description/meshes/r5/link6.glb
- link link7: geometry collision mesh filename=package://arx5_description/meshes/r5/link7.glb; visual mesh filename=package://arx5_description/meshes/r5/link7.glb
- link link8: geometry collision mesh filename=package://arx5_description/meshes/r5/link8.glb; visual mesh filename=package://arx5_description/meshes/r5/link8.glb

File: arx5_description/urdf/arx5_ac1.urdf (robot description, URDF)
Before this commit: robot ARX 5, 14 links, 13 joints
Links:
- link base_link: mass 0.42272 -> 0.43995; geometry collision mesh filename=package://arx5_description/meshes/x5/base_link.glb; visual mesh filename=package://arx5_description/meshes/x5/base_link.glb
- link camera: geometry visual mesh filename=file:///home/fiveages/ros2_ws/install/sensor_models/share/s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
- link link1: mass 0.096804 -> 0.066982; geometry collision mesh filename=package://arx5_description/meshes/x5/link1.glb; visual mesh filename=package://arx5_description/meshes/x5/link1.glb
- link link2: mass 1.1988 -> 1.1068; geometry collision mesh filename=package://arx5_description/meshes/x5/link2.glb; visual mesh filename=package://arx5_description/meshes/x5/link2.glb
- link link3: mass 0.84082 -> 0.54534; geometry collision mesh filename=package://arx5_description/meshes/x5/link3.glb; visual mesh filename=package://arx5_description/meshes/x5/link3.glb
- link link4: mass 0.12432 -> 0.11714; geometry collision mesh filename=package://arx5_description/meshes/x5/link4.glb; visual mesh filename=package://arx5_description/meshes/x5/link4.glb
- link link5: mass 0.63601 -> 0.63488; geometry collision mesh filename=package://arx5_description/meshes/x5/link5.glb; visual mesh filename=package://arx5_description/meshes/x5/link5.glb
- link link6: geometry collision mesh filename=package://arx5_description/meshes/ac1/link6.glb; visual mesh filename=package://arx5_description/meshes/ac1/link6.glb
- link link7: geometry collision mesh filename=package://arx5_description/meshes/ac1/link7.glb; visual mesh filename=package://arx5_description/meshes/ac1/link7.glb
- link link8: mass 0.0647981725781684 -> 0.064798; geometry collision mesh filename=package://arx5_description/meshes/ac1/link8.glb; visual mesh filename=package://arx5_description/meshes/ac1/link8.glb
Joints:
- joint gripper_center_fixed: origin xyz=0.08657 0 0 -> xyz=0.145 0 0.006376
- joint joint1: limit lower=-2.618 upper=2.168 effort=100 velocity=5 -> lower=-2.094 upper=3.1416 effort=27 velocity=5.5; origin xyz=0 0 0.0565 -> xyz=0 0 0.0605
- joint joint2: origin xyz=0.02 0 0.047 -> xyz=0.02 0 0.04
- joint joint3: origin xyz=-0.264 0 0 rpy=-3.1416 0 0 -> xyz=-0.264 0 0 rpy=3.1416 0 0
- joint joint4: origin xyz=0.245 -5E-05 -0.06 -> xyz=0.245 0 -0.056
- joint joint5: origin xyz=0.0702 5E-05 -0.083391 -> xyz=0.06775 0.0005 -0.0865
- joint joint6: origin xyz=0.025286 0 0.083391 rpy=3.1416 0 0 -> xyz=0.02895 0 0.0865 rpy=-3.1416 0 0
- joint left_pad_joint: origin xyz=0.05843 -0.0249 0 -> xyz=0.05843 -0.0249 0.006376
- joint right_pad_joint: origin xyz=0.05843 0.0249 0 -> xyz=0.05843 0.0249 0.006376

File: arx5_description/urdf/arx5_r5.urdf (robot description, URDF)
Before this commit: robot ARX 5, 14 links, 13 joints
Links:
- link base_link: geometry collision mesh filename=package://arx5_description/meshes/r5/base_link.glb; visual mesh filename=package://arx5_description/meshes/r5/base_link.glb
- link camera: geometry visual mesh filename=package://sensor_models/meshes/d405/d405.glb
- link camera_support: geometry visual mesh filename=package://arx5_description/meshes/camera_stand/stand_d405.g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
- link link1: geometry collision mesh filename=package://arx5_description/meshes/r5/link1.glb; visual mesh filename=package://arx5_description/meshes/r5/link1.glb
- link link2: geometry collision mesh filename=package://arx5_description/meshes/r5/link2.glb; visual mesh filename=package://arx5_description/meshes/r5/link2.glb
- link link3: geometry collision mesh filename=package://arx5_description/meshes/r5/link3.glb; visual mesh filename=package://arx5_description/meshes/r5/link3.glb
- link link4: geometry collision mesh filename=package://arx5_description/meshes/r5/link4.glb; visual mesh filename=package://arx5_description/meshes/r5/link4.glb
- link link5: geometry collision mesh filename=package://arx5_description/meshes/r5/link5.glb; visual mesh filename=package://arx5_description/meshes/r5/link5.glb
- link link6: geometry collision mesh filename=package://arx5_description/meshes/r5/link6.glb; visual mesh filename=package://arx5_description/meshes/r5/link6.glb
- link link7: geometry collision mesh filename=package://arx5_description/meshes/r5/link7.glb; visual mesh filename=package://arx5_description/meshes/r5/link7.glb
- link link8: geometry collision mesh filename=package://arx5_description/meshes/r5/link8.glb; visual mesh filename=package://arx5_description/meshes/r5/link8.glb

File: arx5_description/xacro/R5.xacro (robot description, xacro)
@@ -17,10 +17,10 @@
 			<visual>
 				<geometry>
-					<mesh filename="file://$(find arx5_description)/meshes/r5/base_link.obj"/>
-				</geometry>
-			</visual>
-			<collision>
-				<geometry>
-					<mesh filename="file://$(find arx5_description)/meshes/r5/base_link.obj"/>
+					<mesh filename="file://$(find arx5_description)/meshes/r5/base_link.glb"/>
+				</geometry>
+			</visual>
+			<collision>
+				<geometry>
+					<mesh filename="file://$(find arx5_description)/meshes/r5/base_link.glb"/>
 				</geometry>
 			</collision>
@@ -40,10 +40,10 @@
 			<visual>
 				<geometry>
-					<mesh filename="file://$(find arx5_description)/meshes/r5/link1.obj"/>
-				</geometry>
-			</visual>
-			<collision>
-				<geometry>
-					<mesh filename="file://$(find arx5_description)/meshes/r5/link1.obj"/>
+					<mesh filename="file://$(find arx5_description)/meshes/r5/link1.glb"/>
+				</geometry>
+			</visual>
+			<collision>
+				<geometry>
+					<mesh filename="file://$(find arx5_description)/meshes/r5/link1.glb"/>
 				</geometry>
 			</collision>
@@ -71,8 +71,8 @@
 				<geometry>
 					<xacro:if value="${style == 'agilex'}">
-						<mesh filename="file://$(find arx5_description)/meshes/r5/link2_agilex.obj"/>
+						<mesh filename="file://$(find arx5_description)/meshes/r5/link2_agilex.glb"/>
 					</xacro:if>
 					<xacro:if value="${style == 'default'}">
-						<mesh filename="file://$(find arx5_description)/meshes/r5/link2.obj"/>
+						<mesh filename="file://$(find arx5_description)/meshes/r5/link2.glb"/>
 					</xacro:if>
 				</geometry>
@@ -80,5 +80,5 @@
 			<collision>
 				<geometry>
-					<mesh filename="file://$(find arx5_description)/meshes/r5/link2.obj"/>
+					<mesh filename="file://$(find arx5_description)/meshes/r5/link2.glb"/>
 				</geometry>
 			</collision>
@@ -106,8 +106,8 @@
 				<geometry>
 					<xacro:if value="${style == 'agilex'}">
-						<mesh filename="file://$(find arx5_description)/meshes/r5/link3_agilex.obj"/>
+						<mesh filename="file://$(find arx5_description)/meshes/r5/link3_agilex.glb"/>
 					</xacro:if>
 					<xacro:if value="${style == 'default'}">
-						<mesh filename="file://$(find arx5_description)/meshes/r5/link3.obj"/>
+						<mesh filename="file://$(find arx5_description)/meshes/r5/link3.glb"/>
 					</xacro:if>
 				</geometry>
@@ -115,5 +115,5 @@
 			<collision>
 				<geometry>
-					<mesh filename="file://$(find arx5_description)/meshes/r5/link3.obj"/>
+					<mesh filename="file://$(find arx5_description)/meshes/r5/link3.glb"/>
 				</geometry>
 			</collision>
@@ -140,10 +140,10 @@
 			<visual>
 				<geometry>
-					<mesh filename="file://$(find arx5_description)/meshes/r5/link4.obj"/>
-				</geometry>
-			</visual>
-			<collision>
-				<geometry>
-					<mesh filename="file://$(find arx5_description)/meshes/r5/link4.obj"/>
+					<mesh filename="file://$(find arx5_description)/meshes/r5/link4.glb"/>
+				</geometry>
+			</visual>
+			<collision>
+				<geometry>
+					<mesh filename="file://$(find arx5_description)/meshes/r5/link4.glb"/>
 				</geometry>
 			</collision>
@@ -170,10 +170,10 @@
 			<visual>
 				<geometry>
-					<mesh filename="file://$(find arx5_description)/meshes/r5/link5.obj"/>
-				</geometry>
-			</visual>
-			<collision>
-				<geometry>
-					<mesh filename="file://$(find arx5_description)/meshes/r5/link5.obj"/>
+					<mesh filename="file://$(find arx5_description)/meshes/r5/link5.glb"/>
+				</geometry>
+			</visual>
+			<collision>
+				<geometry>
+					<mesh filename="file://$(find arx5_description)/meshes/r5/link5.glb"/>
 				</geometry>
 			</collision>
@@ -200,10 +200,10 @@
 			<visual>
 				<geometry>
-					<mesh filename="file://$(find arx5_description)/meshes/r5/link6.obj"/>
-				</geometry>
-			</visual>
-			<collision>
-				<geometry>
-					<mesh filename="file://$(find arx5_description)/meshes/r5/link6.obj"/>
+					<mesh filename="file://$(find arx5_description)/meshes/r5/link6.glb"/>
+				</geometry>
+			</visual>
+			<collision>
+				<geometry>
+					<mesh filename="file://$(find arx5_description)/meshes/r5/link6.glb"/>
 				</geometry>
 			</collision>
@@ -230,10 +230,10 @@
 			<visual>
 				<geometry>
-					<mesh filename="file://$(find arx5_description)/meshes/r5/link7.obj"/>
-				</geometry>
-			</visual>
-			<collision>
-				<geometry>
-					<mesh filename="file://$(find arx5_description)/meshes/r5/link7.obj"/>
+					<mesh filename="file://$(find arx5_description)/meshes/r5/link7.glb"/>
+				</geometry>
+			</visual>
+			<collision>
+				<geometry>
+					<mesh filename="file://$(find arx5_description)/meshes/r5/link7.glb"/>
 				</geometry>
 			</collision>
@@ -260,10 +260,10 @@
 			<visual>
 				<geometry>
-					<mesh filename="file://$(find arx5_description)/meshes/r5/link8.obj"/>
-				</geometry>
-			</visual>
-			<collision>
-				<geometry>
-					<mesh filename="file://$(find arx5_description)/meshes/r5/link8.obj"/>
+					<mesh filename="file://$(find arx5_description)/meshes/r5/link8.glb"/>
+				</geometry>
+			</visual>
+			<collision>
+				<geometry>
+					<mesh filename="file://$(find arx5_description)/meshes/r5/link8.glb"/>
 				</geometry>
 			</collision>
@@ -299,5 +299,5 @@
 				<visual>
 					<geometry>
-						<mesh filename="file://$(find arx5_description)/meshes/camera_stand/stand_d405.obj"/>
+						<mesh filename="file://$(find arx5_description)/meshes/camera_stand/stand_d405.glb"/>
 					</geometry>
 				</visual>
@@ -311,5 +311,5 @@
 				<visual>
 					<geometry>
-						<mesh filename="file://$(find sensor_models)/meshes/d405/d405.obj"/>
+						<mesh filename="file://$(find sensor_models)/meshes/d405.glb"/>
 					</geometry>
 				</visual>
@@ -325,5 +325,5 @@
 				<visual>
 					<geometry>
-						<mesh filename="file://$(find arx5_description)/meshes/camera_stand/stand_d435.obj"/>
+						<mesh filename="file://$(find arx5_description)/meshes/camera_stand/stand_d435.glb"/>
 					</geometry>
 				</visual>
@@ -337,5 +337,5 @@
 				<visual>
 					<geometry>
-						<mesh filename="file://$(find sensor_models)/meshes/d435/d435.obj"/>
+						<mesh filename="file://$(find sensor_models)/meshes/d435.glb"/>
 					</geometry>
 				</visual>

File: arx5_description/xacro/X5_ac1.xacro (robot description, xacro)
@@ -29,12 +29,12 @@
       <inertial>
         <origin xyz="0.0054231 -0.0080289 0.017086"/>
-        <mass value="0.066982"/>
-        <inertia
-            ixx="0.00008"
-            ixy="0.00000"
-            ixz="0.00001"
-            iyy="0.00003"
-            iyz="0.00000"
-            izz="0.00008"/>
+        <mass value="0.066982" />
+        <inertia
+            ixx="0.00008086"
+            ixy="0.00000207"
+            ixz="-0.00000876"
+            iyy="0.00003211"
+            iyz="0.00000440"
+            izz="0.00007702" />
       </inertial>
       <visual>
@@ -54,17 +54,17 @@
       <child link="${prefix}link1"/>
       <axis xyz="0 0 1"/>
-      <limit lower="-2.87" upper="3.14" effort="100" velocity="5"/>
+      <limit lower="-2.094" upper="3.1416" effort="27" velocity="5.5" />
     </joint>
     <link name="${prefix}link2">
       <inertial>
-        <origin xyz="-0.13237 0.0020852 0.00010549"/>
-        <mass value="1.0795"/>
-        <inertia
-            ixx="0.00051"
-            ixy="0.00001"
-            ixz="-0.00004"
-            iyy="0.01599"
-            iyz="0.00000"
-            izz="0.01605"/>
+        <origin xyz="-0.13234 -0.0040166 0.00010941" />
+        <mass value="1.1068" />
+        <inertia
+            ixx="0.00054299"
+            ixy="-0.00000184"
+            ixz="0.00003884"
+            iyy="0.01652639"
+            iyz="-0.00000035"
+            izz="0.01654931" />
       </inertial>
       <visual>
@@ -191,10 +191,10 @@
       <visual>
         <geometry>
-          <mesh filename="file://$(find arx5_description)/meshes/r5/link6.glb"/>
-        </geometry>
-      </visual>
-      <collision>
-        <geometry>
-          <mesh filename="file://$(find arx5_description)/meshes/r5/link6.glb"/>
+          <mesh filename="file://$(find arx5_description)/meshes/ac1/link6.glb"/>
+        </geometry>
+      </visual>
+      <collision>
+        <geometry>
+          <mesh filename="file://$(find arx5_description)/meshes/ac1/link6.glb"/>
         </geometry>
       </collision>
@@ -221,10 +221,10 @@
       <visual>
         <geometry>
-          <mesh filename="file://$(find arx5_description)/meshes/r5/link7.glb"/>
-        </geometry>
-      </visual>
-      <collision>
-        <geometry>
-          <mesh filename="file://$(find arx5_description)/meshes/r5/link7.glb"/>
+          <mesh filename="file://$(find arx5_description)/meshes/ac1/link7.glb"/>
+        </geometry>
+      </visual>
+      <collision>
+        <geometry>
+          <mesh filename="file://$(find arx5_description)/meshes/ac1/link7.glb"/>
         </geometry>
       </collision>
@@ -251,10 +251,10 @@
       <visual>
         <geometry>
-          <mesh filename="file://$(find arx5_description)/meshes/r5/link8.glb"/>
-        </geometry>
-      </visual>
-      <collision>
-        <geometry>
-          <mesh filename="file://$(find arx5_description)/meshes/r5/link8.glb"/>
+          <mesh filename="file://$(find arx5_description)/meshes/ac1/link8.glb"/>
+        </geometry>
+      </visual>
+      <collision>
+        <geometry>
+          <mesh filename="file://$(find arx5_description)/meshes/ac1/link8.glb"/>
         </geometry>
       </collision>
@@ -272,5 +272,5 @@
       <parent link="${prefix}link6"/>
       <child link="${prefix}gripper_center"/>
-      <origin xyz="0.145 0 0" />
+      <origin xyz="0.145 0 0.006376" />
     </joint>
     <link name="${prefix}left_pad"/>
@@ -278,5 +278,5 @@
       <parent link="${prefix}link7"/>
       <child link="${prefix}left_pad"/>
-      <origin xyz="0.05843 -0.0249 0" />
+      <origin xyz="0.05843 -0.0249 0.006376" />
     </joint>
     <link name="${prefix}right_pad"/>
@@ -284,5 +284,5 @@
       <parent link="${prefix}link8"/>
       <child link="${prefix}right_pad"/>
-      <origin xyz="0.05843 0.0249 0" />
+      <origin xyz="0.05843 0.0249 0.006376" />
     </joint>
     <xacro:if value="${camera == 'd405'}">
@@ -328,5 +328,5 @@
         <visual>
           <geometry>
-            <mesh filename="file://$(find sensor_models)/meshes/d435/d435.glb"/>
+            <mesh filename="file://$(find sensor_models)/meshes/d435.glb"/>
           </geometry>
         </visual>

File: arx5_description/xacro/robot.xacro (robot description, xacro)
@@ -10,4 +10,8 @@
     <xacro:X5 name=""/>
   </xacro:if>
+  <xacro:if value="${'$(arg type)' == 'ac1'}">
+    <xacro:include filename="$(find arx5_description)/xacro/X5_ac1.xacro"/>
+    <xacro:X5 name=""/>
+  </xacro:if>
   <xacro:if value="${'$(arg type)' == 'agilex'}">
     <xacro:include filename="$(find arx5_description)/xacro/R5.xacro"/>
