Commit message: 修复模型路径问题，补充完整r5和agilex设置

File: arx5_description/urdf/arx5.urdf (robot description, URDF)
Before this commit: robot ARX 5, 14 links, 13 joints
Links:
- link base_link: geometry collision cylinder length=0.03125 radius=0.031; visual mesh filename=package://arx5_description/meshes/x5/base_link.glb
- link camera: geometry collision box size=0.0231 0.0421 0.042; visual mesh filename=package://sensor_models/meshes/d405/d405.obj
- link camera_support: geometry collision box size=0.01 0.05 0.03; collision box size=0.01 0.05 0.06
- link link1: geometry collision mesh filename=package://arx5_description/meshes/x5/link1.glb; visual mesh filename=package://arx5_description/meshes/x5/link1.glb
- link link2: geometry collision box size=0.264 0.05 0.05; collision cylinder length=0.0665 radius=0.028
- link link3: geometry collision box size=0.2 0.04 0.045; collision cylinder length=0.049 radius=0.03
- link link4: geometry collision cylinder length=0.04 radius=0.0315; visual mesh filename=package://arx5_description/meshes/x5/link4.glb
- link link5: geometry collision cylinder length=0.013 radius=0.03145; collision cylinder length=0.045 radius=0.03145
- link link6: geometry collision cylinder length=0.064 radius=0.03015; visual mesh filename=package://arx5_description/meshes/r5/link6.glb
- link link7: geometry collision box size=0.08 0.04 0.0640; visual mesh filename=package://arx5_description/meshes/r5/link7.glb
- link link8: geometry collision box size=0.08 0.04 0.0640; visual mesh filename=package://arx5_description/meshes/r5/link8.glb

File: arx5_description/urdf/arx5_ac1.urdf (robot description, URDF)
Before this commit: robot ARX 5, 14 links, 13 joints
Links:
- link base_link: geometry collision cylinder length=0.03125 radius=0.031; visual mesh filename=package://arx5_description/meshes/x5/base_link.glb
- link camera: geometry collision box size=0.0231 0.0421 0.042; visual mesh filename=package://sensor_models/meshes/d405/d405.obj
- link camera_support: geometry collision box size=0.01 0.05 0.03; collision box size=0.01 0.05 0.06
- link link1: geometry collision mesh filename=package://arx5_description/meshes/x5/link1.glb; visual mesh filename=package://arx5_description/meshes/x5/link1.glb
- link link2: geometry collision box size=0.264 0.05 0.05; collision cylinder length=0.0665 radius=0.028
- link link3: geometry collision box size=0.2 0.04 0.045; collision cylinder length=0.049 radius=0.03
- link link4: geometry collision cylinder length=0.04 radius=0.0315; visual mesh filename=package://arx5_description/meshes/x5/link4.glb
- link link5: geometry collision cylinder length=0.013 radius=0.03145; collision cylinder length=0.045 radius=0.03145
- link link6: geometry collision cylinder length=0.064 radius=0.03015; visual mesh filename=package://arx5_description/meshes/ac1/link6.glb
- link link7: geometry collision box size=0.08 0.04 0.0640; visual mesh filename=package://arx5_description/meshes/ac1/link7.glb
- link link8: geometry collision box size=0.08 0.04 0.0640; visual mesh filename=package://arx5_description/meshes/ac1/link8.glb

File: arx5_description/urdf/arx5_agilex.urdf (robot description, URDF)
Before this commit: robot ARX 5, 14 links, 13 joints
Links:
- link base_link: geometry collision cylinder length=0.0625 radius=0.0305; visual mesh filename=package://arx5_description/meshes/r5/base_link.glb
- link camera: geometry collision box size=0.0231 0.0421 0.042; visual mesh filename=package://sensor_models/meshes/d405/d405.obj
- link camera_support: geometry collision box size=0.01 0.05 0.03; collision box size=0.01 0.05 0.06
- link link2: geometry collision box size=0.264 0.051 0.05; collision cylinder length=0.0665 radius=0.03
- link link3: geometry collision box size=0.25 0.048 0.05; collision cylinder length=0.054 radius=0.032
- link link4: geometry collision cylinder length=0.04 radius=0.0315; visual mesh filename=package://arx5_description/meshes/r5/link4.glb
- link link5: geometry collision cylinder length=0.013 radius=0.03145; collision cylinder length=0.045 radius=0.03145
- link link6: geometry collision cylinder length=0.064 radius=0.03015; visual mesh filename=package://arx5_description/meshes/r5/link6.glb
- link link7: geometry collision box size=0.08 0.04 0.0640; visual mesh filename=package://arx5_description/meshes/r5/link7.glb
- link link8: geometry collision box size=0.08 0.04 0.0640; visual mesh filename=package://arx5_description/meshes/r5/link8.glb

File: arx5_description/urdf/arx5_r5.urdf (robot description, URDF)
Before this commit: robot ARX 5, 14 links, 13 joints
Links:
- link base_link: geometry collision cylinder length=0.0625 radius=0.0305; visual mesh filename=package://arx5_description/meshes/r5/base_link.glb
- link camera: geometry collision box size=0.0231 0.0421 0.042; visual mesh filename=package://sensor_models/meshes/d405/d405.obj
- link camera_support: geometry collision box size=0.01 0.05 0.03; collision box size=0.01 0.05 0.06
- link link1: geometry collision mesh filename=package://arx5_description/meshes/r5/link1.glb; visual mesh filename=package://arx5_description/meshes/r5/link1.glb
- link link2: geometry collision box size=0.264 0.051 0.05; collision cylinder length=0.0665 radius=0.03
- link link3: geometry collision box size=0.25 0.048 0.05; collision cylinder length=0.054 radius=0.032
- link link4: geometry collision cylinder length=0.04 radius=0.0315; visual mesh filename=package://arx5_description/meshes/r5/link4.glb
- link link5: geometry collision cylinder length=0.013 radius=0.03145; collision cylinder length=0.045 radius=0.03145
- link link6: geometry collision cylinder length=0.064 radius=0.03015; visual mesh filename=package://arx5_description/meshes/r5/link6.glb
- link link7: geometry collision box size=0.08 0.04 0.0640; visual mesh filename=package://arx5_description/meshes/r5/link7.glb
- link link8: geometry collision box size=0.08 0.04 0.0640; visual mesh filename=package://arx5_description/meshes/r5/link8.glb

File: arx5_description/xacro/R5.xacro (robot description, xacro)
@@ -439,5 +439,5 @@
 				<visual>
 					<geometry>
-						<mesh filename="file://$(find sensor_models)/meshes/d405.glb"/>
+						<mesh filename="file://$(find sensor_models)/meshes/d405/d405.obj"/>
 					</geometry>
 				</visual>
@@ -445,5 +445,5 @@
 					<collision>
 						<geometry>
-							<mesh filename="file://$(find sensor_models)/meshes/d405.glb"/>
+							<mesh filename="file://$(find sensor_models)/meshes/d405/d405.obj"/>
 						</geometry>
 					</collision>
@@ -495,5 +495,5 @@
 				<visual>
 					<geometry>
-						<mesh filename="file://$(find sensor_models)/meshes/d435.glb"/>
+						<mesh filename="file://$(find sensor_models)/meshes/d435/d435.obj"/>
 					</geometry>
 				</visual>
@@ -501,5 +501,5 @@
 					<collision>
 						<geometry>
-							<mesh filename="file://$(find sensor_models)/meshes/d435.glb"/>
+							<mesh filename="file://$(find sensor_models)/meshes/d435/d435.obj"/>
 						</geometry>
 					</collision>

File: arx5_description/xacro/X5.xacro (robot description, xacro)
@@ -430,5 +430,5 @@
                 <visual>
                     <geometry>
-                        <mesh filename="file://$(find sensor_models)/meshes/d405.glb"/>
+                        <mesh filename="file://$(find sensor_models)/meshes/d405/d405.obj"/>
                     </geometry>
                 </visual>
@@ -436,5 +436,5 @@
                     <collision>
                         <geometry>
-                            <mesh filename="file://$(find sensor_models)/meshes/d405.glb"/>
+                            <mesh filename="file://$(find sensor_models)/meshes/d405/d405.obj"/>
                         </geometry>
                     </collision>
@@ -486,10 +486,10 @@
                 <visual>
                     <geometry>
-                        <mesh filename="file://$(find sensor_models)/meshes/d435.glb"/>
+                        <mesh filename="file://$(find sensor_models)/meshes/d435/d435.obj"/>
                     </geometry>
                 </visual>
                 <xacro:if value="${collider == 'convex'}">
                     <geometry>
-                        <mesh filename="file://$(find sensor_models)/meshes/d435.glb"/>
+                        <mesh filename="file://$(find sensor_models)/meshes/d435/d435.obj"/>
                     </geometry>
                 </xacro:if>

File: arx5_description/xacro/X5_ac1.xacro (robot description, xacro)
@@ -433,5 +433,5 @@
 				<visual>
 					<geometry>
-						<mesh filename="file://$(find sensor_models)/meshes/d405.glb"/>
+						<mesh filename="file://$(find sensor_models)/meshes/d405/d405.obj"/>
 					</geometry>
 				</visual>
@@ -439,5 +439,5 @@
 					<collision>
 						<geometry>
-							<mesh filename="file://$(find sensor_models)/meshes/d405.glb"/>
+							<mesh filename="file://$(find sensor_models)/meshes/d405/d405.obj"/>
 						</geometry>
 					</collision>
@@ -489,10 +489,10 @@
 				<visual>
 					<geometry>
-						<mesh filename="file://$(find sensor_models)/meshes/d435.glb"/>
+						<mesh filename="file://$(find sensor_models)/meshes/d435/d435.obj"/>
 					</geometry>
 				</visual>
 				<xacro:if value="${collider == 'convex'}">
 					<geometry>
-						<mesh filename="file://$(find sensor_models)/meshes/d435.glb"/>
+						<mesh filename="file://$(find sensor_models)/meshes/d435/d435.obj"/>
 					</geometry>
 				</xacro:if>

File: arx_lift2s_description/urdf/arx_lift2s.urdf (robot description, URDF)
Before this commit: robot arx_lift2s, 35 links, 34 joints
Links:
- link base_link: geometry collision mesh filename=package://arx_lift2s_description/meshes/chassis/base_link.g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; visual mesh filename=package://arx_lift2s_description/meshes/chassis/base_link.g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
- link body_link: geometry collision box size=0.04 0.06 0.1; collision box size=0.04 0.06 0.3
- link head_camera: geometry visual mesh filename=package://sensor_models/meshes/d405/d405.obj
- link left_base_link: geometry collision cylinder length=0.03125 radius=0.031; visual mesh filename=package://arx5_description/meshes/x5/base_link.glb
- link left_camera: geometry collision box size=0.0231 0.0421 0.042; visual mesh filename=package://sensor_models/meshes/d405/d405.obj
- link left_camera_support: geometry collision box size=0.01 0.05 0.03; collision box size=0.01 0.05 0.06
- link left_link1: geometry collision mesh filename=package://arx5_description/meshes/x5/link1.glb; visual mesh filename=package://arx5_description/meshes/x5/link1.glb
- link left_link2: geometry collision box size=0.264 0.05 0.05; collision cylinder length=0.0665 radius=0.028
- link left_link3: geometry collision box size=0.2 0.04 0.045; collision cylinder length=0.049 radius=0.03
- link left_link4: geometry collision cylinder length=0.04 radius=0.0315; visual mesh filename=package://arx5_description/meshes/x5/link4.glb
- link left_link5: geometry collision cylinder length=0.013 radius=0.03145; collision cylinder length=0.045 radius=0.03145
- link left_link6: geometry collision cylinder length=0.064 radius=0.03015; visual mesh filename=package://arx5_description/meshes/r5/link6.glb
- link left_link7: geometry collision box size=0.08 0.04 0.0640; visual mesh filename=package://arx5_description/meshes/r5/link7.glb
- link left_link8: geometry collision box size=0.08 0.04 0.0640; visual mesh filename=package://arx5_description/meshes/r5/link8.glb
- link lift_link: geometry collision mesh filename=package://arx_lift2s_description/meshes/chassis/lift.glb; visual mesh filename=package://arx_lift2s_description/meshes/chassis/lift.glb
- link right_base_link: geometry collision cylinder length=0.03125 radius=0.031; visual mesh filename=package://arx5_description/meshes/x5/base_link.glb
- link right_camera: geometry collision box size=0.0231 0.0421 0.042; visual mesh filename=package://sensor_models/meshes/d405/d405.obj
- link right_camera_support: geometry collision box size=0.01 0.05 0.03; collision box size=0.01 0.05 0.06
- link right_link1: geometry collision mesh filename=package://arx5_description/meshes/x5/link1.glb; visual mesh filename=package://arx5_description/meshes/x5/link1.glb
- link right_link2: geometry collision box size=0.264 0.05 0.05; collision cylinder length=0.0665 radius=0.028
- link right_link3: geometry collision box size=0.2 0.04 0.045; collision cylinder length=0.049 radius=0.03
- link right_link4: geometry collision cylinder length=0.04 radius=0.0315; visual mesh filename=package://arx5_description/meshes/x5/link4.glb
- link right_link5: geometry collision cylinder length=0.013 radius=0.03145; collision cylinder length=0.045 radius=0.03145
- link right_link6: geometry collision cylinder length=0.064 radius=0.03015; visual mesh filename=package://arx5_description/meshes/r5/link6.glb
- link right_link7: geometry collision box size=0.08 0.04 0.0640; visual mesh filename=package://arx5_description/meshes/r5/link7.glb
- link right_link8: geometry collision box size=0.08 0.04 0.0640; visual mesh filename=package://arx5_description/meshes/r5/link8.glb
- link wheel_1: geometry visual mesh filename=package://arx_lift2s_description/meshes/chassis/wheel.glb
- link wheel_2: geometry visual mesh filename=package://arx_lift2s_description/meshes/chassis/wheel.glb
- link wheel_3: geometry visual mesh filename=package://arx_lift2s_description/meshes/chassis/wheel.glb

File: arx_lift2s_description/urdf/arx_lift2s_acone_x5.urdf (robot description, URDF)
Before this commit: robot arx_lift2s, 31 links, 30 joints
Links:
- link body_link: geometry collision box size=0.04 0.06 0.1; collision box size=0.04 0.06 0.3
- link head_camera: geometry visual mesh filename=package://sensor_models/meshes/d405/d405.obj
- link left_base_link: geometry collision cylinder length=0.03125 radius=0.031; visual mesh filename=package://arx5_description/meshes/x5/base_link.glb
- link left_camera: geometry collision box size=0.0231 0.0421 0.042; visual mesh filename=package://sensor_models/meshes/d405/d405.obj
- link left_camera_support: geometry collision box size=0.01 0.05 0.03; collision box size=0.01 0.05 0.06
- link left_link1: geometry collision mesh filename=package://arx5_description/meshes/x5/link1.glb; visual mesh filename=package://arx5_description/meshes/x5/link1.glb
- link left_link2: geometry collision box size=0.264 0.05 0.05; collision cylinder length=0.0665 radius=0.028
- link left_link3: geometry collision box size=0.2 0.04 0.045; collision cylinder length=0.049 radius=0.03
- link left_link4: geometry collision cylinder length=0.04 radius=0.0315; visual mesh filename=package://arx5_description/meshes/x5/link4.glb
- link left_link5: geometry collision cylinder length=0.013 radius=0.03145; collision cylinder length=0.045 radius=0.03145
- link left_link6: geometry collision cylinder length=0.064 radius=0.03015; visual mesh filename=package://arx5_description/meshes/r5/link6.glb
- link left_link7: geometry collision box size=0.08 0.04 0.0640; visual mesh filename=package://arx5_description/meshes/r5/link7.glb
- link left_link8: geometry collision box size=0.08 0.04 0.0640; visual mesh filename=package://arx5_description/meshes/r5/link8.glb
- link right_base_link: geometry collision cylinder length=0.03125 radius=0.031; visual mesh filename=package://arx5_description/meshes/x5/base_link.glb
- link right_camera: geometry collision box size=0.0231 0.0421 0.042; visual mesh filename=package://sensor_models/meshes/d405/d405.obj
- link right_camera_support: geometry collision box size=0.01 0.05 0.03; collision box size=0.01 0.05 0.06
- link right_link1: geometry collision mesh filename=package://arx5_description/meshes/x5/link1.glb; visual mesh filename=package://arx5_description/meshes/x5/link1.glb
- link right_link2: geometry collision box size=0.264 0.05 0.05; collision cylinder length=0.0665 radius=0.028
- link right_link3: geometry collision box size=0.2 0.04 0.045; collision cylinder length=0.049 radius=0.03
- link right_link4: geometry collision cylinder length=0.04 radius=0.0315; visual mesh filename=package://arx5_description/meshes/x5/link4.glb
- link right_link5: geometry collision cylinder length=0.013 radius=0.03145; collision cylinder length=0.045 radius=0.03145
- link right_link6: geometry collision cylinder length=0.064 radius=0.03015; visual mesh filename=package://arx5_description/meshes/r5/link6.glb
- link right_link7: geometry collision box size=0.08 0.04 0.0640; visual mesh filename=package://arx5_description/meshes/r5/link7.glb
- link right_link8: geometry collision box size=0.08 0.04 0.0640; visual mesh filename=package://arx5_description/meshes/r5/link8.glb

Commit message: move to realsense glb

File: arx5_description/urdf/arx5.urdf (robot description, URDF)
Before this commit: robot ARX 5, 14 links, 13 joints
Links:
- link camera: geometry collision box size=0.0231 0.0421 0.042; visual mesh filename=package://sensor_models/meshes/realsense/d405.glb

File: arx5_description/urdf/arx5_ac1.urdf (robot description, URDF)
Before this commit: robot ARX 5, 14 links, 13 joints
Links:
- link camera: geometry collision box size=0.0231 0.0421 0.042; visual mesh filename=package://sensor_models/meshes/realsense/d405.glb

File: arx5_description/urdf/arx5_agilex.urdf (robot description, URDF)
Before this commit: robot ARX 5, 14 links, 13 joints
Links:
- link camera: geometry collision box size=0.0231 0.0421 0.042; visual mesh filename=package://sensor_models/meshes/realsense/d405.glb

File: arx5_description/urdf/arx5_r5.urdf (robot description, URDF)
Before this commit: robot ARX 5, 14 links, 13 joints
Links:
- link camera: geometry collision box size=0.0231 0.0421 0.042; visual mesh filename=package://sensor_models/meshes/realsense/d405.glb

File: arx_lift2s_description/urdf/arx_lift2s.urdf (robot description, URDF)
Before this commit: robot arx_lift2s, 35 links, 34 joints
Links:
- link head_camera: geometry visual mesh filename=package://sensor_models/meshes/realsense/d405.glb
- link left_camera: geometry collision box size=0.0231 0.0421 0.042; visual mesh filename=package://sensor_models/meshes/realsense/d405.glb
- link right_camera: geometry collision box size=0.0231 0.0421 0.042; visual mesh filename=package://sensor_models/meshes/realsense/d405.glb

File: arx_lift2s_description/urdf/arx_lift2s_acone_x5.urdf (robot description, URDF)
Before this commit: robot arx_lift2s, 31 links, 30 joints
Links:
- link head_camera: geometry visual mesh filename=package://sensor_models/meshes/realsense/d405.glb
- link left_camera: geometry collision box size=0.0231 0.0421 0.042; visual mesh filename=package://sensor_models/meshes/realsense/d405.glb
- link right_camera: geometry collision box size=0.0231 0.0421 0.042; visual mesh filename=package://sensor_models/meshes/realsense/d405.glb

File: arx_lift_description/urdf/arx_lift.urdf (robot description, URDF)
Before this commit: robot arx_lift, 37 links, 36 joints
Links:
- link head_camera: geometry visual mesh filename=package://sensor_models/meshes/realsense/d405.glb
- link left_camera: geometry visual mesh filename=package://sensor_models/meshes/realsense/d405.glb
- link right_camera: geometry visual mesh filename=package://sensor_models/meshes/realsense/d405.glb

File: arx_lift_description/urdf/arx_lift_r5.urdf (robot description, URDF)
Before this commit: robot arx_lift, 37 links, 36 joints
Links:
- link head_camera: geometry visual mesh filename=package://sensor_models/meshes/realsense/d405.glb
- link left_camera: geometry visual mesh filename=package://sensor_models/meshes/realsense/d405.glb
- link right_camera: geometry visual mesh filename=package://sensor_models/meshes/realsense/d405.glb

File: arx_x7s_description/urdf/arx_x7s.urdf (robot description, URDF)
Before this commit: robot ARX X7S, 30 links, 29 joints
Links:
- link head_camera: geometry visual mesh filename=package://sensor_models/meshes/realsense/d405.glb
