Commit message: add acone config

File: arx_lift2s_description/urdf/arx_lift2s.urdf (robot description, URDF)
Before this commit: robot arx_lift2s, 34 links, 33 joints
Links:
- link base_link: geometry collision mesh filename=file:///home/shimanliang/ros2_ws/install/arx_lift2s_descrip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; visual mesh filename=file:///home/shimanliang/ros2_ws/install/arx_lift2s_descrip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
- link body_link: geometry collision mesh filename=file:///home/shimanliang/ros2_ws/install/arx_lift2s_descrip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; visual mesh filename=file:///home/shimanliang/ros2_ws/install/arx_lift2s_descrip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
- link left_base_link: geometry collision mesh filename=file:///home/shimanliang/ros2_ws/install/arx5_description/s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; visual mesh filename=file:///home/shimanliang/ros2_ws/install/arx5_description/s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
- link left_camera: geometry visual mesh filename=file:///home/shimanliang/ros2_ws/install/sensor_models/shar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
- link left_camera_support: geometry visual mesh filename=file:///home/shimanliang/ros2_ws/install/arx5_description/s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
- link left_link1: geometry collision mesh filename=file:///home/shimanliang/ros2_ws/install/arx5_description/s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; visual mesh filename=file:///home/shimanliang/ros2_ws/install/arx5_description/s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
- link left_link2: geometry collision mesh filename=file:///home/shimanliang/ros2_ws/install/arx5_description/s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; visual mesh filename=file:///home/shimanliang/ros2_ws/install/arx5_description/s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
- link left_link3: geometry collision mesh filename=file:///home/shimanliang/ros2_ws/install/arx5_description/s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; visual mesh filename=file:///home/shimanliang/ros2_ws/install/arx5_description/s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
- link left_link4: geometry collision mesh filename=file:///home/shimanliang/ros2_ws/install/arx5_description/s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; visual mesh filename=file:///home/shimanliang/ros2_ws/install/arx5_description/s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
- link left_link5: geometry collision mesh filename=file:///home/shimanliang/ros2_ws/install/arx5_description/s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; visual mesh filename=file:///home/shimanliang/ros2_ws/install/arx5_description/s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
- link left_link6: geometry collision mesh filename=file:///home/shimanliang/ros2_ws/install/arx5_description/s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; visual mesh filename=file:///home/shimanliang/ros2_ws/install/arx5_description/s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
- link left_link7: geometry collision mesh filename=file:///home/shimanliang/ros2_ws/install/arx5_description/s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; visual mesh filename=file:///home/shimanliang/ros2_ws/install/arx5_description/s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
- link left_link8: geometry collision mesh filename=file:///home/shimanliang/ros2_ws/install/arx5_description/s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; visual mesh filename=file:///home/shimanliang/ros2_ws/install/arx5_description/s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
- link lift_link: geometry collision mesh filename=file:///home/shimanliang/ros2_ws/install/arx_lift2s_descrip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; visual mesh filename=file:///home/shimanliang/ros2_ws/install/arx_lift2s_descrip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
- link right_base_link: geometry collision mesh filename=file:///home/shimanliang/ros2_ws/install/arx5_description/s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; visual mesh filename=file:///home/shimanliang/ros2_ws/install/arx5_description/s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
- link right_camera: geometry visual mesh filename=file:///home/shimanliang/ros2_ws/install/sensor_models/shar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
- link right_camera_support: geometry visual mesh filename=file:///home/shimanliang/ros2_ws/install/arx5_description/s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
- link right_link1: geometry collision mesh filename=file:///home/shimanliang/ros2_ws/install/arx5_description/s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; visual mesh filename=file:///home/shimanliang/ros2_ws/install/arx5_description/s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
- link right_link2: geometry collision mesh filename=file:///home/shimanliang/ros2_ws/install/arx5_description/s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; visual mesh filename=file:///home/shimanliang/ros2_ws/install/arx5_description/s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
- link right_link3: geometry collision mesh filename=file:///home/shimanliang/ros2_ws/install/arx5_description/s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; visual mesh filename=file:///home/shimanliang/ros2_ws/install/arx5_description/s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
- link right_link4: geometry collision mesh filename=file:///home/shimanliang/ros2_ws/install/arx5_description/s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; visual mesh filename=file:///home/shimanliang/ros2_ws/install/arx5_description/s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
- link right_link5: geometry collision mesh filename=file:///home/shimanliang/ros2_ws/install/arx5_description/s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; visual mesh filename=file:///home/shimanliang/ros2_ws/install/arx5_description/s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
- link right_link6: geometry collision mesh filename=file:///home/shimanliang/ros2_ws/install/arx5_description/s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; visual mesh filename=file:///home/shimanliang/ros2_ws/install/arx5_description/s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
- link right_link7: geometry collision mesh filename=file:///home/shimanliang/ros2_ws/install/arx5_description/s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; visual mesh filename=file:///home/shimanliang/ros2_ws/install/arx5_description/s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
- link right_link8: geometry collision mesh filename=file:///home/shimanliang/ros2_ws/install/arx5_description/s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; visual mesh filename=file:///home/shimanliang/ros2_ws/install/arx5_description/s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
- link wheel_1: geometry collision mesh filename=file:///home/shimanliang/ros2_ws/install/arx_lift2s_descrip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; visual mesh filename=file:///home/shimanliang/ros2_ws/install/arx_lift2s_descrip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
- link wheel_2: geometry collision mesh filename=file:///home/shimanliang/ros2_ws/install/arx_lift2s_descrip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; visual mesh filename=file:///home/shimanliang/ros2_ws/install/arx_lift2s_descrip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
- link wheel_3: geometry collision mesh filename=file:///home/shimanliang/ros2_ws/install/arx_lift2s_descrip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; visual mesh filename=file:///home/shimanliang/ros2_ws/install/arx_lift2s_descrip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
Joints:
- joint wheel1_joint: type continuous -> fixed
- joint wheel2_joint: type continuous -> fixed
- joint wheel3_joint: type continuous -> fixed

File: arx_lift2s_description/xacro/component.xacro (robot description, xacro)
@@ -5,15 +5,28 @@
 <!-- =================================================================================== -->
 <robot name="ARX_Lift2S" xmlns:xacro="http://www.ros.org/wiki/xacro">
-    <xacro:property name="PI" value="3.1415926535897931"/>
-    <xacro:arg name="type" default="base"/>
-    <xacro:if value="${'$(arg type)' == 'base'}">
-        <!-- Include Chassis -->
-        <xacro:include filename="$(find arx_lift2s_description)/xacro/components/base.xacro"/>
-        <xacro:Base/>
-    </xacro:if>
-    <xacro:if value="${'$(arg type)' == 'wheel'}">
-        <!-- Include Wheel -->
-        <xacro:include filename="$(find arx_lift2s_description)/xacro/components/wheel.xacro"/>
-        <xacro:wheel wheel_name="wheel" enable_passive_wheels="true"/>
-    </xacro:if>
+	<xacro:property name="PI" value="3.1415926535897931"/>
+	<xacro:arg name="type" default="chassis"/>
+	<xacro:if value="${'$(arg type)' == 'chassis'}">
+		<!-- Include Chassis -->
+		<xacro:include filename="$(find arx_lift2s_description)/xacro/components/chassis.xacro"/>
+		<xacro:chassis/>
+	</xacro:if>
+	<xacro:if value="${'$(arg type)' == 'ac_one'}">
+		<link name="base_link"/>
+		<joint name="base_joint" type="fixed">
+			<parent link="base_link"/>
+			<child link="body_link"/>
+		</joint>
+		<xacro:include filename="$(find arx_lift2s_description)/xacro/components/ac_one.xacro"/>
+		<xacro:ac_one />
+	</xacro:if>
+	<xacro:if value="${'$(arg type)' == 'wheel'}">
+		<xacro:include filename="$(find arx_lift2s_description)/xacro/components/wheel.xacro"/>
+		<xacro:wheel wheel_name="wheel" enable_passive_wheels="true"/>
+		<link name="base_link"/>
+		<joint name="base_joint" type="fixed">
+			<parent link="base_link"/>
+			<child link="wheel"/>
+		</joint>
+	</xacro:if>
 </robot>

File: arx_lift2s_description/xacro/components/wheel.xacro (robot description, xacro)
@@ -1,81 +1,77 @@
 <?xml version="1.0"?>
 <robot xmlns:xacro="http://www.ros.org/wiki/xacro">
-    <xacro:property name="PI" value="3.1415926535897931"/>
-    <xacro:macro name="passive_wheel" params="parent_link passive_wheel_name radius angle sphere_radius:='0.06'">
-        <link name="${passive_wheel_name}">
-            <inertial>
-                <origin xyz="0 0 0"/>
-                <mass value="0.01"/> <inertia ixx="0.0001" ixy="0.0" ixz="0.0" iyy="0.0001" iyz="0.0" izz="0.0001"/>
-            </inertial>
-            <collision>
-                <geometry>
-                    <sphere radius="${float(sphere_radius)}"/>
-                </geometry>
-            </collision>
-        </link>
-        <joint name="${passive_wheel_name}_joint" type="continuous">
-            <origin xyz="0 ${float(radius) * cos(float(angle))} ${float(radius) * sin(float(angle))}" rpy="${float(angle)} 0 0"/>
-            <parent link="${parent_link}"/>
-            <child link="${passive_wheel_name}"/>
-            <axis xyz="0 0 1"/>
-        </joint>
-    </xacro:macro>
-    <xacro:macro name="create_passive_wheels" params="parent_link wheel_name indices:=^ angle_step passive_wheel_radius_actual">
-        <xacro:if value="${indices}">
-            <xacro:property name="index" value="${indices.pop(0)}"/>
-            <xacro:property name="angle" value="${float(index) * float(angle_step)}"/>
-            <xacro:passive_wheel
-                    parent_link="${parent_link}"
-                    passive_wheel_name="${wheel_name}_passive_${index}"
-                    radius="${passive_wheel_radius_actual}"
-                    angle="${angle}"/>
-            <xacro:create_passive_wheels
-                    parent_link="${parent_link}"
-                    wheel_name="${wheel_name}"
-                    indices="${indices}"
-                    angle_step="${angle_step}"
-                    passive_wheel_radius_actual="${passive_wheel_radius_actual}"/>
-        </xacro:if>
-    </xacro:macro>
-    <xacro:macro name="wheel" params="wheel_name
+	<xacro:property name="PI" value="3.1415926535897931"/>
+	<xacro:macro name="passive_wheel" params="parent_link passive_wheel_name radius angle sphere_radius:='0.06'">
+		<link name="${passive_wheel_name}">
+			<inertial>
+				<origin xyz="0 0 0"/>
+				<mass value="0.01"/>
+				<inertia ixx="0.0001" ixy="0.0" ixz="0.0" iyy="0.0001" iyz="0.0" izz="0.0001"/>
+			</inertial>
+			<collision>
+				<geometry>
+					<sphere radius="${float(sphere_radius)}"/>
+				</geometry>
+			</collision>
+		</link>
+		<joint name="${passive_wheel_name}_joint" type="continuous">
+			<origin xyz="0.0385 ${float(radius) * cos(float(angle))} ${float(radius) * sin(float(angle))}"
+							rpy="${float(angle)} 0 0"/>
+			<parent link="${parent_link}"/>
+			<child link="${passive_wheel_name}"/>
+			<axis xyz="0 0 1"/>
+		</joint>
+	</xacro:macro>
+	<xacro:macro name="create_passive_wheels"
+							 params="parent_link wheel_name indices:=^ angle_step passive_wheel_radius_actual">
+		<xacro:if value="${indices}">
+			<xacro:property name="index" value="${indices.pop(0)}"/>
+			<xacro:property name="angle" value="${float(index) * float(angle_step)}"/>
+			<xacro:passive_wheel
+					parent_link="${parent_link}"
+					passive_wheel_name="${wheel_name}_passive_${index}"
+					radius="${passive_wheel_radius_actual}"
+					angle="${angle}"/>
+			<xacro:create_passive_wheels
+					parent_link="${parent_link}"
+					wheel_name="${wheel_name}"
+					indices="${indices}"
+					angle_step="${angle_step}"
+					passive_wheel_radius_actual="${passive_wheel_radius_actual}"/>
+		</xacro:if>
+	</xacro:macro>
+	<xacro:macro name="wheel" params="wheel_name
                                     enable_passive_wheels:='false'
-                                    mesh_rpy:='0 0 0'
                                     passive_wheel_radius:='0.02'
-                                    num_passive_wheels:='10'">
-        <link name="${wheel_name}">
-            <inertial>
-                <origin xyz="0.035966 2.6831E-06 8.693E-07" rpy="${mesh_rpy}" />
-                <mass value="0.5746" />
-                <inertia
-                        ixx="0.00142306"
-                        ixy="0.00000000"
-                        ixz="0.00000000"
-                        iyy="0.00084449"
-                        iyz="0.00000002"
-                        izz="0.00084474" />
-            </inertial>
-            <visual>
-                <origin xyz="0 0 0" rpy="${mesh_rpy}" />
-                <geometry>
-                    <mesh filename="file://$(find arx_lift2s_description)/meshes/wheel.glb" />
-                </geometry>
-            </visual>
-            <collision>
-                <origin xyz="0 0 0" rpy="${mesh_rpy}" />
-                <geometry>
-                    <mesh filename="file://$(find arx_lift2s_description)/meshes/wheel.glb" />
-                </geometry>
-            </collision>
-        </link>
-        <xacro:if value="${enable_passive_wheels}">
-            <xacro:property name="num_passive_wheels_float" value="${float(num_passive_wheels)}"/>
-            <xacro:property name="angle_step" value="${2*PI / num_passive_wheels_float}"/>
-            <xacro:property name="indices" value="${[0,1,2,3,4,5,6,7,8,9]}"/> <xacro:create_passive_wheels
-                parent_link="${wheel_name}"
-                wheel_name="${wheel_name}"
-                indices="${list(indices)}"
-                angle_step="${angle_step}"
-                passive_wheel_radius_actual="${passive_wheel_radius}"/>
-        </xacro:if>
-    </xacro:macro>
+                                    num_passive_wheels:='9'">
+		<link name="${wheel_name}">
+			<inertial>
+				<origin xyz="0.035966 2.6831E-06 8.693E-07"/>
+				<mass value="0.5746"/>
+				<inertia
+						ixx="0.00142306"
+						ixy="0.00000000"
+						ixz="0.00000000"
+						iyy="0.00084449"
+						iyz="0.00000002"
+						izz="0.00084474"/>
+			</inertial>
+			<visual>
+				<geometry>
+					<mesh filename="file://$(find arx_lift2s_description)/meshes/chassis/wheel.glb"/>
+				</geometry>
+			</visual>
+		</link>
+		<xacro:if value="${enable_passive_wheels}">
+			<xacro:property name="num_passive_wheels_float" value="${float(num_passive_wheels)}"/>
+			<xacro:property name="angle_step" value="${2*PI / num_passive_wheels_float}"/>
+			<xacro:property name="indices" value="${[0,1,2,3,4,5,6,7,8]}"/>
+			<xacro:create_passive_wheels
+					parent_link="${wheel_name}"
+					wheel_name="${wheel_name}"
+					indices="${list(indices)}"
+					angle_step="${angle_step}"
+					passive_wheel_radius_actual="${passive_wheel_radius}"/>
+		</xacro:if>
+	</xacro:macro>
 </robot>

File: arx_lift2s_description/xacro/robot.xacro (robot description, xacro)
@@ -1,39 +1,57 @@
 <robot name="arx_lift2s" xmlns:xacro="http://www.ros.org/wiki/xacro">
-    <xacro:arg name="type" default="x5"/>
-    <xacro:arg name="enable_wheel_joints" default="true"/>
-    <xacro:arg name="ros2_control_hardware_type" default="mock_components"/>
-    <xacro:unless value="${'$(arg type)' == 'wheel'}">
-        <xacro:include filename="$(find arx_lift2s_description)/xacro/components/base.xacro"/>
-        <xacro:Base enable_wheel_joints="$(arg enable_wheel_joints)"/>
-        <xacro:if value="${'$(arg type)' == 'x5'}">
-            <xacro:include filename="$(find arx5_description)/xacro/X5.xacro"/>
-            <xacro:X5 name="left"/>
-            <xacro:X5 name="right"/>
-        </xacro:if>
-        <xacro:if value="${'$(arg type)' == 'r5'}">
-            <xacro:include filename="$(find arx5_description)/xacro/R5.xacro"/>
-            <xacro:R5 name="left"/>
-            <xacro:R5 name="right"/>
-        </xacro:if>
-        <joint name="arm_left_fixed" type="fixed">
-            <parent link="lift_link"/>
-            <child link="left_base_link"/>
-            <origin xyz="0.113964 0.253848 0.012392" rpy="0 0 0"/>
-        </joint>
-        <joint name="arm_right_fixed" type="fixed">
-            <parent link="lift_link"/>
-            <child link="right_base_link"/>
-            <origin xyz="0.113964 -0.246152 0.012392" rpy="0 0 0"/>
-        </joint>
-    </xacro:unless>
-    <xacro:if value="${'$(arg type)' == 'wheel'}">
-        <xacro:include filename="$(find arx_lift2s_description)/xacro/components/wheel.xacro"/>
-        <link name="world"/>
-        <xacro:wheel wheel_name="wheel_test" enable_passive_wheels="false"/>
-        <joint name="world_to_wheel" type="fixed">
-            <parent link="world"/>
-            <child link="wheel_test"/>
-            <origin xyz="0 0 0" rpy="0 0 0"/>
-        </joint>
-    </xacro:if>
+	<xacro:arg name="type" default="x5"/>
+	<xacro:arg name="enable_wheel_joints" default="true"/>
+	<xacro:arg name="ros2_control_hardware_type" default="mock_components"/>
+	<xacro:property name="type_arg" value="$(arg type)"/>
+	<xacro:property name="selected_arm_type" value="x5"/>
+	<xacro:property name="selected_base_type" value="lift2s"/>
+	<xacro:if value="${type_arg == 'r5'}">
+		<xacro:property name="selected_arm_type" value="r5"/>
+	</xacro:if>
+	<xacro:if value="${type_arg == 'acone_x5'}">
+		<xacro:property name="selected_base_type" value="acone"/>
+	</xacro:if>
+	<xacro:if value="${type_arg == 'acone_r5'}">
+		<xacro:property name="selected_arm_type" value="r5"/>
+		<xacro:property name="selected_base_type" value="acone"/>
+	</xacro:if>
+	<xacro:if value="${selected_base_type == 'lift2s'}">
+		<xacro:include filename="$(find arx_lift2s_description)/xacro/components/chassis.xacro"/>
+		<xacro:chassis enable_wheel_joints="$(arg enable_wheel_joints)"/>
+		<joint name="body_joint" type="fixed">
+			<origin xyz="0.13 0.001801 0.0529" rpy="0 0 0"/>
+			<parent link="lift_link"/>
+			<child link="body_link"/>
+			<axis xyz="0 0 1"/>
+		</joint>
+	</xacro:if>
+	<xacro:unless value="${selected_base_type == 'lift2s'}">
+		<link name="base_link"/>
+		<joint name="base_joint" type="fixed">
+			<parent link="base_link"/>
+			<child link="body_link"/>
+		</joint>
+	</xacro:unless>
+	<xacro:include filename="$(find arx_lift2s_description)/xacro/components/ac_one.xacro"/>
+	<xacro:ac_one/>
+	<xacro:if value="${selected_arm_type == 'x5'}">
+		<xacro:include filename="$(find arx5_description)/xacro/X5.xacro"/>
+		<xacro:X5 name="left"/>
+		<xacro:X5 name="right"/>
+	</xacro:if>
+	<xacro:if value="${selected_arm_type == 'r5'}">
+		<xacro:include filename="$(find arx5_description)/xacro/R5.xacro"/>
+		<xacro:R5 name="left"/>
+		<xacro:R5 name="right"/>
+	</xacro:if>
+	<joint name="arm_left_fixed" type="fixed">
+		<parent link="body_link"/>
+		<child link="left_base_link"/>
+		<origin xyz="-0.01602 0.25 -0.035"/>
+	</joint>
+	<joint name="arm_right_fixed" type="fixed">
+		<parent link="body_link"/>
+		<child link="right_base_link"/>
+		<origin xyz="-0.01602 -0.25 -0.035"/>
+	</joint>
 </robot>

File: arx_lift2s_description/xacro/ros2_control/robot.xacro (robot description, xacro)
@@ -2,5 +2,5 @@
 <robot xmlns:xacro="http://www.ros.org/wiki/xacro" name="arx_lift2s">
     <xacro:arg name="type" default="x5"/>
-    <xacro:arg name="enable_wheel_joints" default="false"/>
+    <xacro:arg name="enable_wheel_joints" default="true"/>
     <xacro:arg name="ros2_control_hardware_type" default="mock_components"/>
     <xacro:include filename="$(find arx_lift2s_description)/xacro/robot.xacro"/>

File: arx_lift_description/xacro/component.xacro (robot description, xacro)
@@ -16,5 +16,5 @@
 	<xacro:if value="${'$(arg type)' == 'wheel'}">
 		<!-- Include Wheel -->
-		<xacro:include filename="$(find arx_lift_description)/xacro/components/wheel.xacro"/>
+		<xacro:include filename="$(find component_models)/xacro/angellun_omniwheel.xacro"/>
 		<xacro:wheel wheel_name="wheel" enable_passive_wheels="true"/>
 	</xacro:if>

File: arx_lift_description/xacro/components/mobile_base.xacro (robot description, xacro)
@@ -2,5 +2,5 @@
 <robot xmlns:xacro="http://www.ros.org/wiki/xacro">
   <!-- 包含轮子模块 -->
-  <xacro:include filename="$(find arx_lift_description)/xacro/components/wheel.xacro"/>
+  <xacro:include filename="$(find component_models)/xacro/angellun_omniwheel.xacro"/>
   <xacro:property name="PI" value="3.1415926535897931"/>
   <xacro:macro name="MobileBase" params="enable_wheel_joints:='true'">
