Commit message: update acone config

File: arx_lift2s_description/urdf/arx_lift2s.urdf (robot description, URDF)
Before this commit: robot arx_lift2s, 34 links, 33 joints
Links:
- link base_link: geometry collision mesh filename=package://arx_lift2s_description/meshes/base_link.glb; visual mesh filename=package://arx_lift2s_description/meshes/base_link.glb
- link body_link: geometry collision mesh filename=package://arx_lift2s_description/meshes/body4_2.glb; visual mesh filename=package://arx_lift2s_description/meshes/body4_2.glb
- link left_base_link: geometry collision mesh filename=package://arx5_description/meshes/x5/base_link.obj; visual mesh filename=package://arx5_description/meshes/x5/base_link.obj
- link left_camera: geometry visual mesh filename=package://sensor_models/meshes/d405/d405.obj
- link left_camera_support: geometry visual mesh filename=package://arx5_description/meshes/camera_stand/stand_d405.o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
- link left_link1: geometry collision mesh filename=package://arx5_description/meshes/x5/link1.obj; visual mesh filename=package://arx5_description/meshes/x5/link1.obj
- link left_link2: geometry collision mesh filename=package://arx5_description/meshes/x5/link2.obj; visual mesh filename=package://arx5_description/meshes/x5/link2.obj
- link left_link3: geometry collision mesh filename=package://arx5_description/meshes/x5/link3.obj; visual mesh filename=package://arx5_description/meshes/x5/link3.obj
- link left_link4: geometry collision mesh filename=package://arx5_description/meshes/x5/link4.obj; visual mesh filename=package://arx5_description/meshes/x5/link4.obj
- link left_link5: geometry collision mesh filename=package://arx5_description/meshes/x5/link5.obj; visual mesh filename=package://arx5_description/meshes/x5/link5.obj
- link left_link6: geometry collision mesh filename=package://arx5_description/meshes/x5/link6.obj; visual mesh filename=package://arx5_description/meshes/x5/link6.obj
- link left_link7: geometry collision mesh filename=package://arx5_description/meshes/x5/link7.obj; visual mesh filename=package://arx5_description/meshes/x5/link7.obj
- link left_link8: geometry collision mesh filename=package://arx5_description/meshes/x5/link8.obj; visual mesh filename=package://arx5_description/meshes/x5/link8.obj
- link lift_link: geometry collision mesh filename=package://arx_lift2s_description/meshes/body4_1.glb; visual mesh filename=package://arx_lift2s_description/meshes/body4_1.glb
- link right_base_link: geometry collision mesh filename=package://arx5_description/meshes/x5/base_link.obj; visual mesh filename=package://arx5_description/meshes/x5/base_link.obj
- link right_camera: geometry visual mesh filename=package://sensor_models/meshes/d405/d405.obj
- link right_camera_support: geometry visual mesh filename=package://arx5_description/meshes/camera_stand/stand_d405.o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
- link right_link1: geometry collision mesh filename=package://arx5_description/meshes/x5/link1.obj; visual mesh filename=package://arx5_description/meshes/x5/link1.obj
- link right_link2: geometry collision mesh filename=package://arx5_description/meshes/x5/link2.obj; visual mesh filename=package://arx5_description/meshes/x5/link2.obj
- link right_link3: geometry collision mesh filename=package://arx5_description/meshes/x5/link3.obj; visual mesh filename=package://arx5_description/meshes/x5/link3.obj
- link right_link4: geometry collision mesh filename=package://arx5_description/meshes/x5/link4.obj; visual mesh filename=package://arx5_description/meshes/x5/link4.obj
- link right_link5: geometry collision mesh filename=package://arx5_description/meshes/x5/link5.obj; visual mesh filename=package://arx5_description/meshes/x5/link5.obj
- link right_link6: geometry collision mesh filename=package://arx5_description/meshes/x5/link6.obj; visual mesh filename=package://arx5_description/meshes/x5/link6.obj
- link right_link7: geometry collision mesh filename=package://arx5_description/meshes/x5/link7.obj; visual mesh filename=package://arx5_description/meshes/x5/link7.obj
- link right_link8: geometry collision mesh filename=package://arx5_description/meshes/x5/link8.obj; visual mesh filename=package://arx5_description/meshes/x5/link8.obj
- link wheel_1: geometry collision mesh filename=package://arx_lift2s_description/meshes/wheel.glb; visual mesh filename=package://arx_lift2s_description/meshes/wheel.glb
- link wheel_2: geometry collision mesh filename=package://arx_lift2s_description/meshes/wheel.glb; visual mesh filename=package://arx_lift2s_description/meshes/wheel.glb
- link wheel_3: geometry collision mesh filename=package://arx_lift2s_description/meshes/wheel.glb; visual mesh filename=package://arx_lift2s_description/meshes/wheel.glb

File: arx_lift2s_description/xacro/ros2_control/interfaces.xacro (robot description, xacro)
@@ -3,11 +3,13 @@
     <!-- ARX LIFT 2S 基座关节接口宏定义 -->
     <xacro:macro name="arx_lift2s_base_interfaces">
-        <!-- 升降关节接口定义 -->
-        <joint name="lift_joint">
-            <command_interface name="position"/>
-            <state_interface name="position"/>
-            <state_interface name="velocity"/>
-            <state_interface name="effort"/>
-        </joint>
+        <!-- 升降关节接口定义 (仅 lift2s 底盘需要) -->
+        <xacro:if value="${selected_base_type == 'lift2s'}">
+            <joint name="lift_joint">
+                <command_interface name="position"/>
+                <state_interface name="position"/>
+                <state_interface name="velocity"/>
+                <state_interface name="effort"/>
+            </joint>
+        </xacro:if>
     </xacro:macro>
 </robot>

Commit message: update

File: arx_lift2s_description/urdf/arx_lift2s.urdf (robot description, URDF)
Before this commit: robot arx_lift2s, 34 links, 33 joints
Links:
- added link head_camera; visual mesh filename=package://sensor_models/meshes/d405/d405.obj
- link base_link: geometry collision mesh filename=package://arx_lift2s_description/meshes/chassis/base_link.g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; visual mesh filename=package://arx_lift2s_description/meshes/chassis/base_link.g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
- link body_link: mass 1.0 -> 5.6137; geometry collision mesh filename=package://arx_lift2s_description/meshes/ac_one/base.glb; visual mesh filename=package://arx_lift2s_description/meshes/ac_one/base.glb
- link left_base_link: geometry collision mesh filename=package://arx5_description/meshes/x5/base_link.glb; visual mesh filename=package://arx5_description/meshes/x5/base_link.glb
- link left_camera: geometry visual mesh filename=package://sensor_models/meshes/d405.glb
- link left_camera_support: geometry visual mesh filename=package://arx5_description/meshes/camera_stand/stand_d405.g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
- link left_link1: geometry collision mesh filename=package://arx5_description/meshes/x5/link1.glb; visual mesh filename=package://arx5_description/meshes/x5/link1.glb
- link left_link2: mass 1.0795 -> 1.1068; geometry collision mesh filename=package://arx5_description/meshes/x5/link2.glb; visual mesh filename=package://arx5_description/meshes/x5/link2.glb
- link left_link3: mass 0.54534 -> 0.54316; geometry collision mesh filename=package://arx5_description/meshes/x5/link3.glb; visual mesh filename=package://arx5_description/meshes/x5/link3.glb
- link left_link4: mass 0.11714 -> 0.11827; geometry collision mesh filename=package://arx5_description/meshes/x5/link4.glb; visual mesh filename=package://arx5_description/meshes/x5/link4.glb
- link left_link5: mass 0.63488 -> 0.67398; geometry collision mesh filename=package://arx5_description/meshes/ac1/link5.glb; visual mesh filename=package://arx5_description/meshes/ac1/link5.glb
- link left_link6: mass 0.44089 -> 0.34667; geometry collision mesh filename=package://arx5_description/meshes/ac1/link6.glb; visual mesh filename=package://arx5_description/meshes/ac1/link6.glb
- link left_link7: mass 0.064798 -> 0.08924; geometry collision mesh filename=package://arx5_description/meshes/ac1/link7.glb; visual mesh filename=package://arx5_description/meshes/ac1/link7.glb
- link left_link8: mass 0.064798 -> 0.089402; geometry collision mesh filename=package://arx5_description/meshes/ac1/link8.glb; visual mesh filename=package://arx5_description/meshes/ac1/link8.glb
- link lift_link: geometry collision mesh filename=package://arx_lift2s_description/meshes/chassis/lift.glb; visual mesh filename=package://arx_lift2s_description/meshes/chassis/lift.glb
- link right_base_link: geometry collision mesh filename=package://arx5_description/meshes/x5/base_link.glb; visual mesh filename=package://arx5_description/meshes/x5/base_link.glb
- link right_camera: geometry visual mesh filename=package://sensor_models/meshes/d405.glb
- link right_camera_support: geometry visual mesh filename=package://arx5_description/meshes/camera_stand/stand_d405.g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
- link right_link1: geometry collision mesh filename=package://arx5_description/meshes/x5/link1.glb; visual mesh filename=package://arx5_description/meshes/x5/link1.glb
- link right_link2: mass 1.0795 -> 1.1068; geometry collision mesh filename=package://arx5_description/meshes/x5/link2.glb; visual mesh filename=package://arx5_description/meshes/x5/link2.glb
- link right_link3: mass 0.54534 -> 0.54316; geometry collision mesh filename=package://arx5_description/meshes/x5/link3.glb; visual mesh filename=package://arx5_description/meshes/x5/link3.glb
- link right_link4: mass 0.11714 -> 0.11827; geometry collision mesh filename=package://arx5_description/meshes/x5/link4.glb; visual mesh filename=package://arx5_description/meshes/x5/link4.glb
- link right_link5: mass 0.63488 -> 0.67398; geometry collision mesh filename=package://arx5_description/meshes/ac1/link5.glb; visual mesh filename=package://arx5_description/meshes/ac1/link5.glb
- link right_link6: mass 0.44089 -> 0.34667; geometry collision mesh filename=package://arx5_description/meshes/ac1/link6.glb; visual mesh filename=package://arx5_description/meshes/ac1/link6.glb
- link right_link7: mass 0.064798 -> 0.08924; geometry collision mesh filename=package://arx5_description/meshes/ac1/link7.glb; visual mesh filename=package://arx5_description/meshes/ac1/link7.glb
- link right_link8: mass 0.064798 -> 0.089402; geometry collision mesh filename=package://arx5_description/meshes/ac1/link8.glb; visual mesh filename=package://arx5_description/meshes/ac1/link8.glb
- link wheel_1: geometry visual mesh filename=package://arx_lift2s_description/meshes/chassis/wheel.glb
- link wheel_2: geometry visual mesh filename=package://arx_lift2s_description/meshes/chassis/wheel.glb
- link wheel_3: geometry visual mesh filename=package://arx_lift2s_description/meshes/chassis/wheel.glb
Joints:
- added joint head_camera_joint: type fixed, parent body_link, child head_camera, origin xyz=0.090415 0.002 0.2285 rpy=0 1.0472 0
- joint arm_left_fixed: origin xyz=0.113964 0.253848 0.012392 rpy=0 0 0 -> xyz=-0.01602 0.25 -0.035; parent lift_link -> body_link
- joint arm_right_fixed: origin xyz=0.113964 -0.246152 0.012392 rpy=0 0 0 -> xyz=-0.01602 -0.25 -0.035; parent lift_link -> body_link
- joint body_joint: origin xyz=0.138047 0.001801 0.114163 rpy=0 0 0 -> xyz=0.13 0.001801 0.0529 rpy=0 0 0
- joint left_gripper_center_fixed: origin xyz=0.145 0 0 -> xyz=0.1424 0 0.0001057
- joint left_gripper_joint: origin xyz=0.08657 0.024896 -0.0002436 -> xyz=0.08397 0.02721 -0.0062702
- joint left_joint1: limit lower=-2.87 upper=3.14 effort=100 velocity=5 -> lower=-2.094 upper=3.141592653589793 effort=27 velocity=5.5
- joint left_joint2: limit lower=0 upper=3.66 effort=100 velocity=5 -> lower=0 upper=3.665 effort=27 velocity=5.5
- joint left_joint3: axis 0 1 0 -> 0 -1 0; limit lower=0 upper=3.14 effort=100 velocity=5 -> lower=0 upper=3.24 effort=27 velocity=5.5; origin xyz=-0.264 0 0 rpy=3.1416 0 0 -> xyz=-0.264 0 0 rpy=0 0 0
- joint left_joint4: axis 0 1 0 -> 0 -1 0; limit lower=-1.57 upper=1.57 effort=100 velocity=5 -> lower=-1.671 upper=1.671 effort=7 velocity=20; origin xyz=0.245 0 -0.056 -> xyz=0.245 0 0.056
- joint left_joint5: axis 0 0 1 -> 0 0 -1; limit lower=-1.57 upper=1.57 effort=100 velocity=5 -> lower=-1.671 upper=1.671 effort=7 velocity=20; origin xyz=0.06775 0.0005 -0.0865 -> xyz=0.06775 0 0.0845
- joint left_joint6: limit lower=-1.57 upper=1.57 effort=100 velocity=5 -> lower=-2.094 upper=2.094 effort=7 velocity=20; origin xyz=0.02895 0 0.0865 rpy=-3.1416 0 0 -> xyz=0.02895 0 -0.0845
- joint left_joint8: origin xyz=0.08657 -0.0249 -0.00024366 -> xyz=0.08397 -0.023638 -0.0062703
- joint left_left_pad_joint: origin xyz=0.05843 -0.0249 0 -> xyz=0.05843 -0.0249 0.006376
- joint left_right_pad_joint: origin xyz=0.05843 0.0249 0 -> xyz=0.05843 0.0249 0.006376
- joint right_gripper_center_fixed: origin xyz=0.145 0 0 -> xyz=0.1424 0 0.0001057
- joint right_gripper_joint: origin xyz=0.08657 0.024896 -0.0002436 -> xyz=0.08397 0.02721 -0.0062702
- joint right_joint1: limit lower=-2.87 upper=3.14 effort=100 velocity=5 -> lower=-2.094 upper=3.141592653589793 effort=27 velocity=5.5
- joint right_joint2: limit lower=0 upper=3.66 effort=100 velocity=5 -> lower=0 upper=3.665 effort=27 velocity=5.5
- joint right_joint3: axis 0 1 0 -> 0 -1 0; limit lower=0 upper=3.14 effort=100 velocity=5 -> lower=0 upper=3.24 effort=27 velocity=5.5; origin xyz=-0.264 0 0 rpy=3.1416 0 0 -> xyz=-0.264 0 0 rpy=0 0 0
- joint right_joint4: axis 0 1 0 -> 0 -1 0; limit lower=-1.57 upper=1.57 effort=100 velocity=5 -> lower=-1.671 upper=1.671 effort=7 velocity=20; origin xyz=0.245 0 -0.056 -> xyz=0.245 0 0.056
- joint right_joint5: axis 0 0 1 -> 0 0 -1; limit lower=-1.57 upper=1.57 effort=100 velocity=5 -> lower=-1.671 upper=1.671 effort=7 velocity=20; origin xyz=0.06775 0.0005 -0.0865 -> xyz=0.06775 0 0.0845
- joint right_joint6: limit lower=-1.57 upper=1.57 effort=100 velocity=5 -> lower=-2.094 upper=2.094 effort=7 velocity=20; origin xyz=0.02895 0 0.0865 rpy=-3.1416 0 0 -> xyz=0.02895 0 -0.0845
- joint right_joint8: origin xyz=0.08657 -0.0249 -0.00024366 -> xyz=0.08397 -0.023638 -0.0062703
- joint right_left_pad_joint: origin xyz=0.05843 -0.0249 0 -> xyz=0.05843 -0.0249 0.006376
- joint right_right_pad_joint: origin xyz=0.05843 0.0249 0 -> xyz=0.05843 0.0249 0.006376
- joint wheel1_joint: axis 1 0 0 -> (none)
- joint wheel2_joint: axis 1 0 0 -> (none)
- joint wheel3_joint: axis -1 0 0 -> (none); origin xyz=-0.35293 0 -0.093 rpy=0.0 0.0 0 -> xyz=-0.35293 0 -0.093 rpy=0.0 0.0 3.1415

File: arx_lift2s_description/urdf/arx_lift2s_acone_x5.urdf (robot description, URDF)
Before this commit: robot arx_lift2s, 30 links, 29 joints
Links:
- added link head_camera; visual mesh filename=package://sensor_models/meshes/d405/d405.obj
- link left_base_link: geometry collision mesh filename=package://arx5_description/meshes/x5/base_link.glb; visual mesh filename=package://arx5_description/meshes/x5/base_link.glb
- link left_camera: geometry visual mesh filename=package://sensor_models/meshes/d405.glb
- link left_camera_support: geometry visual mesh filename=package://arx5_description/meshes/camera_stand/stand_d405.g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
- link left_link1: geometry collision mesh filename=package://arx5_description/meshes/x5/link1.glb; visual mesh filename=package://arx5_description/meshes/x5/link1.glb
- link left_link2: mass 1.0795 -> 1.1068; geometry collision mesh filename=package://arx5_description/meshes/x5/link2.glb; visual mesh filename=package://arx5_description/meshes/x5/link2.glb
- link left_link3: mass 0.54534 -> 0.54316; geometry collision mesh filename=package://arx5_description/meshes/x5/link3.glb; visual mesh filename=package://arx5_description/meshes/x5/link3.glb
- link left_link4: mass 0.11714 -> 0.11827; geometry collision mesh filename=package://arx5_description/meshes/x5/link4.glb; visual mesh filename=package://arx5_description/meshes/x5/link4.glb
- link left_link5: mass 0.63488 -> 0.67398; geometry collision mesh filename=package://arx5_description/meshes/ac1/link5.glb; visual mesh filename=package://arx5_description/meshes/ac1/link5.glb
- link left_link6: mass 0.44089 -> 0.34667; geometry collision mesh filename=package://arx5_description/meshes/ac1/link6.glb; visual mesh filename=package://arx5_description/meshes/ac1/link6.glb
- link left_link7: mass 0.064798 -> 0.08924; geometry collision mesh filename=package://arx5_description/meshes/ac1/link7.glb; visual mesh filename=package://arx5_description/meshes/ac1/link7.glb
- link left_link8: mass 0.064798 -> 0.089402; geometry collision mesh filename=package://arx5_description/meshes/ac1/link8.glb; visual mesh filename=package://arx5_description/meshes/ac1/link8.glb
- link right_base_link: geometry collision mesh filename=package://arx5_description/meshes/x5/base_link.glb; visual mesh filename=package://arx5_description/meshes/x5/base_link.glb
- link right_camera: geometry visual mesh filename=package://sensor_models/meshes/d405.glb
- link right_camera_support: geometry visual mesh filename=package://arx5_description/meshes/camera_stand/stand_d405.g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
- link right_link1: geometry collision mesh filename=package://arx5_description/meshes/x5/link1.glb; visual mesh filename=package://arx5_description/meshes/x5/link1.glb
- link right_link2: mass 1.0795 -> 1.1068; geometry collision mesh filename=package://arx5_description/meshes/x5/link2.glb; visual mesh filename=package://arx5_description/meshes/x5/link2.glb
- link right_link3: mass 0.54534 -> 0.54316; geometry collision mesh filename=package://arx5_description/meshes/x5/link3.glb; visual mesh filename=package://arx5_description/meshes/x5/link3.glb
- link right_link4: mass 0.11714 -> 0.11827; geometry collision mesh filename=package://arx5_description/meshes/x5/link4.glb; visual mesh filename=package://arx5_description/meshes/x5/link4.glb
- link right_link5: mass 0.63488 -> 0.67398; geometry collision mesh filename=package://arx5_description/meshes/ac1/link5.glb; visual mesh filename=package://arx5_description/meshes/ac1/link5.glb
- link right_link6: mass 0.44089 -> 0.34667; geometry collision mesh filename=package://arx5_description/meshes/ac1/link6.glb; visual mesh filename=package://arx5_description/meshes/ac1/link6.glb
- link right_link7: mass 0.064798 -> 0.08924; geometry collision mesh filename=package://arx5_description/meshes/ac1/link7.glb; visual mesh filename=package://arx5_description/meshes/ac1/link7.glb
- link right_link8: mass 0.064798 -> 0.089402; geometry collision mesh filename=package://arx5_description/meshes/ac1/link8.glb; visual mesh filename=package://arx5_description/meshes/ac1/link8.glb
Joints:
- added joint head_camera_joint: type fixed, parent body_link, child head_camera, origin xyz=0.090415 0.002 0.2285 rpy=0 1.0472 0
- joint left_gripper_center_fixed: origin xyz=0.145 0 0 -> xyz=0.1424 0 0.0001057
- joint left_gripper_joint: origin xyz=0.08657 0.024896 -0.0002436 -> xyz=0.08397 0.02721 -0.0062702
- joint left_joint1: limit lower=-2.87 upper=3.14 effort=100 velocity=5 -> lower=-2.094 upper=3.141592653589793 effort=27 velocity=5.5
- joint left_joint2: limit lower=0 upper=3.66 effort=100 velocity=5 -> lower=0 upper=3.665 effort=27 velocity=5.5
- joint left_joint3: axis 0 1 0 -> 0 -1 0; limit lower=0 upper=3.14 effort=100 velocity=5 -> lower=0 upper=3.24 effort=27 velocity=5.5; origin xyz=-0.264 0 0 rpy=3.1416 0 0 -> xyz=-0.264 0 0 rpy=0 0 0
- joint left_joint4: axis 0 1 0 -> 0 -1 0; limit lower=-1.57 upper=1.57 effort=100 velocity=5 -> lower=-1.671 upper=1.671 effort=7 velocity=20; origin xyz=0.245 0 -0.056 -> xyz=0.245 0 0.056
- joint left_joint5: axis 0 0 1 -> 0 0 -1; limit lower=-1.57 upper=1.57 effort=100 velocity=5 -> lower=-1.671 upper=1.671 effort=7 velocity=20; origin xyz=0.06775 0.0005 -0.0865 -> xyz=0.06775 0 0.0845
- joint left_joint6: limit lower=-1.57 upper=1.57 effort=100 velocity=5 -> lower=-2.094 upper=2.094 effort=7 velocity=20; origin xyz=0.02895 0 0.0865 rpy=-3.1416 0 0 -> xyz=0.02895 0 -0.0845
- joint left_joint8: origin xyz=0.08657 -0.0249 -0.00024366 -> xyz=0.08397 -0.023638 -0.0062703
- joint left_left_pad_joint: origin xyz=0.05843 -0.0249 0 -> xyz=0.05843 -0.0249 0.006376
- joint left_right_pad_joint: origin xyz=0.05843 0.0249 0 -> xyz=0.05843 0.0249 0.006376
- joint right_gripper_center_fixed: origin xyz=0.145 0 0 -> xyz=0.1424 0 0.0001057
- joint right_gripper_joint: origin xyz=0.08657 0.024896 -0.0002436 -> xyz=0.08397 0.02721 -0.0062702
- joint right_joint1: limit lower=-2.87 upper=3.14 effort=100 velocity=5 -> lower=-2.094 upper=3.141592653589793 effort=27 velocity=5.5
- joint right_joint2: limit lower=0 upper=3.66 effort=100 velocity=5 -> lower=0 upper=3.665 effort=27 velocity=5.5
- joint right_joint3: axis 0 1 0 -> 0 -1 0; limit lower=0 upper=3.14 effort=100 velocity=5 -> lower=0 upper=3.24 effort=27 velocity=5.5; origin xyz=-0.264 0 0 rpy=3.1416 0 0 -> xyz=-0.264 0 0 rpy=0 0 0
- joint right_joint4: axis 0 1 0 -> 0 -1 0; limit lower=-1.57 upper=1.57 effort=100 velocity=5 -> lower=-1.671 upper=1.671 effort=7 velocity=20; origin xyz=0.245 0 -0.056 -> xyz=0.245 0 0.056
- joint right_joint5: axis 0 0 1 -> 0 0 -1; limit lower=-1.57 upper=1.57 effort=100 velocity=5 -> lower=-1.671 upper=1.671 effort=7 velocity=20; origin xyz=0.06775 0.0005 -0.0865 -> xyz=0.06775 0 0.0845
- joint right_joint6: limit lower=-1.57 upper=1.57 effort=100 velocity=5 -> lower=-2.094 upper=2.094 effort=7 velocity=20; origin xyz=0.02895 0 0.0865 rpy=-3.1416 0 0 -> xyz=0.02895 0 -0.0845
- joint right_joint8: origin xyz=0.08657 -0.0249 -0.00024366 -> xyz=0.08397 -0.023638 -0.0062703
- joint right_left_pad_joint: origin xyz=0.05843 -0.0249 0 -> xyz=0.05843 -0.0249 0.006376
- joint right_right_pad_joint: origin xyz=0.05843 0.0249 0 -> xyz=0.05843 0.0249 0.006376

File: arx_lift2s_description/xacro/robot.xacro (robot description, xacro)
@@ -36,5 +36,5 @@
 	<xacro:ac_one/>
 	<xacro:if value="${selected_arm_type == 'x5'}">
-		<xacro:include filename="$(find arx5_description)/xacro/X5.xacro"/>
+		<xacro:include filename="$(find arx5_description)/xacro/X5_ac1.xacro"/>
 		<xacro:X5 name="left"/>
 		<xacro:X5 name="right"/>
