Commit message: update

File: arx_lift2s_description/urdf/arx_lift2s_acone_x5.urdf (robot description, URDF)
Before this commit: robot arx_lift2s, 31 links, 30 joints
Links:
- removed link head_camera
Joints:
- removed joint head_camera_joint

File: arx_lift2s_description/xacro/ros2_control/robot.xacro (robot description, xacro)
@@ -1,6 +1,4 @@
 <?xml version="1.0"?>
 <robot xmlns:xacro="http://www.ros.org/wiki/xacro" name="arx_lift2s">
-    <xacro:arg name="type" default="x5"/>
-    <xacro:arg name="enable_wheel_joints" default="true"/>
     <xacro:arg name="ros2_control_hardware_type" default="mock_components"/>
     <xacro:include filename="$(find arx_lift2s_description)/xacro/robot.xacro"/>
@@ -29,9 +27,9 @@
             </xacro:if>
         </hardware>
-        <xacro:arx_lift2s_base_interfaces/>
-        <xacro:unless value="${'$(arg type)' == 'wheel'}">
-            <xacro:arx5_interfaces name="left"/>
-            <xacro:arx5_interfaces name="right"/>
-        </xacro:unless>
+        <xacro:if value="${selected_base_type == 'lift2s'}">
+            <xacro:arx_lift2s_base_interfaces/>
+        </xacro:if>
+        <xacro:arx5_interfaces name="left"/>
+        <xacro:arx5_interfaces name="right"/>
     </ros2_control>
     <xacro:if value="$(arg gazebo)">

Commit message: ACONE简单碰撞体及自碰撞已配置

File: arx_lift2s_description/urdf/arx_lift2s_acone_x5.urdf (robot description, URDF)
Before this commit: robot arx_lift2s, 31 links, 30 joints
Links:
- link body_link: geometry collision box size=0.04 0.06 0.1; collision box size=0.04 0.06 0.3
- link head_camera: geometry visual mesh filename=file:///home/shimanliang/ros2_ws/install/sensor_models/shar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
- link left_base_link: geometry collision cylinder length=0.03125 radius=0.031; visual mesh filename=file:///home/shimanliang/ros2_ws/install/arx5_description/s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
- link left_camera: geometry collision box size=0.0231 0.0421 0.042; visual mesh filename=file:///home/shimanliang/ros2_ws/install/sensor_models/shar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
- link left_camera_support: geometry collision box size=0.01 0.05 0.03; collision box size=0.01 0.05 0.06
- link left_link1: geometry collision mesh filename=file:///home/shimanliang/ros2_ws/install/arx5_description/s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; visual mesh filename=file:///home/shimanliang/ros2_ws/install/arx5_description/s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
- link left_link2: geometry collision box size=0.264 0.05 0.05; collision cylinder length=0.0665 radius=0.028
- link left_link3: geometry collision box size=0.2 0.04 0.045; collision cylinder length=0.049 radius=0.03
- link left_link4: geometry collision cylinder length=0.04 radius=0.0315; visual mesh filename=file:///home/shimanliang/ros2_ws/install/arx5_description/s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
- link left_link5: geometry collision cylinder length=0.013 radius=0.03145; collision cylinder length=0.045 radius=0.03145
- link left_link6: geometry collision cylinder length=0.064 radius=0.03015; visual mesh filename=file:///home/shimanliang/ros2_ws/install/arx5_description/s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
- link left_link7: geometry collision box size=0.08 0.04 0.0640; visual mesh filename=file:///home/shimanliang/ros2_ws/install/arx5_description/s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
- link left_link8: geometry collision box size=0.08 0.04 0.0640; visual mesh filename=file:///home/shimanliang/ros2_ws/install/arx5_description/s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
- link right_base_link: geometry collision cylinder length=0.03125 radius=0.031; visual mesh filename=file:///home/shimanliang/ros2_ws/install/arx5_description/s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
- link right_camera: geometry collision box size=0.0231 0.0421 0.042; visual mesh filename=file:///home/shimanliang/ros2_ws/install/sensor_models/shar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
- link right_camera_support: geometry collision box size=0.01 0.05 0.03; collision box size=0.01 0.05 0.06
- link right_link1: geometry collision mesh filename=file:///home/shimanliang/ros2_ws/install/arx5_description/s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; visual mesh filename=file:///home/shimanliang/ros2_ws/install/arx5_description/s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
- link right_link2: geometry collision box size=0.264 0.05 0.05; collision cylinder length=0.0665 radius=0.028
- link right_link3: geometry collision box size=0.2 0.04 0.045; collision cylinder length=0.049 radius=0.03
- link right_link4: geometry collision cylinder length=0.04 radius=0.0315; visual mesh filename=file:///home/shimanliang/ros2_ws/install/arx5_description/s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
- link right_link5: geometry collision cylinder length=0.013 radius=0.03145; collision cylinder length=0.045 radius=0.03145
- link right_link6: geometry collision cylinder length=0.064 radius=0.03015; visual mesh filename=file:///home/shimanliang/ros2_ws/install/arx5_description/s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
- link right_link7: geometry collision box size=0.08 0.04 0.0640; visual mesh filename=file:///home/shimanliang/ros2_ws/install/arx5_description/s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
- link right_link8: geometry collision box size=0.08 0.04 0.0640; visual mesh filename=file:///home/shimanliang/ros2_ws/install/arx5_description/s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

Commit message: x5_ac1碰撞体添加

File: arx_lift2s_description/urdf/arx_lift2s_acone_x5.urdf (robot description, URDF)
Before this commit: robot arx_lift2s, 31 links, 30 joints
Links:
- link left_link2: mass 1.0795 -> 1.1068
- link left_link3: mass 0.54534 -> 0.54316
- link left_link4: mass 0.11714 -> 0.11827
- link left_link5: mass 0.63488 -> 0.67398; geometry collision cylinder length=0.013 radius=0.03145; collision cylinder length=0.045 radius=0.03145
- link left_link6: mass 0.44089 -> 0.34667; geometry collision cylinder length=0.064 radius=0.03015; visual mesh filename=package://arx5_description/meshes/ac1/link6.glb
- link left_link7: mass 0.064798 -> 0.08924; geometry collision box size=0.08 0.04 0.0640; visual mesh filename=package://arx5_description/meshes/ac1/link7.glb
- link left_link8: mass 0.064798 -> 0.089402; geometry collision box size=0.08 0.04 0.0640; visual mesh filename=package://arx5_description/meshes/ac1/link8.glb
- link right_link2: mass 1.0795 -> 1.1068
- link right_link3: mass 0.54534 -> 0.54316
- link right_link4: mass 0.11714 -> 0.11827
- link right_link5: mass 0.63488 -> 0.67398; geometry collision cylinder length=0.013 radius=0.03145; collision cylinder length=0.045 radius=0.03145
- link right_link6: mass 0.44089 -> 0.34667; geometry collision cylinder length=0.064 radius=0.03015; visual mesh filename=package://arx5_description/meshes/ac1/link6.glb
- link right_link7: mass 0.064798 -> 0.08924; geometry collision box size=0.08 0.04 0.0640; visual mesh filename=package://arx5_description/meshes/ac1/link7.glb
- link right_link8: mass 0.064798 -> 0.089402; geometry collision box size=0.08 0.04 0.0640; visual mesh filename=package://arx5_description/meshes/ac1/link8.glb
Joints:
- joint left_gripper_center_fixed: origin xyz=0.145 0 0 -> xyz=0.1424 0 0.0001057
- joint left_gripper_joint: origin xyz=0.08657 0.024896 -0.0002436 -> xyz=0.08397 0.02721 -0.0062702
- joint left_joint1: limit lower=-2.87 upper=3.14 effort=100 velocity=5 -> lower=-2.094 upper=3.141592653589793 effort=27 velocity=5.5
- joint left_joint2: limit lower=0 upper=3.66 effort=100 velocity=5 -> lower=0 upper=3.665 effort=27 velocity=5.5
- joint left_joint3: axis 0 1 0 -> 0 -1 0; limit lower=0 upper=3.14 effort=100 velocity=5 -> lower=0 upper=3.24 effort=27 velocity=5.5; origin xyz=-0.264 0 0 rpy=3.1416 0 0 -> xyz=-0.264 0 0 rpy=0 0 0
- joint left_joint4: axis 0 1 0 -> 0 -1 0; limit lower=-1.57 upper=1.57 effort=100 velocity=5 -> lower=-1.671 upper=1.671 effort=7 velocity=20; origin xyz=0.245 0 -0.056 -> xyz=0.245 0 0.056
- joint left_joint5: axis 0 0 1 -> 0 0 -1; limit lower=-1.57 upper=1.57 effort=100 velocity=5 -> lower=-1.671 upper=1.671 effort=7 velocity=20; origin xyz=0.06775 0.0005 -0.0865 -> xyz=0.06775 0 0.0845
- joint left_joint6: limit lower=-1.57 upper=1.57 effort=100 velocity=5 -> lower=-2.094 upper=2.094 effort=7 velocity=20; origin xyz=0.02895 0 0.0865 rpy=-3.1416 0 0 -> xyz=0.02895 0 -0.0845
- joint left_joint8: origin xyz=0.08657 -0.0249 -0.00024366 -> xyz=0.08397 -0.023638 -0.0062703
- joint left_left_pad_joint: origin xyz=0.05843 -0.0249 0 -> xyz=0.05843 -0.0249 0.006376
- joint left_right_pad_joint: origin xyz=0.05843 0.0249 0 -> xyz=0.05843 0.0249 0.006376
- joint right_gripper_center_fixed: origin xyz=0.145 0 0 -> xyz=0.1424 0 0.0001057
- joint right_gripper_joint: origin xyz=0.08657 0.024896 -0.0002436 -> xyz=0.08397 0.02721 -0.0062702
- joint right_joint1: limit lower=-2.87 upper=3.14 effort=100 velocity=5 -> lower=-2.094 upper=3.141592653589793 effort=27 velocity=5.5
- joint right_joint2: limit lower=0 upper=3.66 effort=100 velocity=5 -> lower=0 upper=3.665 effort=27 velocity=5.5
- joint right_joint3: axis 0 1 0 -> 0 -1 0; limit lower=0 upper=3.14 effort=100 velocity=5 -> lower=0 upper=3.24 effort=27 velocity=5.5; origin xyz=-0.264 0 0 rpy=3.1416 0 0 -> xyz=-0.264 0 0 rpy=0 0 0
- joint right_joint4: axis 0 1 0 -> 0 -1 0; limit lower=-1.57 upper=1.57 effort=100 velocity=5 -> lower=-1.671 upper=1.671 effort=7 velocity=20; origin xyz=0.245 0 -0.056 -> xyz=0.245 0 0.056
- joint right_joint5: axis 0 0 1 -> 0 0 -1; limit lower=-1.57 upper=1.57 effort=100 velocity=5 -> lower=-1.671 upper=1.671 effort=7 velocity=20; origin xyz=0.06775 0.0005 -0.0865 -> xyz=0.06775 0 0.0845
- joint right_joint6: limit lower=-1.57 upper=1.57 effort=100 velocity=5 -> lower=-2.094 upper=2.094 effort=7 velocity=20; origin xyz=0.02895 0 0.0865 rpy=-3.1416 0 0 -> xyz=0.02895 0 -0.0845
- joint right_joint8: origin xyz=0.08657 -0.0249 -0.00024366 -> xyz=0.08397 -0.023638 -0.0062703
- joint right_left_pad_joint: origin xyz=0.05843 -0.0249 0 -> xyz=0.05843 -0.0249 0.006376
- joint right_right_pad_joint: origin xyz=0.05843 0.0249 0 -> xyz=0.05843 0.0249 0.006376

File: arx_lift2s_description/xacro/robot.xacro (robot description, xacro)
@@ -37,5 +37,5 @@
 	<xacro:ac_one collider="$(arg collider)"/>
 	<xacro:if value="${selected_arm_type == 'x5'}">
-		<xacro:include filename="$(find arx5_description)/xacro/X5.xacro"/>
+		<xacro:include filename="$(find arx5_description)/xacro/X5_ac1.xacro"/>
 		<xacro:X5 name="left" collider="$(arg collider)"/>
 		<xacro:X5 name="right" collider="$(arg collider)"/>
