Commit message: 改为单hardware

File: arx5_description/xacro/ros2_control/robot.xacro (robot description, xacro)
@@ -1,53 +1,58 @@
 <?xml version="1.0"?>
 <robot xmlns:xacro="http://www.ros.org/wiki/xacro" name="R5a">
-  <xacro:arg name="ros2_control_hardware_type" default="mock_components" />
-  <link name="world"/>
-  <joint name="world_fixed" type="fixed">
-    <parent link="world"/>
-    <child link="base_link"/>
-  </joint>
-  <!-- Include the base robot structure -->
-  <xacro:include filename="$(find arx5_description)/xacro/robot.xacro"/>
-  <xacro:include filename="$(find arx5_description)/xacro/ros2_control/interfaces.xacro"/>
-  <ros2_control name="arx5_system" type="system">
-    <hardware>
-      <xacro:if value="${'$(arg ros2_control_hardware_type)' == 'gz'}">
-        <plugin>gz_ros2_control/GazeboSimSystem</plugin>
-      </xacro:if>
-      <xacro:if value="${'$(arg ros2_control_hardware_type)' == 'mock_components'}">
-        <plugin>mock_components/GenericSystem</plugin>
-      </xacro:if>
-      <xacro:if value="${'$(arg ros2_control_hardware_type)' == 'isaac'}">
-        <plugin>topic_based_ros2_control/TopicBasedSystem</plugin>
-        <param name="joint_commands_topic">/isaac/joint_command</param>
-        <param name="joint_states_topic">/isaac/joint_states</param>
-      </xacro:if>
-      <xacro:if value="${'$(arg ros2_control_hardware_type)' == 'real'}">
-        <plugin>arx_ros2_control/ArxX5Hardware</plugin>
-        <param name="arm_config">LEFT</param>
-        <param name="robot_model">X5</param>
-        <param name="can_interface">can1</param>
-        <!-- 单臂默认增益，可按需修改 -->
-        <param name="joint_k_gains">[80.0, 70.0, 70.0, 30.0, 30.0, 20.0]</param>
-        <param name="joint_d_gains">[2.0, 2.0, 2.0, 1.0, 1.0, 0.7]</param>
-        <param name="gripper_kp">5.0</param>
-        <param name="gripper_kd">0.2</param>
-      </xacro:if>
-    </hardware>
-    <!-- 基座接口 -->
-    <xacro:arx5_interfaces name=""/>
-  </ros2_control>
-  <xacro:arg name="gazebo" default="false" />
-  <xacro:if value="$(arg gazebo)">
-    <gazebo>
-      <plugin filename="gz_ros2_control-system" name="gz_ros2_control::GazeboSimROS2ControlPlugin">
-        <xacro:if value="${'$(arg type)' == 'r5'}">
-          <parameters>$(find arx5_description)/config/ros2_control/arx_r5.yaml</parameters>
-        </xacro:if>
-        <xacro:if value="${'$(arg type)' == 'x5'}">
-          <parameters>$(find arx5_description)/config/ros2_control/ros2_controllers.yaml</parameters>
-        </xacro:if>
-      </plugin>
-    </gazebo>
-  </xacro:if>
+    <xacro:arg name="ros2_control_hardware_type" default="mock_components"/>
+    <xacro:arg name="gazebo" default="false"/>
+    <xacro:arg name="type" default="x5"/>
+    <link name="world"/>
+    <joint name="world_fixed" type="fixed">
+        <parent link="world"/>
+        <child link="base_link"/>
+    </joint>
+    <xacro:include filename="$(find arx5_description)/xacro/robot.xacro"/>
+    <xacro:include filename="$(find arx5_description)/xacro/ros2_control/interfaces.xacro"/>
+    <xacro:if value="${'$(arg ros2_control_hardware_type)' == 'real'}">
+        <ros2_control name="arx5_system" type="system">
+            <hardware>
+                <plugin>arx_ros2_control/ArxX5Hardware</plugin>
+                <param name="robot_model">X5</param>
+                <param name="can_interface">can1</param>
+                <param name="joint_k_gains">[80.0, 70.0, 70.0, 30.0, 30.0, 20.0]</param>
+                <param name="joint_d_gains">[2.0, 2.0, 2.0, 1.0, 1.0, 0.7]</param>
+                <!-- 可选：夹爪增益，不写则用默认 -->
+                <!-- <param name="gripper_kp">5.0</param> -->
+                <!-- <param name="gripper_kd">0.2</param> -->
+            </hardware>
+            <xacro:arx5_interfaces name=""/>
+        </ros2_control>
+    </xacro:if>
+    <xacro:unless value="${'$(arg ros2_control_hardware_type)' == 'real'}">
+        <ros2_control name="arx5_system" type="system">
+            <hardware>
+                <xacro:if value="${'$(arg ros2_control_hardware_type)' == 'gz'}">
+                    <plugin>gz_ros2_control/GazeboSimSystem</plugin>
+                </xacro:if>
+                <xacro:if value="${'$(arg ros2_control_hardware_type)' == 'mock_components'}">
+                    <plugin>mock_components/GenericSystem</plugin>
+                </xacro:if>
+                <xacro:if value="${'$(arg ros2_control_hardware_type)' == 'isaac'}">
+                    <plugin>topic_based_ros2_control/TopicBasedSystem</plugin>
+                    <param name="joint_commands_topic">/isaac/joint_command</param>
+                    <param name="joint_states_topic">/isaac/joint_states</param>
+                </xacro:if>
+            </hardware>
+            <xacro:arx5_interfaces name=""/>
+        </ros2_control>
+    </xacro:unless>
+    <xacro:if value="$(arg gazebo)">
+        <gazebo>
+            <plugin filename="gz_ros2_control-system" name="gz_ros2_control::GazeboSimROS2ControlPlugin">
+                <xacro:if value="${'$(arg type)' == 'r5'}">
+                    <parameters>$(find arx5_description)/config/ros2_control/arx_r5.yaml</parameters>
+                </xacro:if>
+                <xacro:if value="${'$(arg type)' == 'x5'}">
+                    <parameters>$(find arx5_description)/config/ros2_control/ros2_controllers.yaml</parameters>
+                </xacro:if>
+            </plugin>
+        </gazebo>
+    </xacro:if>
 </robot>

File: arx_lift2s_description/xacro/ros2_control/robot.xacro (robot description, xacro)
@@ -2,45 +2,58 @@
 <robot xmlns:xacro="http://www.ros.org/wiki/xacro" name="arx_lift2s">
     <xacro:arg name="ros2_control_hardware_type" default="mock_components"/>
+    <xacro:arg name="gazebo" default="false"/>
     <xacro:include filename="$(find arx_lift2s_description)/xacro/robot.xacro"/>
     <xacro:include filename="$(find arx5_description)/xacro/ros2_control/interfaces.xacro"/>
     <xacro:include filename="$(find arx_lift2s_description)/xacro/ros2_control/interfaces.xacro"/>
-    <ros2_control name="arx_lift2s_unified_system" type="system">
-        <hardware>
-            <xacro:if value="${'$(arg ros2_control_hardware_type)' == 'gz'}">
-                <plugin>gz_ros2_control/GazeboSimSystem</plugin>
+    <xacro:if value="${'$(arg ros2_control_hardware_type)' == 'real'}">
+        <ros2_control name="arx_lift2s_left_system" type="system">
+            <hardware>
+                <plugin>arx_ros2_control/ArxX5Hardware</plugin>
+                <param name="robot_model">X5</param>
+                <param name="can_interface">can1</param>
+                <param name="joint_k_gains">[80.0, 70.0, 70.0, 30.0, 30.0, 20.0]</param>
+                <param name="joint_d_gains">[2.0, 2.0, 2.0, 1.0, 1.0, 0.7]</param>
+                <!-- 可选：夹爪增益，不写则用默认 -->
+                <!-- <param name="gripper_kp">5.0</param> -->
+                <!-- <param name="gripper_kd">0.2</param> -->
+            </hardware>
+            <xacro:arx5_interfaces name="left"/>
+        </ros2_control>
+        <ros2_control name="arx_lift2s_right_system" type="system">
+            <hardware>
+                <plugin>arx_ros2_control/ArxX5Hardware</plugin>
+                <param name="robot_model">X5</param>
+                <param name="can_interface">can3</param>
+                <param name="joint_k_gains">[80.0, 70.0, 70.0, 30.0, 30.0, 20.0]</param>
+                <param name="joint_d_gains">[2.0, 2.0, 2.0, 1.0, 1.0, 0.7]</param>
+                <!-- 可选：夹爪增益，不写则用默认 -->
+                <!-- <param name="gripper_kp">5.0</param> -->
+                <!-- <param name="gripper_kd">0.2</param> -->
+            </hardware>
+            <xacro:arx5_interfaces name="right"/>
+        </ros2_control>
+    </xacro:if>
+    <xacro:unless value="${'$(arg ros2_control_hardware_type)' == 'real'}">
+        <ros2_control name="arx_lift2s_system" type="system">
+            <hardware>
+                <xacro:if value="${'$(arg ros2_control_hardware_type)' == 'gz'}">
+                    <plugin>gz_ros2_control/GazeboSimSystem</plugin>
+                </xacro:if>
+                <xacro:if value="${'$(arg ros2_control_hardware_type)' == 'mock_components'}">
+                    <plugin>mock_components/GenericSystem</plugin>
+                </xacro:if>
+                <xacro:if value="${'$(arg ros2_control_hardware_type)' == 'isaac'}">
+                    <plugin>topic_based_ros2_control/TopicBasedSystem</plugin>
+                    <param name="joint_commands_topic">/isaac/joint_command</param>
+                    <param name="joint_states_topic">/isaac/joint_states</param>
+                </xacro:if>
+            </hardware>
+            <xacro:if value="${selected_base_type == 'lift2s'}">
+                <xacro:arx_lift2s_base_interfaces/>
             </xacro:if>
-            <xacro:if value="${'$(arg ros2_control_hardware_type)' == 'mock_components'}">
-                <plugin>mock_components/GenericSystem</plugin>
-            </xacro:if>
-            <xacro:if value="${'$(arg ros2_control_hardware_type)' == 'isaac'}">
-                <plugin>topic_based_ros2_control/TopicBasedSystem</plugin>
-                <param name="joint_commands_topic">/isaac/joint_command</param>
-                <param name="joint_states_topic">/isaac/joint_states</param>
-            </xacro:if>
-            <xacro:if value="${'$(arg ros2_control_hardware_type)' == 'real'}">
-                <plugin>arx_ros2_control/ArxX5Hardware</plugin>
-                <param name="arm_config">DUAL</param>
-                <param name="left_robot_model">X5</param>
-                <param name="right_robot_model">X5</param>
-                <param name="left_can_interface">can1</param>
-                <param name="right_can_interface">can3</param>
-                <!-- 双臂初始增益：可为左右臂设置不同的 kp/kd，不写则两臂使用相同默认值 -->
-                <param name="left_joint_k_gains">[80.0, 70.0, 70.0, 30.0, 30.0, 20.0]</param>
-                <param name="left_joint_d_gains">[2.0, 2.0, 2.0, 1.0, 1.0, 0.7]</param>
-                <param name="right_joint_k_gains">[80.0, 70.0, 70.0, 30.0, 30.0, 20.0]</param>
-                <param name="right_joint_d_gains">[2.0, 2.0, 2.0, 1.0, 1.0, 0.7]</param>
-                <!-- 可选：左右夹爪增益，不写则用默认 -->
-                <!-- <param name="left_gripper_kp">5.0</param> -->
-                <!-- <param name="left_gripper_kd">0.2</param> -->
-                <!-- <param name="right_gripper_kp">5.0</param> -->
-                <!-- <param name="right_gripper_kd">0.2</param> -->
-            </xacro:if>
-        </hardware>
-        <xacro:if value="${selected_base_type == 'lift2s'}">
-            <xacro:arx_lift2s_base_interfaces/>
-        </xacro:if>
-        <xacro:arx5_interfaces name="left"/>
-        <xacro:arx5_interfaces name="right"/>
-    </ros2_control>
+            <xacro:arx5_interfaces name="left"/>
+            <xacro:arx5_interfaces name="right"/>
+        </ros2_control>
+    </xacro:unless>
     <xacro:if value="$(arg gazebo)">
         <gazebo>
