Commit message: add feedforward for arm

File: arx5_description/xacro/ros2_control/interfaces.xacro (robot description, xacro)
@@ -4,5 +4,89 @@
         <xacro:property name="prefix" value="${name + '_' if name else ''}"/>
         <xacro:arg name="gazebo" default="false"/>
-        <!-- 关节接口定义 -->
+        <!-- Arm joints: always declare MIX interfaces (control_mode selects write usage). -->
+        <joint name="${prefix}joint1">
+            <command_interface name="position"/>
+            <command_interface name="velocity"/>
+            <command_interface name="effort"/>
+            <command_interface name="kp"/>
+            <command_interface name="kd"/>
+            <state_interface name="position"/>
+            <state_interface name="velocity"/>
+            <state_interface name="effort"/>
+        </joint>
+        <joint name="${prefix}joint2">
+            <command_interface name="position"/>
+            <command_interface name="velocity"/>
+            <command_interface name="effort"/>
+            <command_interface name="kp"/>
+            <command_interface name="kd"/>
+            <state_interface name="position">
+                <param name="initial_value">0.4</param>
+            </state_interface>
+            <state_interface name="velocity"/>
+            <state_interface name="effort"/>
+        </joint>
+        <joint name="${prefix}joint3">
+            <command_interface name="position"/>
+            <command_interface name="velocity"/>
+            <command_interface name="effort"/>
+            <command_interface name="kp"/>
+            <command_interface name="kd"/>
+            <state_interface name="position">
+                <param name="initial_value">0.12</param>
+            </state_interface>
+            <state_interface name="velocity"/>
+            <state_interface name="effort"/>
+        </joint>
+        <joint name="${prefix}joint4">
+            <command_interface name="position"/>
+            <command_interface name="velocity"/>
+            <command_interface name="effort"/>
+            <command_interface name="kp"/>
+            <command_interface name="kd"/>
+            <state_interface name="position">
+                <param name="initial_value">0.26</param>
+            </state_interface>
+            <state_interface name="velocity"/>
+            <state_interface name="effort"/>
+        </joint>
+        <joint name="${prefix}joint5">
+            <command_interface name="position"/>
+            <command_interface name="velocity"/>
+            <command_interface name="effort"/>
+            <command_interface name="kp"/>
+            <command_interface name="kd"/>
+            <state_interface name="position"/>
+            <state_interface name="velocity"/>
+            <state_interface name="effort"/>
+        </joint>
+        <joint name="${prefix}joint6">
+            <command_interface name="position"/>
+            <command_interface name="velocity"/>
+            <command_interface name="effort"/>
+            <command_interface name="kp"/>
+            <command_interface name="kd"/>
+            <state_interface name="position"/>
+            <state_interface name="velocity"/>
+            <state_interface name="effort"/>
+        </joint>
+        <!-- Gripper stays position-only (AdaptiveGripperController). -->
+        <joint name="${prefix}gripper_joint">
+            <command_interface name="position"/>
+            <state_interface name="position"/>
+            <state_interface name="velocity"/>
+            <state_interface name="effort"/>
+        </joint>
+        <xacro:if value="$(arg gazebo)">
+            <joint name="${prefix}joint8">
+                <state_interface name="position"/>
+                <state_interface name="velocity"/>
+                <state_interface name="effort"/>
+            </joint>
+        </xacro:if>
+    </xacro:macro>
+    <!-- Position-only arm interfaces for official arxlift2s_ros2_control (Lift2S). -->
+    <xacro:macro name="arx5_interfaces_position" params="name">
+        <xacro:property name="prefix" value="${name + '_' if name else ''}"/>
         <joint name="${prefix}joint1">
             <command_interface name="position"/>
@@ -53,11 +137,4 @@
             <state_interface name="effort"/>
         </joint>
-        <xacro:if value="$(arg gazebo)">
-            <joint name="${prefix}joint8">
-                <state_interface name="position"/>
-                <state_interface name="velocity"/>
-                <state_interface name="effort"/>
-            </joint>
-        </xacro:if>
     </xacro:macro>
 </robot>

File: arx5_description/xacro/ros2_control/robot.xacro (robot description, xacro)
@@ -4,4 +4,6 @@
     <xacro:arg name="gazebo" default="false"/>
     <xacro:arg name="type" default="x5"/>
+    <!-- full_control (default, OCS2 MIX) | position (legacy: pos + param kp/kd) -->
+    <xacro:arg name="control_mode" default="full_control"/>
     <link name="world"/>
     <joint name="world_fixed" type="fixed">
@@ -17,4 +19,5 @@
                 <param name="robot_model">X5</param>
                 <param name="can_interface">can1</param>
+                <param name="control_mode">$(arg control_mode)</param>
                 <param name="joint_k_gains">[80.0, 70.0, 70.0, 30.0, 30.0, 20.0]</param>
                 <param name="joint_d_gains">[2.0, 2.0, 2.0, 1.0, 1.0, 0.7]</param>

File: arx_acone_description/xacro/ros2_control/robot.xacro (robot description, xacro)
@@ -3,12 +3,16 @@
 	<xacro:arg name="ros2_control_hardware_type" default="mock_components"/>
 	<xacro:arg name="gazebo" default="false"/>
+	<!-- full_control (default, OCS2 MIX) | position (legacy) — Stanford HI only -->
+	<xacro:arg name="control_mode" default="full_control"/>
 	<xacro:include filename="$(find arx_acone_description)/xacro/robot.xacro"/>
 	<xacro:include filename="$(find arx5_description)/xacro/ros2_control/interfaces.xacro"/>
 	<xacro:if value="${'$(arg ros2_control_hardware_type)' == 'real'}">
+		<!-- Dual-arm real: Stanford arx5-sdk (same stack as arx5 single-arm). -->
 		<ros2_control name="arx_acone_left_system" type="system">
 			<hardware>
-				<plugin>arxlift2s_ros2_control/ArxX5Hardware</plugin>
+				<plugin>arx_ros2_control/ArxX5Hardware</plugin>
 				<param name="robot_model">X5</param>
 				<param name="can_interface">can1</param>
+				<param name="control_mode">$(arg control_mode)</param>
 				<param name="joint_k_gains">[80.0, 70.0, 70.0, 30.0, 30.0, 20.0]</param>
 				<param name="joint_d_gains">[2.0, 2.0, 2.0, 1.0, 1.0, 0.7]</param>
@@ -18,7 +22,8 @@
 		<ros2_control name="arx_acone_right_system" type="system">
 			<hardware>
-				<plugin>arxlift2s_ros2_control/ArxX5Hardware</plugin>
+				<plugin>arx_ros2_control/ArxX5Hardware</plugin>
 				<param name="robot_model">X5</param>
 				<param name="can_interface">can3</param>
+				<param name="control_mode">$(arg control_mode)</param>
 				<param name="joint_k_gains">[80.0, 70.0, 70.0, 30.0, 30.0, 20.0]</param>
 				<param name="joint_d_gains">[2.0, 2.0, 2.0, 1.0, 1.0, 0.7]</param>

File: arx_lift2s_description/xacro/ros2_control/robot.xacro (robot description, xacro)
@@ -16,5 +16,6 @@
 				<param name="joint_d_gains">[2.0, 2.0, 2.0, 1.0, 1.0, 0.7]</param>
 			</hardware>
-			<xacro:arx5_interfaces name="left"/>
+			<!-- Official HI exports position only — do not use MIX arx5_interfaces. -->
+			<xacro:arx5_interfaces_position name="left"/>
 		</ros2_control>
 		<ros2_control name="arx_lift2s_right_system" type="system">
@@ -26,5 +27,5 @@
 				<param name="joint_d_gains">[2.0, 2.0, 2.0, 1.0, 1.0, 0.7]</param>
 			</hardware>
-			<xacro:arx5_interfaces name="right"/>
+			<xacro:arx5_interfaces_position name="right"/>
 		</ros2_control>
 		<!-- Lift column: official LIFT2S lift HW (can5) -->
@@ -53,6 +54,7 @@
 			</hardware>
 			<xacro:arx_lift2s_base_interfaces/>
-			<xacro:arx5_interfaces name="left"/>
-			<xacro:arx5_interfaces name="right"/>
+			<!-- Sim/mock: keep position-only to match Lift2S official real HI. -->
+			<xacro:arx5_interfaces_position name="left"/>
+			<xacro:arx5_interfaces_position name="right"/>
 		</ros2_control>
 	</xacro:unless>

Commit message: update the descritpionf

File: arx5_description/xacro/ros2_control/interfaces.xacro (robot description, xacro)
@@ -4,5 +4,5 @@
         <xacro:property name="prefix" value="${name + '_' if name else ''}"/>
         <xacro:arg name="gazebo" default="false"/>
-        <!-- Arm joints: always declare MIX interfaces (control_mode selects write usage). -->
+        <!-- Arm joints: MIX interfaces for full_control (MIT). -->
         <joint name="${prefix}joint1">
             <command_interface name="position"/>
@@ -86,55 +86,3 @@
         </xacro:if>
     </xacro:macro>
-    <!-- Position-only arm interfaces for official arxlift2s_ros2_control (Lift2S). -->
-    <xacro:macro name="arx5_interfaces_position" params="name">
-        <xacro:property name="prefix" value="${name + '_' if name else ''}"/>
-        <joint name="${prefix}joint1">
-            <command_interface name="position"/>
-            <state_interface name="position"/>
-            <state_interface name="velocity"/>
-            <state_interface name="effort"/>
-        </joint>
-        <joint name="${prefix}joint2">
-            <command_interface name="position"/>
-            <state_interface name="position">
-                <param name="initial_value">0.4</param>
-            </state_interface>
-            <state_interface name="velocity"/>
-            <state_interface name="effort"/>
-        </joint>
-        <joint name="${prefix}joint3">
-            <command_interface name="position"/>
-            <state_interface name="position">
-                <param name="initial_value">0.12</param>
-            </state_interface>
-            <state_interface name="velocity"/>
-            <state_interface name="effort"/>
-        </joint>
-        <joint name="${prefix}joint4">
-            <command_interface name="position"/>
-            <state_interface name="position">
-                <param name="initial_value">0.26</param>
-            </state_interface>
-            <state_interface name="velocity"/>
-            <state_interface name="effort"/>
-        </joint>
-        <joint name="${prefix}joint5">
-            <command_interface name="position"/>
-            <state_interface name="position"/>
-            <state_interface name="velocity"/>
-            <state_interface name="effort"/>
-        </joint>
-        <joint name="${prefix}joint6">
-            <command_interface name="position"/>
-            <state_interface name="position"/>
-            <state_interface name="velocity"/>
-            <state_interface name="effort"/>
-        </joint>
-        <joint name="${prefix}gripper_joint">
-            <command_interface name="position"/>
-            <state_interface name="position"/>
-            <state_interface name="velocity"/>
-            <state_interface name="effort"/>
-        </joint>
-    </xacro:macro>
 </robot>

File: arx5_description/xacro/ros2_control/robot.xacro (robot description, xacro)
@@ -4,8 +4,6 @@
     <xacro:arg name="gazebo" default="false"/>
     <xacro:arg name="type" default="x5"/>
-    <!-- panthera-ht-aligned: full_control (default, OCS2 MIX, recommended) |
-         position (legacy real pos + joint_k/d_gains) | pd_control (alias of position).
-         URDF always declares MIX IFs; mode only affects HI write(). -->
-    <xacro:arg name="control_mode" default="full_control"/>
+    <!-- Arm: full_control only (MIT MIX). Single-arm side via can_interface (can1 left / can3 right). -->
+    <xacro:arg name="can_interface" default="can1"/>
     <link name="world"/>
     <joint name="world_fixed" type="fixed">
@@ -20,6 +18,6 @@
                 <plugin>arx_ros2_control/ArxX5Hardware</plugin>
                 <param name="robot_model">X5</param>
-                <param name="can_interface">can1</param>
-                <param name="control_mode">$(arg control_mode)</param>
+                <param name="can_interface">$(arg can_interface)</param>
+                <param name="control_mode">full_control</param>
                 <param name="joint_k_gains">[80.0, 70.0, 70.0, 30.0, 30.0, 20.0]</param>
                 <param name="joint_d_gains">[2.0, 2.0, 2.0, 1.0, 1.0, 0.7]</param>

File: arx_acone_description/xacro/ros2_control/robot.xacro (robot description, xacro)
@@ -3,12 +3,9 @@
 	<xacro:arg name="ros2_control_hardware_type" default="mock_components"/>
 	<xacro:arg name="gazebo" default="false"/>
-	<!-- panthera-ht-aligned: full_control (default, OCS2 MIX, recommended) |
-	     position (legacy real pos + joint_k/d_gains) | pd_control (alias of position).
-	     URDF always declares MIX IFs; mode only affects HI write(). Stanford HI only. -->
-	<xacro:arg name="control_mode" default="full_control"/>
+	<!-- Arms: full_control only (MIT MIX). Left can1 / right can3. -->
 	<xacro:include filename="$(find arx_acone_description)/xacro/robot.xacro"/>
 	<xacro:include filename="$(find arx5_description)/xacro/ros2_control/interfaces.xacro"/>
 	<xacro:if value="${'$(arg ros2_control_hardware_type)' == 'real'}">
-		<!-- Dual-arm real: Stanford arx5-sdk (same stack as arx5 single-arm). -->
+		<!-- Dual-arm real: Stanford arx5-sdk via arx_ros2_control. -->
 		<ros2_control name="arx_acone_left_system" type="system">
 			<hardware>
@@ -16,5 +13,5 @@
 				<param name="robot_model">X5</param>
 				<param name="can_interface">can1</param>
-				<param name="control_mode">$(arg control_mode)</param>
+				<param name="control_mode">full_control</param>
 				<param name="joint_k_gains">[80.0, 70.0, 70.0, 30.0, 30.0, 20.0]</param>
 				<param name="joint_d_gains">[2.0, 2.0, 2.0, 1.0, 1.0, 0.7]</param>
@@ -27,5 +24,5 @@
 				<param name="robot_model">X5</param>
 				<param name="can_interface">can3</param>
-				<param name="control_mode">$(arg control_mode)</param>
+				<param name="control_mode">full_control</param>
 				<param name="joint_k_gains">[80.0, 70.0, 70.0, 30.0, 30.0, 20.0]</param>
 				<param name="joint_d_gains">[2.0, 2.0, 2.0, 1.0, 1.0, 0.7]</param>

File: arx_lift2s_description/xacro/ros2_control/interfaces.xacro (robot description, xacro)
@@ -2,6 +2,5 @@
 <robot xmlns:xacro="http://www.ros.org/wiki/xacro">
 	<!-- ARX LIFT 2S lift column: MIX IFs so ocs2_wbc can claim.
-	     WBC/full_body 真机推荐 soft_p：只跟 position，忽略 vel/effort/kp/kd。
-	     hybrid（多用分体）：position 斜坡 + 可选 effort→τ_ff；增益 arx_lift.hybrid_kp/kd。 -->
+	     默认 hybrid：pos+vel + HI τ_ff（忽略 effort）；soft_p 仅功能保留。 -->
 	<xacro:macro name="arx_lift2s_base_interfaces">
 		<joint name="lift_joint">

File: arx_lift2s_description/xacro/ros2_control/robot.xacro (robot description, xacro)
@@ -3,6 +3,5 @@
 	<xacro:arg name="ros2_control_hardware_type" default="mock_components"/>
 	<xacro:arg name="gazebo" default="false"/>
-	<!-- Arms: full_control (MIX) | position; live: ros2 param set <arm_node> control_mode ... -->
-	<xacro:arg name="control_mode" default="full_control"/>
+	<!-- Arms: full_control only (MIT MIX). -->
 	<!-- Lift: soft_p|position | hybrid. hybrid 直跟 pos+vel，HI 重力+摩擦（忽略 effort） -->
 	<xacro:arg name="lift_motor_mode" default="hybrid"/>
@@ -11,27 +10,14 @@
 	<xacro:include filename="$(find arx_lift2s_description)/xacro/ros2_control/interfaces.xacro"/>
 	<xacro:if value="${'$(arg ros2_control_hardware_type)' == 'real'}">
-		<!-- Dual arms: Stanford arx5-sdk via arxlift2s ArxX5Hardware (can1 / can3) -->
+		<!-- Dual arms: Stanford arx5-sdk via arx_ros2_control (can1 / can3) -->
 		<ros2_control name="arx_lift2s_left_system" type="system">
 			<hardware>
-				<plugin>arxlift2s_ros2_control/ArxX5Hardware</plugin>
+				<plugin>arx_ros2_control/ArxX5Hardware</plugin>
 				<param name="robot_model">X5</param>
 				<param name="can_interface">can1</param>
-				<param name="control_mode">$(arg control_mode)</param>
-				<!-- Dual gain sets: auto-selected by HI based on control_mode -->
-				<param name="joint_k_gains_full_control">[20.0, 20.0, 20.0, 20.0, 10.0, 10.0]</param>
-				<param name="joint_d_gains_full_control">[0.8, 0.8, 0.8, 0.8, 0.5, 0.5]</param>
-				<param name="joint_k_gains_position">[80.0, 70.0, 70.0, 30.0, 30.0, 20.0]</param>
-				<param name="joint_d_gains_position">[2.0, 2.0, 2.0, 1.0, 1.0, 0.7]</param>
-				<!-- Backward-compatible aliases (seed active gains on startup) -->
-				<!-- position: same defaults as arx-ros2-control -->
-		<xacro:if value="${'$(arg control_mode)' == 'position'}">
-					<param name="joint_k_gains">[80.0, 70.0, 70.0, 30.0, 30.0, 20.0]</param>
-					<param name="joint_d_gains">[2.0, 2.0, 2.0, 1.0, 1.0, 0.7]</param>
-				</xacro:if>
-				<!-- full_control: Lift2S field-tuned MIX defaults -->
-		<xacro:unless value="${'$(arg control_mode)' == 'position'}">
-					<param name="joint_k_gains">[20.0, 20.0, 20.0, 20.0, 10.0, 10.0]</param>
-					<param name="joint_d_gains">[0.8, 0.8, 0.8, 0.8, 0.5, 0.5]</param>
-				</xacro:unless>
+				<param name="control_mode">full_control</param>
+				<!-- Lift2S field-tuned MIX defaults -->
+				<param name="joint_k_gains">[20.0, 20.0, 20.0, 20.0, 10.0, 10.0]</param>
+				<param name="joint_d_gains">[0.8, 0.8, 0.8, 0.8, 0.5, 0.5]</param>
 				<param name="gripper_kp">5.0</param>
 				<param name="gripper_kd">0.2</param>
@@ -46,25 +32,12 @@
 		<ros2_control name="arx_lift2s_right_system" type="system">
 			<hardware>
-				<plugin>arxlift2s_ros2_control/ArxX5Hardware</plugin>
+				<plugin>arx_ros2_control/ArxX5Hardware</plugin>
 				<param name="robot_model">X5</param>
 				<param name="can_interface">can3</param>
-				<param name="control_mode">$(arg control_mode)</param>
-				<!-- Dual gain sets: auto-selected by HI based on control_mode -->
-				<param name="joint_k_gains_full_control">[20.0, 20.0, 20.0, 20.0, 10.0, 10.0]</param>
-				<param name="joint_d_gains_full_control">[0.8, 0.8, 0.8, 0.8, 0.5, 0.5]</param>
-				<param name="joint_k_gains_position">[80.0, 70.0, 70.0, 30.0, 30.0, 20.0]</param>
-				<param name="joint_d_gains_position">[2.0, 2.0, 2.0, 1.0, 1.0, 0.7]</param>
-				<!-- Backward-compatible aliases (seed active gains on startup) -->
-				<xacro:if value="${'$(arg control_mode)' == 'position'}">
-					<param name="joint_k_gains">[80.0, 70.0, 70.0, 30.0, 30.0, 20.0]</param>
-					<param name="joint_d_gains">[2.0, 2.0, 2.0, 1.0, 1.0, 0.7]</param>
-				</xacro:if>
-				<xacro:unless value="${'$(arg control_mode)' == 'position'}">
-					<param name="joint_k_gains">[20.0, 20.0, 20.0, 20.0, 10.0, 10.0]</param>
-					<param name="joint_d_gains">[0.8, 0.8, 0.8, 0.8, 0.5, 0.5]</param>
-				</xacro:unless>
+				<param name="control_mode">full_control</param>
+				<param name="joint_k_gains">[20.0, 20.0, 20.0, 20.0, 10.0, 10.0]</param>
+				<param name="joint_d_gains">[0.8, 0.8, 0.8, 0.8, 0.5, 0.5]</param>
 				<param name="gripper_kp">5.0</param>
 				<param name="gripper_kd">0.2</param>
-				<!-- Ctrl+C: interpolate to home_2 (all-zero) then damping (match left) -->
 				<param name="shutdown_return_home">true</param>
 				<param name="shutdown_home">[0.0, 0.0, 0.0, 0.0, 0.0, 0.0]</param>
@@ -77,5 +50,5 @@
 		<ros2_control name="arx_lift2s_lift_system" type="system">
 			<hardware>
-				<plugin>arxlift2s_ros2_control/ArxLiftHardware</plugin>
+				<plugin>arx_ros2_control/ArxLiftHardware</plugin>
 				<param name="can_name">can5</param>
 				<param name="robot_type">2</param>
