Commit message: Merge pull request #4 from fiveages-sim/feature/lift2s-MIT
Feature/lift2s mit：Add AC One package and Lift2S MIT / hybrid descriptions for OCS2

File: arx5_description/xacro/ros2_control/interfaces.xacro (robot description, xacro)
@@ -4,7 +4,11 @@
         <xacro:property name="prefix" value="${name + '_' if name else ''}"/>
         <xacro:arg name="gazebo" default="false"/>
-        <!-- 关节接口定义 -->
+        <!-- Arm joints: MIX interfaces for full_control (MIT). -->
         <joint name="${prefix}joint1">
             <command_interface name="position"/>
+            <command_interface name="velocity"/>
+            <command_interface name="effort"/>
+            <command_interface name="kp"/>
+            <command_interface name="kd"/>
             <state_interface name="position"/>
             <state_interface name="velocity"/>
@@ -13,4 +17,8 @@
         <joint name="${prefix}joint2">
             <command_interface name="position"/>
+            <command_interface name="velocity"/>
+            <command_interface name="effort"/>
+            <command_interface name="kp"/>
+            <command_interface name="kd"/>
             <state_interface name="position">
                 <param name="initial_value">0.4</param>
@@ -21,4 +29,8 @@
         <joint name="${prefix}joint3">
             <command_interface name="position"/>
+            <command_interface name="velocity"/>
+            <command_interface name="effort"/>
+            <command_interface name="kp"/>
+            <command_interface name="kd"/>
             <state_interface name="position">
                 <param name="initial_value">0.12</param>
@@ -29,4 +41,8 @@
         <joint name="${prefix}joint4">
             <command_interface name="position"/>
+            <command_interface name="velocity"/>
+            <command_interface name="effort"/>
+            <command_interface name="kp"/>
+            <command_interface name="kd"/>
             <state_interface name="position">
                 <param name="initial_value">0.26</param>
@@ -37,4 +53,8 @@
         <joint name="${prefix}joint5">
             <command_interface name="position"/>
+            <command_interface name="velocity"/>
+            <command_interface name="effort"/>
+            <command_interface name="kp"/>
+            <command_interface name="kd"/>
             <state_interface name="position"/>
             <state_interface name="velocity"/>
@@ -43,8 +63,13 @@
         <joint name="${prefix}joint6">
             <command_interface name="position"/>
+            <command_interface name="velocity"/>
+            <command_interface name="effort"/>
+            <command_interface name="kp"/>
+            <command_interface name="kd"/>
             <state_interface name="position"/>
             <state_interface name="velocity"/>
             <state_interface name="effort"/>
         </joint>
+        <!-- Gripper stays position-only (AdaptiveGripperController). -->
         <joint name="${prefix}gripper_joint">
             <command_interface name="position"/>

File: arx5_description/xacro/ros2_control/robot.xacro (robot description, xacro)
@@ -4,4 +4,6 @@
     <xacro:arg name="gazebo" default="false"/>
     <xacro:arg name="type" default="x5"/>
+    <!-- Arm: full_control only (MIT MIX). Single-arm side via can_interface (can1 left / can3 right). -->
+    <xacro:arg name="can_interface" default="can1"/>
     <link name="world"/>
     <joint name="world_fixed" type="fixed">
@@ -16,7 +18,9 @@
                 <plugin>arx_ros2_control/ArxX5Hardware</plugin>
                 <param name="robot_model">X5</param>
-                <param name="can_interface">can1</param>
-                <param name="joint_k_gains">[80.0, 70.0, 70.0, 30.0, 30.0, 20.0]</param>
-                <param name="joint_d_gains">[2.0, 2.0, 2.0, 1.0, 1.0, 0.7]</param>
+                <param name="can_interface">$(arg can_interface)</param>
+                <param name="control_mode">full_control</param>
+                <!-- Align with Lift2S field-tuned MIX defaults -->
+                <param name="joint_k_gains">[20.0, 20.0, 20.0, 20.0, 10.0, 10.0]</param>
+                <param name="joint_d_gains">[0.8, 0.8, 0.8, 0.8, 0.5, 0.5]</param>
                 <!-- 可选：夹爪增益，不写则用默认 -->
                 <!-- <param name="gripper_kp">5.0</param> -->

File: arx_acone_description/xacro/robot.xacro (robot description, xacro)
@@ -1,7 +1,7 @@
-<robot name="arx_lift2s" xmlns:xacro="http://www.ros.org/wiki/xacro">
+<?xml version="1.0"?>
+<robot name="arx_acone" xmlns:xacro="http://www.ros.org/wiki/xacro">
 	<xacro:arg name="type" default="x5"/>
-	<xacro:arg name="enable_wheel_joints" default="false"/>
+	<xacro:arg name="collider" default="simple"/>
 	<xacro:arg name="ros2_control_hardware_type" default="mock_components"/>
-	<xacro:arg name="collider" default="simple"/>
 	<xacro:property name="type_arg" value="$(arg type)"/>
 	<xacro:property name="selected_arm_type" value="x5"/>
@@ -9,13 +9,10 @@
 		<xacro:property name="selected_arm_type" value="r5"/>
 	</xacro:if>
-	<!-- Lift chassis + prismatic lift_joint -->
-	<xacro:include filename="$(find arx_lift2s_description)/xacro/components/chassis.xacro"/>
-	<xacro:chassis enable_wheel_joints="$(arg enable_wheel_joints)" collider="$(arg collider)"/>
-	<joint name="body_joint" type="fixed">
-		<origin xyz="0.13 0.001801 0.0529"/>
-		<parent link="lift_link"/>
+	<!-- Fixed-base dual-arm torso (no lift chassis) -->
+	<link name="base_link"/>
+	<joint name="base_joint" type="fixed">
+		<parent link="base_link"/>
 		<child link="body_link"/>
 	</joint>
-	<!-- AC One torso + dual arms from arx_acone_description -->
 	<xacro:include filename="$(find arx_acone_description)/xacro/components/ac_one.xacro"/>
 	<xacro:ac_one collider="$(arg collider)"/>

File: arx_lift2s_description/xacro/component.xacro (robot description, xacro)
@@ -1,23 +1,13 @@
 <?xml version="1.0" ?>
 <!-- =================================================================================== -->
-<!-- |    Complete Robot Description for ARX LIFT2S                                     | -->
-<!-- |    This file includes the base robot structure and both arms                    | -->
+<!-- |    Component visualization for ARX LIFT2S                                         | -->
 <!-- =================================================================================== -->
-<robot name="AC One" xmlns:xacro="http://www.ros.org/wiki/xacro">
+<robot name="ARX Lift2S" xmlns:xacro="http://www.ros.org/wiki/xacro">
 	<xacro:property name="PI" value="3.1415926535897931"/>
 	<xacro:arg name="type" default="chassis"/>
+	<xacro:arg name="collider" default="simple"/>
 	<xacro:if value="${'$(arg type)' == 'chassis'}">
-		<!-- Include Chassis -->
 		<xacro:include filename="$(find arx_lift2s_description)/xacro/components/chassis.xacro"/>
-		<xacro:chassis enable_wheel_joints="true"/>
-	</xacro:if>
-	<xacro:if value="${'$(arg type)' == 'ac_one'}">
-		<link name="base_link"/>
-		<joint name="base_joint" type="fixed">
-			<parent link="base_link"/>
-			<child link="body_link"/>
-		</joint>
-		<xacro:include filename="$(find arx_lift2s_description)/xacro/components/ac_one.xacro"/>
-		<xacro:ac_one />
+		<xacro:chassis enable_wheel_joints="true" collider="$(arg collider)"/>
 	</xacro:if>
 	<xacro:if value="${'$(arg type)' == 'wheel'}">

File: arx_lift2s_description/xacro/components/chassis.xacro (robot description, xacro)
@@ -2,5 +2,5 @@
 <robot xmlns:xacro="http://www.ros.org/wiki/xacro" name="arx_lift2s_base">
 	<xacro:arg name="robot_name" default="arx_lift2s_base"/>
-	<xacro:macro name="chassis" params="enable_wheel_joints:='false'">
+	<xacro:macro name="chassis" params="enable_wheel_joints:='false' collider:='simple'">
 		<link name="base_link">
 			<inertial>
@@ -15,10 +15,59 @@
 				</geometry>
 			</visual>
-			<collision>
-				<geometry>
-					<mesh filename="file://$(find arx_lift2s_description)/meshes/chassis/base_link.glb"/>
-				</geometry>
-			</collision>
+			<xacro:if value="${collider == 'convex'}">
+				<collision>
+					<geometry>
+						<mesh filename="file://$(find arx_lift2s_description)/meshes/chassis/base_link.glb"/>
+					</geometry>
+				</collision>
+			</xacro:if>
+			<xacro:if value="${collider == 'simple'}">
+				<!-- Main chassis deck (not used in OCS2 arm self-collision pairs) -->
+				<collision name="simple_base_platform">
+					<origin xyz="-0.09 0 0.0" rpy="0 0 0"/>
+					<geometry>
+						<box size="0.52 0.36 0.22"/>
+					</geometry>
+				</collision>
+				<!-- Left / right side skirts -->
+				<collision name="simple_base_left">
+					<origin xyz="0.0 0.24 -0.066" rpy="0 0 0"/>
+					<geometry>
+						<box size="0.44 0.18 0.13"/>
+					</geometry>
+				</collision>
+				<collision name="simple_base_right">
+					<origin xyz="0.0 -0.24 -0.066" rpy="0 0 0"/>
+					<geometry>
+						<box size="0.43 0.18 0.13"/>
+					</geometry>
+				</collision>
+			</xacro:if>
 		</link>
+		<!-- Dedicated mast link so OCS2 pairs hit the lift column, not deck/skirts/rear panel -->
+		<link name="lift_mast_link">
+			<xacro:if value="${collider == 'simple'}">
+				<collision name="simple_lift_mast">
+					<origin xyz="0 0 0" rpy="0 0 0"/>
+					<geometry>
+						<box size="0.13 0.13 0.60"/>
+					</geometry>
+				</collision>
+			</xacro:if>
+			<xacro:if value="${collider == 'convex'}">
+				<!-- approximate mast volume when convex meshes are used on base/lift -->
+				<collision name="simple_lift_mast">
+					<origin xyz="0 0 0" rpy="0 0 0"/>
+					<geometry>
+						<box size="0.13 0.13 0.60"/>
+					</geometry>
+				</collision>
+			</xacro:if>
+		</link>
+		<joint name="lift_mast_joint" type="fixed">
+			<origin xyz="0.01 0 0.50" rpy="0 0 0"/>
+			<parent link="base_link"/>
+			<child link="lift_mast_link"/>
+		</joint>
 		<link name="lift_link">
 			<inertial>
@@ -33,9 +82,20 @@
 				</geometry>
 			</visual>
-			<collision>
-				<geometry>
-					<mesh filename="file://$(find arx_lift2s_description)/meshes/chassis/lift.glb"/>
-				</geometry>
-			</collision>
+			<xacro:if value="${collider == 'convex'}">
+				<collision>
+					<geometry>
+						<mesh filename="file://$(find arx_lift2s_description)/meshes/chassis/lift.glb"/>
+					</geometry>
+				</collision>
+			</xacro:if>
+			<xacro:if value="${collider == 'simple'}">
+				<!-- Carriage plate only (avoid rear upright registering as back screen) -->
+				<collision name="simple_lift_carriage">
+					<origin xyz="-0.015 0 -0.01" rpy="0 0 0"/>
+					<geometry>
+						<box size="0.24 0.16 0.12"/>
+					</geometry>
+				</collision>
+			</xacro:if>
 		</link>
 		<joint name="lift_joint" type="prismatic">
@@ -44,5 +104,7 @@
 			<child link="lift_link"/>
 			<axis xyz="0 0 1"/>
-			<limit lower="0" upper="0.46" effort="400" velocity="0.15"/>
+			<!-- Planning / joint-limit upper aligns with hybrid MIT pack (±12.5 rad / 41.54 ≈ 0.30 m).
+			     soft_p setHeight can still use HI height_span_m≈0.48; OCS2/URDF clamps stay at 0.30. -->
+			<limit lower="0" upper="0.30" effort="400" velocity="0.15"/>
 		</joint>
 		<xacro:property name="wheel_joint_type" value="fixed"/>

File: arx_lift2s_description/xacro/ros2_control/interfaces.xacro (robot description, xacro)
@@ -1,15 +1,17 @@
 <?xml version="1.0"?>
 <robot xmlns:xacro="http://www.ros.org/wiki/xacro">
-    <!-- ARX LIFT 2S 基座关节接口宏定义 -->
-    <xacro:macro name="arx_lift2s_base_interfaces">
-        <!-- 升降关节接口定义 (仅 lift2s 底盘需要) -->
-        <xacro:if value="${selected_base_type == 'lift2s'}">
-            <joint name="lift_joint">
-                <command_interface name="position"/>
-                <state_interface name="position"/>
-                <state_interface name="velocity"/>
-                <state_interface name="effort"/>
-            </joint>
-        </xacro:if>
-    </xacro:macro>
+	<!-- ARX LIFT 2S lift column: MIX IFs so ocs2_wbc can claim.
+	     hybrid（默认）：pos+vel + HI τ_ff（忽略 effort）；soft_p：仅 position。 -->
+	<xacro:macro name="arx_lift2s_base_interfaces">
+		<joint name="lift_joint">
+			<command_interface name="position"/>
+			<command_interface name="velocity"/>
+			<command_interface name="effort"/>
+			<command_interface name="kp"/>
+			<command_interface name="kd"/>
+			<state_interface name="position"/>
+			<state_interface name="velocity"/>
+			<state_interface name="effort"/>
+		</joint>
+	</xacro:macro>
 </robot>

File: arx_lift2s_description/xacro/ros2_control/robot.xacro (robot description, xacro)
@@ -1,65 +1,112 @@
 <?xml version="1.0"?>
 <robot xmlns:xacro="http://www.ros.org/wiki/xacro" name="arx_lift2s">
-    <xacro:arg name="ros2_control_hardware_type" default="mock_components"/>
-    <xacro:arg name="gazebo" default="false"/>
-    <xacro:include filename="$(find arx_lift2s_description)/xacro/robot.xacro"/>
-    <xacro:include filename="$(find arx5_description)/xacro/ros2_control/interfaces.xacro"/>
-    <xacro:include filename="$(find arx_lift2s_description)/xacro/ros2_control/interfaces.xacro"/>
-    <xacro:if value="${'$(arg ros2_control_hardware_type)' == 'real'}">
-        <ros2_control name="arx_lift2s_left_system" type="system">
-            <hardware>
-                <plugin>arx_ros2_control/ArxX5Hardware</plugin>
-                <param name="robot_model">X5</param>
-                <param name="can_interface">can1</param>
-                <param name="joint_k_gains">[80.0, 70.0, 70.0, 30.0, 30.0, 20.0]</param>
-                <param name="joint_d_gains">[2.0, 2.0, 2.0, 1.0, 1.0, 0.7]</param>
-                <!-- 可选：夹爪增益，不写则用默认 -->
-                <!-- <param name="gripper_kp">5.0</param> -->
-                <!-- <param name="gripper_kd">0.2</param> -->
-            </hardware>
-            <xacro:arx5_interfaces name="left"/>
-        </ros2_control>
-        <ros2_control name="arx_lift2s_right_system" type="system">
-            <hardware>
-                <plugin>arx_ros2_control/ArxX5Hardware</plugin>
-                <param name="robot_model">X5</param>
-                <param name="can_interface">can3</param>
-                <param name="joint_k_gains">[80.0, 70.0, 70.0, 30.0, 30.0, 20.0]</param>
-                <param name="joint_d_gains">[2.0, 2.0, 2.0, 1.0, 1.0, 0.7]</param>
-                <!-- 可选：夹爪增益，不写则用默认 -->
-                <!-- <param name="gripper_kp">5.0</param> -->
-                <!-- <param name="gripper_kd">0.2</param> -->
-            </hardware>
-            <xacro:arx5_interfaces name="right"/>
-        </ros2_control>
-    </xacro:if>
-    <xacro:unless value="${'$(arg ros2_control_hardware_type)' == 'real'}">
-        <ros2_control name="arx_lift2s_system" type="system">
-            <hardware>
-                <xacro:if value="${'$(arg ros2_control_hardware_type)' == 'gz'}">
-                    <plugin>gz_ros2_control/GazeboSimSystem</plugin>
-                </xacro:if>
-                <xacro:if value="${'$(arg ros2_control_hardware_type)' == 'mock_components'}">
-                    <plugin>mock_components/GenericSystem</plugin>
-                </xacro:if>
-                <xacro:if value="${'$(arg ros2_control_hardware_type)' == 'isaac'}">
-                    <plugin>topic_based_ros2_control/TopicBasedSystem</plugin>
-                    <param name="joint_commands_topic">/isaac/joint_command</param>
-                    <param name="joint_states_topic">/isaac/joint_states</param>
-                </xacro:if>
-            </hardware>
-            <xacro:if value="${selected_base_type == 'lift2s'}">
-                <xacro:arx_lift2s_base_interfaces/>
-            </xacro:if>
-            <xacro:arx5_interfaces name="left"/>
-            <xacro:arx5_interfaces name="right"/>
-        </ros2_control>
-    </xacro:unless>
-    <xacro:if value="$(arg gazebo)">
-        <gazebo>
-            <plugin filename="gz_ros2_control-system" name="gz_ros2_control::GazeboSimROS2ControlPlugin">
-                <parameters>$(find arx_lift2s_description)/config/ros2_control/ros2_controllers.yaml</parameters>
-            </plugin>
-        </gazebo>
-    </xacro:if>
+	<xacro:arg name="ros2_control_hardware_type" default="mock_components"/>
+	<xacro:arg name="gazebo" default="false"/>
+	<!-- Arms: full_control only (MIT MIX). -->
+	<!-- Lift: soft_p|position | hybrid. hybrid 直跟 pos+vel，HI 重力+摩擦（忽略 effort） -->
+	<xacro:arg name="lift_motor_mode" default="hybrid"/>
+	<xacro:include filename="$(find arx_lift2s_description)/xacro/robot.xacro"/>
+	<xacro:include filename="$(find arx5_description)/xacro/ros2_control/interfaces.xacro"/>
+	<xacro:include filename="$(find arx_lift2s_description)/xacro/ros2_control/interfaces.xacro"/>
+	<xacro:if value="${'$(arg ros2_control_hardware_type)' == 'real'}">
+		<!-- Dual arms: Stanford arx5-sdk via arx_ros2_control (can1 / can3) -->
+		<ros2_control name="arx_lift2s_left_system" type="system">
+			<hardware>
+				<plugin>arx_ros2_control/ArxX5Hardware</plugin>
+				<param name="robot_model">X5</param>
+				<param name="can_interface">can1</param>
+				<param name="control_mode">full_control</param>
+				<!-- Lift2S field-tuned MIX defaults -->
+				<param name="joint_k_gains">[20.0, 20.0, 20.0, 20.0, 10.0, 10.0]</param>
+				<param name="joint_d_gains">[0.8, 0.8, 0.8, 0.8, 0.5, 0.5]</param>
+				<param name="gripper_kp">5.0</param>
+				<param name="gripper_kd">0.2</param>
+				<!-- Ctrl+C: interpolate to home_2 (all-zero) then damping -->
+				<param name="shutdown_return_home">true</param>
+				<param name="shutdown_home">[0.0, 0.0, 0.0, 0.0, 0.0, 0.0]</param>
+				<param name="shutdown_home_velocity">0.3</param>
+				<param name="shutdown_home_timeout">2.0</param>
+			</hardware>
+			<xacro:arx5_interfaces name="left"/>
+		</ros2_control>
+		<ros2_control name="arx_lift2s_right_system" type="system">
+			<hardware>
+				<plugin>arx_ros2_control/ArxX5Hardware</plugin>
+				<param name="robot_model">X5</param>
+				<param name="can_interface">can3</param>
+				<param name="control_mode">full_control</param>
+				<param name="joint_k_gains">[20.0, 20.0, 20.0, 20.0, 10.0, 10.0]</param>
+				<param name="joint_d_gains">[0.8, 0.8, 0.8, 0.8, 0.5, 0.5]</param>
+				<param name="gripper_kp">5.0</param>
+				<param name="gripper_kd">0.2</param>
+				<param name="shutdown_return_home">true</param>
+				<param name="shutdown_home">[0.0, 0.0, 0.0, 0.0, 0.0, 0.0]</param>
+				<param name="shutdown_home_velocity">0.3</param>
+				<param name="shutdown_home_timeout">2.0</param>
+			</hardware>
+			<xacro:arx5_interfaces name="right"/>
+		</ros2_control>
+		<!-- Lift column: soft_p | hybrid (live: arx_lift.motor_mode / soft_p_kp / hybrid_kp|kd) -->
+		<ros2_control name="arx_lift2s_lift_system" type="system">
+			<hardware>
+				<plugin>arx_ros2_control/ArxLiftHardware</plugin>
+				<param name="can_name">can5</param>
+				<param name="robot_type">2</param>
+				<!-- soft_p|position: 仅跟踪 position；hybrid: 直跟 pos+vel + HI 重力/摩擦（忽略 effort） -->
+				<param name="lift_motor_mode">$(arg lift_motor_mode)</param>
+				<!-- Soft-P (setHeight/loop); live: arx_lift.soft_p_kp -->
+				<param name="soft_p_kp">50.0</param>
+				<param name="lift_max_vel">0.20</param>
+				<!-- Hybrid MIT; live: arx_lift.hybrid_kp / hybrid_kd / gravity_* / coulomb_* / friction_vel_eps_mps -->
+				<param name="hybrid_kp">5.0</param>
+				<param name="hybrid_kd">2.0</param>
+				<!-- τ_ff = gravity - coulomb * sign(v_cmd); v_cmd 来自上层 velocity [m/s] -->
+				<param name="gravity_compensation_torque">-1.01</param>
+				<param name="coulomb_friction_torque">0.32</param>
+				<param name="friction_vel_eps_mps">0.01</param>
+				<param name="lift_max_torque">15.0</param>
+				<!-- cmd_ramp_vel: soft_p 跟踪与关机插值；hybrid 跟踪不用 -->
+				<param name="cmd_ramp_vel">0.12</param>
+				<param name="max_height_m">0.48</param>
+				<param name="height_span_m">0.48</param>
+				<!-- SDK motor rad / meter -->
+				<param name="height_rad_per_meter">41.54</param>
+				<param name="sdk_max_rad">20.0</param>
+				<!-- Ctrl+C: ramp to home_2 height (0) then soft-stop -->
+				<param name="shutdown_return_home">true</param>
+				<param name="shutdown_height_m">0.0</param>
+				<param name="shutdown_home_velocity">0.10</param>
+				<param name="shutdown_home_timeout">2.0</param>
+			</hardware>
+			<xacro:arx_lift2s_base_interfaces/>
+		</ros2_control>
+	</xacro:if>
+	<xacro:unless value="${'$(arg ros2_control_hardware_type)' == 'real'}">
+		<ros2_control name="arx_lift2s_system" type="system">
+			<hardware>
+				<xacro:if value="${'$(arg ros2_control_hardware_type)' == 'gz'}">
+					<plugin>gz_ros2_control/GazeboSimSystem</plugin>
+				</xacro:if>
+				<xacro:if value="${'$(arg ros2_control_hardware_type)' == 'mock_components'}">
+					<plugin>mock_components/GenericSystem</plugin>
+				</xacro:if>
+				<xacro:if value="${'$(arg ros2_control_hardware_type)' == 'isaac'}">
+					<plugin>topic_based_ros2_control/TopicBasedSystem</plugin>
+					<param name="joint_commands_topic">/isaac/joint_command</param>
+					<param name="joint_states_topic">/isaac/joint_states</param>
+				</xacro:if>
+			</hardware>
+			<xacro:arx_lift2s_base_interfaces/>
+			<!-- Sim: MIX arm IFs to match real Stanford HI / full_control -->
+			<xacro:arx5_interfaces name="left"/>
+			<xacro:arx5_interfaces name="right"/>
+		</ros2_control>
+	</xacro:unless>
+	<xacro:if value="$(arg gazebo)">
+		<gazebo>
+			<plugin filename="gz_ros2_control-system" name="gz_ros2_control::GazeboSimROS2ControlPlugin">
+				<parameters>$(find arx_lift2s_description)/config/ros2_control/ros2_controllers.yaml</parameters>
+			</plugin>
+		</gazebo>
+	</xacro:if>
 </robot>
