Commit message: fix fullbody mode

File: arx5_description/xacro/ros2_control/interfaces.xacro (robot description, xacro)
@@ -1,80 +1,41 @@
 <?xml version="1.0"?>
 <robot xmlns:xacro="http://www.ros.org/wiki/xacro">
-    <xacro:macro name="arx5_interfaces" params="name">
+    <!-- iface_mode: mix = pos/vel/effort (real / mock / gz); position = pos only (Isaac). -->
+    <xacro:macro name="arx5_arm_joint" params="jname iface_mode initial:=''">
+        <joint name="${jname}">
+            <command_interface name="position"/>
+            <xacro:if value="${iface_mode == 'mix'}">
+                <command_interface name="velocity"/>
+                <command_interface name="effort"/>
+            </xacro:if>
+            <state_interface name="position">
+                <xacro:unless value="${initial == ''}">
+                    <param name="initial_value">${initial}</param>
+                </xacro:unless>
+            </state_interface>
+            <xacro:if value="${iface_mode == 'mix'}">
+                <state_interface name="velocity"/>
+                <state_interface name="effort"/>
+            </xacro:if>
+        </joint>
+    </xacro:macro>
+    <xacro:macro name="arx5_interfaces" params="name iface_mode:=mix">
         <xacro:property name="prefix" value="${name + '_' if name else ''}"/>
         <xacro:arg name="gazebo" default="false"/>
-        <!-- Arm joints: MIX interfaces for full_control (MIT). -->
-        <joint name="${prefix}joint1">
-            <command_interface name="position"/>
-            <command_interface name="velocity"/>
-            <command_interface name="effort"/>
-            <command_interface name="kp"/>
-            <command_interface name="kd"/>
-            <state_interface name="position"/>
-            <state_interface name="velocity"/>
-            <state_interface name="effort"/>
-        </joint>
-        <joint name="${prefix}joint2">
-            <command_interface name="position"/>
-            <command_interface name="velocity"/>
-            <command_interface name="effort"/>
-            <command_interface name="kp"/>
-            <command_interface name="kd"/>
-            <state_interface name="position">
-                <param name="initial_value">0.4</param>
-            </state_interface>
-            <state_interface name="velocity"/>
-            <state_interface name="effort"/>
-        </joint>
-        <joint name="${prefix}joint3">
-            <command_interface name="position"/>
-            <command_interface name="velocity"/>
-            <command_interface name="effort"/>
-            <command_interface name="kp"/>
-            <command_interface name="kd"/>
-            <state_interface name="position">
-                <param name="initial_value">0.12</param>
-            </state_interface>
-            <state_interface name="velocity"/>
-            <state_interface name="effort"/>
-        </joint>
-        <joint name="${prefix}joint4">
-            <command_interface name="position"/>
-            <command_interface name="velocity"/>
-            <command_interface name="effort"/>
-            <command_interface name="kp"/>
-            <command_interface name="kd"/>
-            <state_interface name="position">
-                <param name="initial_value">0.26</param>
-            </state_interface>
-            <state_interface name="velocity"/>
-            <state_interface name="effort"/>
-        </joint>
-        <joint name="${prefix}joint5">
-            <command_interface name="position"/>
-            <command_interface name="velocity"/>
-            <command_interface name="effort"/>
-            <command_interface name="kp"/>
-            <command_interface name="kd"/>
-            <state_interface name="position"/>
-            <state_interface name="velocity"/>
-            <state_interface name="effort"/>
-        </joint>
-        <joint name="${prefix}joint6">
-            <command_interface name="position"/>
-            <command_interface name="velocity"/>
-            <command_interface name="effort"/>
-            <command_interface name="kp"/>
-            <command_interface name="kd"/>
-            <state_interface name="position"/>
-            <state_interface name="velocity"/>
-            <state_interface name="effort"/>
-        </joint>
-        <!-- Gripper stays position-only (AdaptiveGripperController). -->
+        <!-- Arm: mix → full_control MIT; position → Isaac TopicBasedSystem. Gains: HI joint_k/d_gains. -->
+        <xacro:arx5_arm_joint jname="${prefix}joint1" iface_mode="${iface_mode}"/>
+        <xacro:arx5_arm_joint jname="${prefix}joint2" iface_mode="${iface_mode}" initial="0.4"/>
+        <xacro:arx5_arm_joint jname="${prefix}joint3" iface_mode="${iface_mode}" initial="0.12"/>
+        <xacro:arx5_arm_joint jname="${prefix}joint4" iface_mode="${iface_mode}" initial="0.26"/>
+        <xacro:arx5_arm_joint jname="${prefix}joint5" iface_mode="${iface_mode}"/>
+        <xacro:arx5_arm_joint jname="${prefix}joint6" iface_mode="${iface_mode}"/>
+        <!-- Gripper: AdaptiveGripperController (effort state only when mix). -->
         <joint name="${prefix}gripper_joint">
             <command_interface name="position"/>
             <state_interface name="position"/>
-            <state_interface name="velocity"/>
-            <state_interface name="effort"/>
+            <xacro:if value="${iface_mode == 'mix'}">
+                <state_interface name="velocity"/>
+                <state_interface name="effort"/>
+            </xacro:if>
         </joint>
         <xacro:if value="$(arg gazebo)">

File: arx_lift2s_description/xacro/components/chassis.xacro (robot description, xacro)
@@ -2,4 +2,6 @@
 <robot xmlns:xacro="http://www.ros.org/wiki/xacro" name="arx_lift2s_base">
 	<xacro:arg name="robot_name" default="arx_lift2s_base"/>
+	<!-- Injected true by robot_common_launch for OCS2 planning URDF; viz / ros2_control keep false -->
+	<xacro:arg name="eef_fixed_joints" default="false"/>
 	<xacro:macro name="chassis" params="enable_wheel_joints:='false' collider:='simple'">
 		<link name="base_link">
@@ -99,4 +101,9 @@
 			</xacro:if>
 		</link>
+		<!-- Same pattern as m6_ccs joint4 + eef_fixed_joints:
+		     planning URDF → 0.30 m (hybrid MIT pack ±12.5 rad / 41.54);
+		     viz / ros2_control → 0.48 m (HI height_span_m / soft_p setHeight). -->
+		<xacro:property name="lift_joint_upper"
+										value="${0.30 if '$(arg eef_fixed_joints)' == 'true' else 0.48}"/>
 		<joint name="lift_joint" type="prismatic">
 			<origin xyz="0.040103 0.0007607 0.221608"/>
@@ -104,7 +111,5 @@
 			<child link="lift_link"/>
 			<axis xyz="0 0 1"/>
-			<!-- Planning / joint-limit upper aligns with hybrid MIT pack (±12.5 rad / 41.54 ≈ 0.30 m).
-			     soft_p setHeight can still use HI height_span_m≈0.48; OCS2/URDF clamps stay at 0.30. -->
-			<limit lower="0" upper="0.30" effort="400" velocity="0.15"/>
+			<limit lower="0" upper="${lift_joint_upper}" effort="400" velocity="0.15"/>
 		</joint>
 		<xacro:property name="wheel_joint_type" value="fixed"/>

File: arx_lift2s_description/xacro/robot.xacro (robot description, xacro)
@@ -4,4 +4,7 @@
 	<xacro:arg name="ros2_control_hardware_type" default="mock_components"/>
 	<xacro:arg name="collider" default="simple"/>
+	<!-- Declared here so planning mappings (eef_fixed_joints:=true) reach chassis.xacro;
+	     same hook m6_ccs uses to tighten joint4 on planning URDF. -->
+	<xacro:arg name="eef_fixed_joints" default="false"/>
 	<xacro:property name="type_arg" value="$(arg type)"/>
 	<xacro:property name="selected_arm_type" value="x5"/>

File: arx_lift2s_description/xacro/ros2_control/interfaces.xacro (robot description, xacro)
@@ -1,16 +1,19 @@
 <?xml version="1.0"?>
 <robot xmlns:xacro="http://www.ros.org/wiki/xacro">
-	<!-- ARX LIFT 2S lift column: MIX IFs so ocs2_wbc can claim.
-	     hybrid（默认）：pos+vel + HI τ_ff（忽略 effort）；soft_p：仅 position。 -->
-	<xacro:macro name="arx_lift2s_base_interfaces">
+	<!-- iface_mode: mix = pos/vel/effort（真机 / mock / gz）；position = 仅 position（Isaac）。
+	     hybrid：pos+vel + HI τ_ff（忽略 effort）；soft_p：仅 position。
+	     Gains: arx_lift.hybrid_kp/kd / soft_p_kp（无 kp/kd command IF）。 -->
+	<xacro:macro name="arx_lift2s_base_interfaces" params="iface_mode:=mix">
 		<joint name="lift_joint">
 			<command_interface name="position"/>
-			<command_interface name="velocity"/>
-			<command_interface name="effort"/>
-			<command_interface name="kp"/>
-			<command_interface name="kd"/>
+			<xacro:if value="${iface_mode == 'mix'}">
+				<command_interface name="velocity"/>
+				<command_interface name="effort"/>
+			</xacro:if>
 			<state_interface name="position"/>
-			<state_interface name="velocity"/>
-			<state_interface name="effort"/>
+			<xacro:if value="${iface_mode == 'mix'}">
+				<state_interface name="velocity"/>
+				<state_interface name="effort"/>
+			</xacro:if>
 		</joint>
 	</xacro:macro>

File: arx_lift2s_description/xacro/ros2_control/robot.xacro (robot description, xacro)
@@ -6,4 +6,6 @@
 	<!-- Lift: soft_p|position | hybrid. hybrid 直跟 pos+vel，HI 重力+摩擦（忽略 effort） -->
 	<xacro:arg name="lift_motor_mode" default="hybrid"/>
+	<!-- Lift HI：可选订阅 /cmd_vel → setChassisCmd（默认关，避免与 WBC 底盘规划抢指令） -->
+	<xacro:arg name="enable_chassis_cmd_vel" default="false"/>
 	<xacro:include filename="$(find arx_lift2s_description)/xacro/robot.xacro"/>
 	<xacro:include filename="$(find arx5_description)/xacro/ros2_control/interfaces.xacro"/>
@@ -78,8 +80,15 @@
 				<param name="shutdown_home_velocity">0.10</param>
 				<param name="shutdown_home_timeout">2.0</param>
+				<!-- 可选：/cmd_vel → 底盘 setChassisCmd；默认关 -->
+				<param name="enable_chassis_cmd_vel">$(arg enable_chassis_cmd_vel)</param>
+				<param name="chassis_cmd_vel_topic">/cmd_vel</param>
+				<param name="chassis_cmd_timeout">0.3</param>
 			</hardware>
 			<xacro:arx_lift2s_base_interfaces/>
 		</ros2_control>
 	</xacro:if>
+	<!-- Isaac: position-only（TopicBasedSystem / 仿真对 effort、velocity 支持差）；mock/gz 仍 MIX -->
+	<xacro:property name="sim_iface_mode"
+		value="${'position' if '$(arg ros2_control_hardware_type)' == 'isaac' else 'mix'}"/>
 	<xacro:unless value="${'$(arg ros2_control_hardware_type)' == 'real'}">
 		<ros2_control name="arx_lift2s_system" type="system">
@@ -97,8 +106,7 @@
 				</xacro:if>
 			</hardware>
-			<xacro:arx_lift2s_base_interfaces/>
-			<!-- Sim: MIX arm IFs to match real Stanford HI / full_control -->
-			<xacro:arx5_interfaces name="left"/>
-			<xacro:arx5_interfaces name="right"/>
+			<xacro:arx_lift2s_base_interfaces iface_mode="${sim_iface_mode}"/>
+			<xacro:arx5_interfaces name="left" iface_mode="${sim_iface_mode}"/>
+			<xacro:arx5_interfaces name="right" iface_mode="${sim_iface_mode}"/>
 		</ros2_control>
 	</xacro:unless>
