Commit message: AC_One简单碰撞体在xacro中已配置完成

File: arx5_description/xacro/R5.xacro (robot description, xacro)
@@ -1,46 +1,57 @@
 <?xml version="1.0"?>
 <robot xmlns:xacro="http://www.ros.org/wiki/xacro">
-	<xacro:macro name="R5" params="name camera:=d405 style:=default">
-		<xacro:property name="prefix" value="${name + '_' if name else ''}"/>
-		<link name="${prefix}base_link">
-			<inertial>
-				<origin xyz="-0.00013359 6.672E-05 0.031672"/>
-				<mass value="0.42272"/>
-				<inertia
-						ixx="0.00019"
-						ixy="0.00000"
-						ixz="0.00000"
-						iyy="0.00019"
-						iyz="0.00000"
-						izz="0.00020"/>
-			</inertial>
-			<visual>
-				<geometry>
-					<mesh filename="file://$(find arx5_description)/meshes/r5/base_link.obj"/>
-				</geometry>
-			</visual>
-			<collision>
-				<geometry>
-					<mesh filename="file://$(find arx5_description)/meshes/r5/base_link.obj"/>
-				</geometry>
-			</collision>
-		</link>
-		<link name="${prefix}link1">
-			<inertial>
-				<origin xyz="0.0050395 -0.0077407 0.020897"/>
-				<mass value="0.096804"/>
-				<inertia
-						ixx="0.00011"
-						ixy="-0.00001"
-						ixz="0.00001"
-						iyy="0.00005"
-						iyz="-0.00001"
-						izz="0.00010"/>
-			</inertial>
-			<visual>
-				<geometry>
-					<mesh filename="file://$(find arx5_description)/meshes/r5/link1.obj"/>
-				</geometry>
-			</visual>
+    <xacro:property name="PI" value="3.1415926535897931"/>
+    <xacro:macro name="R5" params="name camera:=d405 style:=default collider:=convex">
+        <xacro:property name="prefix" value="${name + '_' if name else ''}"/>
+        <link name="${prefix}base_link">
+            <inertial>
+                <origin xyz="-0.00013359 6.672E-05 0.031672"/>
+                <mass value="0.42272"/>
+                <inertia
+                        ixx="0.00019"
+                        ixy="0.00000"
+                        ixz="0.00000"
+                        iyy="0.00019"
+                        iyz="0.00000"
+                        izz="0.00020"/>
+            </inertial>
+            <visual>
+                <geometry>
+                    <mesh filename="file://$(find arx5_description)/meshes/r5/base_link.obj"/>
+                </geometry>
+            </visual>
+            <xacro:if value="${collider == 'convex'}">
+                <collision>
+                    <geometry>
+                        <mesh filename="file://$(find arx5_description)/meshes/r5/base_link.obj"/>
+                    </geometry>
+                </collision>
+            </xacro:if>
+            <xacro:if value="${collider == 'simple'}">
+                <collision>
+                    <origin xyz="0 0 0.0312"/>
+                    <geometry>
+                        <cylinder length="0.0625" radius="0.0305"/>
+                    </geometry>
+                </collision>
+            </xacro:if>
+        </link>
+        <link name="${prefix}link1">
+            <inertial>
+                <origin xyz="0.0050395 -0.0077407 0.020897"/>
+                <mass value="0.096804"/>
+                <inertia
+                        ixx="0.00011"
+                        ixy="-0.00001"
+                        ixz="0.00001"
+                        iyy="0.00005"
+                        iyz="-0.00001"
+                        izz="0.00010"/>
+            </inertial>
+            <visual>
+                <geometry>
+                    <mesh filename="file://$(find arx5_description)/meshes/r5/link1.obj"/>
+                </geometry>
+            </visual>
 			<collision>
 				<geometry>
@@ -48,303 +59,463 @@
 				</geometry>
 			</collision>
-		</link>
-		<joint name="${prefix}joint1" type="revolute">
-			<origin xyz="0 0 0.0565"/>
-			<parent link="${prefix}base_link"/>
-			<child link="${prefix}link1"/>
-			<axis xyz="0 0 1"/>
-			<limit lower="-2.618" upper="2.168" effort="100" velocity="5"/>
-		</joint>
-		<link name="${prefix}link2">
-			<inertial>
-				<origin xyz="-0.12992 -0.0011822 -2.6366E-05"/>
-				<mass value="1.1988"/>
-				<inertia
-						ixx="0.00065"
-						ixy="0.00008"
-						ixz="0.00000"
-						iyy="0.01647"
-						iyz="0.00000"
-						izz="0.01646"/>
-			</inertial>
-			<visual>
-				<geometry>
-					<xacro:if value="${style == 'agilex'}">
-						<mesh filename="file://$(find arx5_description)/meshes/r5/link2_agilex.obj"/>
-					</xacro:if>
-					<xacro:if value="${style == 'default'}">
-						<mesh filename="file://$(find arx5_description)/meshes/r5/link2.obj"/>
-					</xacro:if>
-				</geometry>
-			</visual>
-			<collision>
-				<geometry>
-					<mesh filename="file://$(find arx5_description)/meshes/r5/link2.obj"/>
-				</geometry>
-			</collision>
-		</link>
-		<joint name="${prefix}joint2" type="revolute">
-			<origin xyz="0.02 0 0.047"/>
-			<parent link="${prefix}link1"/>
-			<child link="${prefix}link2"/>
-			<axis xyz="0 1 0"/>
-			<limit lower="0" upper="3.66" effort="100" velocity="5"/>
-		</joint>
-		<link name="${prefix}link3">
-			<inertial>
-				<origin xyz="0.16181 0.0011723 -0.05455"/>
-				<mass value="0.84082"/>
-				<inertia
-						ixx="0.00082"
-						ixy="0.00008"
-						ixz="-0.00074"
-						iyy="0.00849"
-						iyz="0.00001"
-						izz="0.00834"/>
-			</inertial>
-			<visual>
-				<geometry>
-					<xacro:if value="${style == 'agilex'}">
-						<mesh filename="file://$(find arx5_description)/meshes/r5/link3_agilex.obj"/>
-					</xacro:if>
-					<xacro:if value="${style == 'default'}">
-						<mesh filename="file://$(find arx5_description)/meshes/r5/link3.obj"/>
-					</xacro:if>
-				</geometry>
-			</visual>
-			<collision>
-				<geometry>
-					<mesh filename="file://$(find arx5_description)/meshes/r5/link3.obj"/>
-				</geometry>
-			</collision>
-		</link>
-		<joint name="${prefix}joint3" type="revolute">
-			<origin xyz="-0.264 0 0" rpy="-3.1416 0 0"/>
-			<parent link="${prefix}link2"/>
-			<child link="${prefix}link3"/>
-			<axis xyz="0 1 0"/>
-			<limit lower="0" upper="3.14" effort="100" velocity="5"/>
-		</joint>
-		<link name="${prefix}link4">
-			<inertial>
-				<origin xyz="0.041751 0.0054236 -0.03337"/>
-				<mass value="0.12432"/>
-				<inertia
-						ixx="0.00022"
-						ixy="-0.00002"
-						ixz="-0.00009"
-						iyy="0.00025"
-						iyz="0.00002"
-						izz="0.00017"/>
-			</inertial>
-			<visual>
-				<geometry>
-					<mesh filename="file://$(find arx5_description)/meshes/r5/link4.obj"/>
-				</geometry>
-			</visual>
-			<collision>
-				<geometry>
-					<mesh filename="file://$(find arx5_description)/meshes/r5/link4.obj"/>
-				</geometry>
-			</collision>
-		</link>
-		<joint name="${prefix}joint4" type="revolute">
-			<origin xyz="0.245 -5E-05 -0.06"/>
-			<parent link="${prefix}link3"/>
-			<child link="${prefix}link4"/>
-			<axis xyz="0 1 0"/>
-			<limit lower="-1.57" upper="1.57" effort="100" velocity="5"/>
-		</joint>
-		<link name="${prefix}link5">
-			<inertial>
-				<origin xyz="-8.3435E-05 -1.5428E-05 0.052216"/>
-				<mass value="0.63601"/>
-				<inertia
-						ixx="0.00084"
-						ixy="0.00000"
-						ixz="0.00007"
-						iyy="0.00082"
-						iyz="0.00000"
-						izz="0.00026"/>
-			</inertial>
-			<visual>
-				<geometry>
-					<mesh filename="file://$(find arx5_description)/meshes/r5/link5.obj"/>
-				</geometry>
-			</visual>
-			<collision>
-				<geometry>
-					<mesh filename="file://$(find arx5_description)/meshes/r5/link5.obj"/>
-				</geometry>
-			</collision>
-		</link>
-		<joint name="${prefix}joint5" type="revolute">
-			<origin xyz="0.0702 5E-05 -0.083391"/>
-			<parent link="${prefix}link4"/>
-			<child link="${prefix}link5"/>
-			<axis xyz="0 0 1"/>
-			<limit lower="-1.57" upper="1.57" effort="100" velocity="5"/>
-		</joint>
-		<link name="${prefix}link6">
-			<inertial>
-				<origin xyz="0.041697 2.4368E-05 0.00014464"/>
-				<mass value="0.44089"/>
-				<inertia
-						ixx="0.00038"
-						ixy="0.00000"
-						ixz="0.00000"
-						iyy="0.00028"
-						iyz="0.00000"
-						izz="0.00050"/>
-			</inertial>
-			<visual>
-				<geometry>
-					<mesh filename="file://$(find arx5_description)/meshes/r5/link6.obj"/>
-				</geometry>
-			</visual>
-			<collision>
-				<geometry>
-					<mesh filename="file://$(find arx5_description)/meshes/r5/link6.obj"/>
-				</geometry>
-			</collision>
-		</link>
-		<joint name="${prefix}joint6" type="revolute">
-			<origin xyz="0.025286 0 0.083391" rpy="3.1416 0 0"/>
-			<parent link="${prefix}link5"/>
-			<child link="${prefix}link6"/>
-			<axis xyz="1 0 0"/>
-			<limit lower="-1.57" upper="1.57" effort="100" velocity="5"/>
-		</joint>
-		<link name="${prefix}link7">
-			<inertial>
-				<origin xyz="-0.00035522 -0.007827 -0.0029883"/>
-				<mass value="0.064798"/>
-				<inertia
-						ixx="0.00002"
-						ixy="0.00000"
-						ixz="0.00000"
-						iyy="0.00003"
-						iyz="0.00000"
-						izz="0.00003"/>
-			</inertial>
-			<visual>
-				<geometry>
-					<mesh filename="file://$(find arx5_description)/meshes/r5/link7.obj"/>
-				</geometry>
-			</visual>
-			<collision>
-				<geometry>
-					<mesh filename="file://$(find arx5_description)/meshes/r5/link7.obj"/>
-				</geometry>
-			</collision>
-		</link>
-		<joint name="${prefix}gripper_joint" type="prismatic">
-			<origin xyz="0.08657 0.024896 -0.0002436"/>
-			<parent link="${prefix}link6"/>
-			<child link="${prefix}link7"/>
-			<axis xyz="0 1 0"/>
-			<limit lower="0" upper="0.044" effort="100" velocity="5"/>
-		</joint>
-		<link name="${prefix}link8">
-			<inertial>
-				<origin xyz="-0.000355223470270755 0.00782768751820277 0.00242005642879778"/>
-				<mass value="0.0647981725781684"/>
-				<inertia
-						ixx="0.00002"
-						ixy="0.00000"
-						ixz="0.00000"
-						iyy="0.00003"
-						iyz="0.00000"
-						izz="0.00003"/>
-			</inertial>
-			<visual>
-				<geometry>
-					<mesh filename="file://$(find arx5_description)/meshes/r5/link8.obj"/>
-				</geometry>
-			</visual>
-			<collision>
-				<geometry>
-					<mesh filename="file://$(find arx5_description)/meshes/r5/link8.obj"/>
-				</geometry>
-			</collision>
-		</link>
-		<joint name="${prefix}joint8" type="prismatic">
-			<origin xyz="0.08657 -0.0249 -0.00024366"/>
-			<parent link="${prefix}link6"/>
-			<child link="${prefix}link8"/>
-			<axis xyz="0 -1 0"/>
-			<limit lower="0" upper="0.044" effort="100" velocity="5"/>
-			<mimic joint="${prefix}gripper_joint" multiplier="1" offset="0"/>
-		</joint>
-		<link name="${prefix}gripper_center"/>
-		<joint name="${prefix}gripper_center_fixed" type="fixed">
-			<parent link="${prefix}link6"/>
-			<child link="${prefix}gripper_center"/>
-			<origin xyz="0.08657 0 0"/>
-		</joint>
-		<link name="${prefix}left_pad"/>
-		<joint name="${prefix}left_pad_joint" type="fixed">
-			<parent link="${prefix}link7"/>
-			<child link="${prefix}left_pad"/>
-			<origin xyz="0.05843 -0.0249 0"/>
-		</joint>
-		<link name="${prefix}right_pad"/>
-		<joint name="${prefix}right_pad_joint" type="fixed">
-			<parent link="${prefix}link8"/>
-			<child link="${prefix}right_pad"/>
-			<origin xyz="0.05843 0.0249 0"/>
-		</joint>
-		<xacro:if value="${camera == 'd405'}">
-			<link name="${prefix}camera_support">
-				<visual>
+        </link>
+        <joint name="${prefix}joint1" type="revolute">
+            <origin xyz="0 0 0.0565"/>
+            <parent link="${prefix}base_link"/>
+            <child link="${prefix}link1"/>
+            <axis xyz="0 0 1"/>
+            <limit lower="-2.618" upper="2.168" effort="100" velocity="5"/>
+        </joint>
+        <link name="${prefix}link2">
+            <inertial>
+                <origin xyz="-0.12992 -0.0011822 -2.6366E-05"/>
+                <mass value="1.1988"/>
+                <inertia
+                        ixx="0.00065"
+                        ixy="0.00008"
+                        ixz="0.00000"
+                        iyy="0.01647"
+                        iyz="0.00000"
+                        izz="0.01646"/>
+            </inertial>
+            <visual>
+                <geometry>
+                    <xacro:if value="${style == 'agilex'}">
+                        <mesh filename="file://$(find arx5_description)/meshes/r5/link2_agilex.obj"/>
+                    </xacro:if>
+                    <xacro:if value="${style == 'default'}">
+                        <mesh filename="file://$(find arx5_description)/meshes/r5/link2.obj"/>
+                    </xacro:if>
+                </geometry>
+            </visual>
+            <xacro:if value="${collider == 'convex'}">
+                <collision>
+                    <geometry>
+                        <mesh filename="file://$(find arx5_description)/meshes/r5/link2.obj"/>
+                    </geometry>
+                </collision>
+            </xacro:if>
+			<xacro:if value="${collider == 'simple'}">
+				<collision name="simple_link2_1">
+					<origin xyz="0 0.003 0" rpy="${PI/2} 0 0"/>
 					<geometry>
-						<mesh filename="file://$(find arx5_description)/meshes/camera_stand/stand_d405.obj"/>
+						<cylinder length="0.0665" radius="0.03"/>
 					</geometry>
-				</visual>
-			</link>
-			<joint name="${prefix}camera_support_fixed" type="fixed">
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
File: arx5_description/xacro/X5.xacro (robot description, xacro)
@@ -317,4 +317,11 @@
             </xacro:if>
             <xacro:if value="${collider == 'simple'}">
+                <collision name="simple_link7">
+                    <origin xyz="0.0262 0 0.0002" rpy="0 0 0"/>
+                    <geometry>
+                        <box size="0.08 0.04 0.0640"/>
+                    </geometry>
+                </collision>
+            </xacro:if>
         </link>
         <joint name="${prefix}gripper_joint" type="prismatic">
@@ -342,9 +349,19 @@
                 </geometry>
             </visual>
-            <collision>
-                <geometry>
-                    <mesh filename="file://$(find arx5_description)/meshes/x5/link8.obj"/>
-                </geometry>
-            </collision>
+            <xacro:if value="${collider == 'convex'}">
+                <collision>
+                    <geometry>
+                        <mesh filename="file://$(find arx5_description)/meshes/x5/link8.obj"/>
+                    </geometry>
+                </collision>
+            </xacro:if>
+            <xacro:if value="${collider == 'simple'}">
+                <collision name="simple_link8">
+                    <origin xyz="0.0262 0 0.0002" rpy="0 0 0"/>
+                    <geometry>
+                        <box size="0.08 0.04 0.0640"/>
+                    </geometry>
+                </collision>
+            </xacro:if>
         </link>
         <joint name="${prefix}joint8" type="prismatic">
@@ -381,4 +398,25 @@
                     </geometry>
                 </visual>
+                <xacro:if value="${collider == 'convex'}">
+                    <collision>
+                        <geometry>
+                            <mesh filename="file://$(find arx5_description)/meshes/camera_stand/stand_d405.obj"/>
+                        </geometry>
+                    </collision>
+                </xacro:if>
+                <xacro:if value="${collider == 'simple'}">
+                    <collision name="simple_d405_1">
+                        <origin xyz="0.0142 0 0.055" rpy="0 ${PI/6} 0"/>
+                        <geometry>
+                            <box size="0.01 0.05 0.06"/>
+                        </geometry>
+                    </collision>
+                    <collision name="simple_d405_2">
+                        <origin xyz="0.001 0 0.014" rpy="0 0 0"/>
+                        <geometry>
+                            <box size="0.01 0.05 0.03"/>
+                        </geometry>
+                    </collision>
+                </xacro:if>
             </link>
             <joint name="${prefix}camera_support_fixed" type="fixed">
@@ -393,4 +431,19 @@
                     </geometry>
                 </visual>
+                <xacro:if value="${collider == 'convex'}">
+                    <collision>
+                        <geometry>
+                            <mesh filename="file://$(find sensor_models)/meshes/d405/d405.obj"/>
+                        </geometry>
+                    </collision>
+                </xacro:if>
+                <xacro:if value="${collider == 'simple'}">
+                    <collision name="simple_d405camera">
+                        <origin xyz="-0.0115 0 0" rpy="0 0 0"/>
+                        <geometry>
+                            <box size="0.0231 0.0421 0.042"/>
+                        </geometry>
+                    </collision>
+                </xacro:if>
             </link>
             <joint name="${prefix}camera_fixed" type="fixed">
@@ -407,4 +460,19 @@
                     </geometry>
                 </visual>
+                <xacro:if value="${collider == 'convex'}">
+                    <collision>
+                        <geometry>
+                            <mesh filename="file://$(find arx5_description)/meshes/camera_stand/stand_d435.obj"/>
+                        </geometry>
+                    </collision>
+                </xacro:if>
+                <xacro:if value="${collider == 'simple'}">
+                    <collision name="simple_d435">
+                        <origin xyz="0.001 0 0.014" rpy="0 0 0"/>
+                        <geometry>
+                            <box size="0.01 0.05 0.03"/>
+                        </geometry>
+                    </collision>
+                </xacro:if>
             </link>
             <joint name="${prefix}camera_support_fixed" type="fixed">
@@ -419,4 +487,17 @@
                     </geometry>
                 </visual>
+                <xacro:if value="${collider == 'convex'}">
+                    <geometry>
+                        <mesh filename="file://$(find sensor_models)/meshes/d435/d435.obj"/>
+                    </geometry>
+                </xacro:if>
+                <xacro:if value="${collider == 'simple'}">
+                    <collision name="simple_d435camera">
+                        <origin xyz="-0.0125 0 0" rpy="0 0 0"/>
+                        <geometry>
+                            <box size="0.0251 0.0899 0.025"/>
+                        </geometry>
+                    </collision>
+                </xacro:if>
             </link>
             <joint name="${prefix}camera_fixed" type="fixed">

File: arx5_description/xacro/robot.xacro (robot description, xacro)
@@ -5,5 +5,5 @@
   <xacro:if value="${'$(arg type)' == 'r5'}">
     <xacro:include filename="$(find arx5_description)/xacro/R5.xacro"/>
-    <xacro:R5 name=""/>
+    <xacro:R5 name="" collider="$(arg collider)"/>
   </xacro:if>
   <xacro:if value="${'$(arg type)' == 'x5'}">

Commit message: ACone_X5已设置自碰撞

File: arx5_description/xacro/R5.xacro (robot description, xacro)
@@ -1,6 +1,8 @@
 <?xml version="1.0"?>
 <robot xmlns:xacro="http://www.ros.org/wiki/xacro">
+    <xacro:arg name="collider" default="simple"/>
     <xacro:property name="PI" value="3.1415926535897931"/>
-    <xacro:macro name="R5" params="name camera:=d405 style:=default collider:=convex">
+    <xacro:property name="collider_type" value="$(arg collider)"/>
+    <xacro:macro name="R5" params="name camera:=d405 style:=default collider:=simple">
         <xacro:property name="prefix" value="${name + '_' if name else ''}"/>
         <link name="${prefix}base_link">

File: arx5_description/xacro/X5.xacro (robot description, xacro)
@@ -1,6 +1,8 @@
 <?xml version="1.0"?>
 <robot xmlns:xacro="http://www.ros.org/wiki/xacro">
+    <xacro:arg name="collider" default="simple"/>
     <xacro:property name="PI" value="3.1415926535897931"/>
-    <xacro:macro name="X5" params="name camera:=d405 collider:=convex">
+    <xacro:property name="collider_type" value="$(arg collider)"/>
+    <xacro:macro name="X5" params="name collider:=simple camera:=d405">
         <xacro:property name="prefix" value="${name + '_' if name else ''}"/>
         <link name="${prefix}base_link">

File: arx5_description/xacro/robot.xacro (robot description, xacro)
@@ -1,5 +1,5 @@
 <?xml version="1.0"?>
 <robot name="ARX 5" xmlns:xacro="http://www.ros.org/wiki/xacro">
-  <xacro:arg name="collider" default="convex"/>
+  <xacro:arg name="collider" default="simple"/>
   <xacro:arg name="type" default="x5"/>
   <xacro:if value="${'$(arg type)' == 'r5'}">

File: arx_lift2s_description/xacro/robot.xacro (robot description, xacro)
@@ -3,5 +3,5 @@
 	<xacro:arg name="enable_wheel_joints" default="false"/>
 	<xacro:arg name="ros2_control_hardware_type" default="mock_components"/>
-	<xacro:arg name="collider" default ="convex"/>
+	<xacro:arg name="collider" default ="simple"/>
 	<xacro:property name="type_arg" value="$(arg type)"/>
 	<xacro:property name="selected_arm_type" value="x5"/>
@@ -43,6 +43,6 @@
 	<xacro:if value="${selected_arm_type == 'r5'}">
 		<xacro:include filename="$(find arx5_description)/xacro/R5.xacro"/>
-		<xacro:R5 name="left"/>
-		<xacro:R5 name="right"/>
+		<xacro:R5 name="left" collider="$(arg collider)"/>
+		<xacro:R5 name="right" collider="$(arg collider)"/>
 	</xacro:if>
 	<joint name="arm_left_fixed" type="fixed">
