Commit message: modified d405 direction

File: arx5_description/xacro/R5.xacro (robot description, xacro)
@@ -439,5 +439,5 @@
 				<visual>
 					<geometry>
-						<mesh filename="file://$(find sensor_models)/meshes/d405/d405.obj"/>
+						<mesh filename="file://$(find sensor_models)/meshes/realsense/d405.glb"/>
 					</geometry>
 				</visual>
@@ -445,5 +445,5 @@
 					<collision>
 						<geometry>
-							<mesh filename="file://$(find sensor_models)/meshes/d405/d405.obj"/>
+							<mesh filename="file://$(find sensor_models)/meshes/realsense/d405.glb"/>
 						</geometry>
 					</collision>
@@ -459,5 +459,5 @@
 			</link>
 			<joint name="${prefix}camera_fixed" type="fixed">
-				<origin xyz="0.0385 0 0.0475" rpy="0 0.523 0"/>
+				<origin xyz="0.0385 0 0.0475" rpy="-2.093 0 -1.5708"/>
 				<parent link="${prefix}camera_support"/>
 				<child link="${prefix}camera"/>

File: arx5_description/xacro/X5.xacro (robot description, xacro)
@@ -430,5 +430,5 @@
                 <visual>
                     <geometry>
-                        <mesh filename="file://$(find sensor_models)/meshes/d405/d405.obj"/>
+                        <mesh filename="file://$(find sensor_models)/meshes/realsense/d405.glb"/>
                     </geometry>
                 </visual>
@@ -436,5 +436,5 @@
                     <collision>
                         <geometry>
-                            <mesh filename="file://$(find sensor_models)/meshes/d405/d405.obj"/>
+                            <mesh filename="file://$(find sensor_models)/meshes/realsense/d405.glb"/>
                         </geometry>
                     </collision>
@@ -450,5 +450,5 @@
             </link>
             <joint name="${prefix}camera_fixed" type="fixed">
-                <origin xyz="0.0385 0 0.0475" rpy="0 0.523 0"/>
+                <origin xyz="0.0385 0 0.0475" rpy="-2.093 0 -1.5708"/>
                 <parent link="${prefix}camera_support"/>
                 <child link="${prefix}camera"/>

File: arx5_description/xacro/X5_ac1.xacro (robot description, xacro)
@@ -433,5 +433,5 @@
 				<visual>
 					<geometry>
-						<mesh filename="file://$(find sensor_models)/meshes/d405/d405.obj"/>
+						<mesh filename="file://$(find sensor_models)/meshes/realsense/d405.glb"/>
 					</geometry>
 				</visual>
@@ -439,5 +439,5 @@
 					<collision>
 						<geometry>
-							<mesh filename="file://$(find sensor_models)/meshes/d405/d405.obj"/>
+							<mesh filename="file://$(find sensor_models)/meshes/realsense/d405.glb"/>
 						</geometry>
 					</collision>
@@ -453,5 +453,5 @@
 			</link>
 			<joint name="${prefix}camera_fixed" type="fixed">
-				<origin xyz="0.0385 0 0.0475" rpy="0 0.523 0"/>
+				<origin xyz="0.0385 0 0.0475" rpy="-2.093 0 -1.5708"/>
 				<parent link="${prefix}camera_support"/>
 				<child link="${prefix}camera"/>

File: arx_lift2s_description/xacro/components/ac_one.xacro (robot description, xacro)
@@ -51,10 +51,11 @@
 			<visual>
 				<geometry>
-					<mesh filename="file://$(find sensor_models)/meshes/d405/d405.obj"/>
+					<mesh filename="file://$(find sensor_models)/meshes/realsense/d405.glb"/>
 				</geometry>
 			</visual>
 		</link>
 		<joint name="head_camera_joint" type="fixed">
-			<origin xyz="0.090415 0.002 0.2285" rpy="0 1.0472 0"/>
+<!--			<origin xyz="0.090415 0.002 0.2285" rpy="0 1.0472 0"/>-->
+			<origin xyz="0.090415 0.002 0.2285" rpy="-2.618 0 -1.5708"/>
 			<parent link="body_link"/>
 			<child link="head_camera"/>

File: arx_lift_description/xacro/components/body.xacro (robot description, xacro)
@@ -112,10 +112,10 @@
             <visual>
                 <geometry>
-                    <mesh filename="file://$(find sensor_models)/meshes/d405/d405.obj"/>
+                    <mesh filename="file://$(find sensor_models)/meshes/realsense/d405.glb"/>
                 </geometry>
             </visual>
         </link>
         <joint name="head_camera_joint" type="fixed">
-            <origin xyz="0.095 0.025 0.06"/>
+            <origin xyz="0.095 0.025 0.06" rpy="-1.5708 0 -1.5708"/>
             <parent link="head_link2"/>
             <child link="head_camera"/>

File: arx_x7s_description/xacro/components/body.xacro (robot description, xacro)
@@ -96,10 +96,10 @@
       <visual>
         <geometry>
-          <mesh filename="file://$(find sensor_models)/meshes/d405/d405.obj"/>
+          <mesh filename="file://$(find sensor_models)/meshes/realsense/d405.glb"/>
         </geometry>
       </visual>
     </link>
     <joint name="head_camera_joint" type="fixed">
-      <origin xyz="0.095 0.025 0.06"/>
+      <origin xyz="0.095 0.025 0.06" rpy="-1.5708 0 -1.5708"/>
       <parent link="head"/>
       <child link="head_camera"/>
