Commit message: add component xacro

File: arx5_description/xacro/R5.xacro (robot description, xacro)
@@ -4,5 +4,6 @@
 	<xacro:property name="PI" value="3.1415926535897931"/>
 	<xacro:property name="collider_type" value="$(arg collider)"/>
-	<xacro:macro name="R5" params="name camera:=d405 style:=default collider:=simple">
+	<xacro:include filename="$(find arx5_description)/xacro/components/gripper_2023.xacro"/>
+	<xacro:macro name="R5" params="name camera:=d405 style:=default collider:=simple with_gripper:='true'">
 		<xacro:property name="prefix" value="${name + '_' if name else ''}"/>
 		<link name="${prefix}base_link">
@@ -263,260 +264,18 @@
 			<limit lower="-1.57" upper="1.57" effort="100" velocity="5"/>
 		</joint>
-		<link name="${prefix}link6">
-			<inertial>
-				<origin xyz="0.041697 2.4368E-05 0.00014464"/>
-				<mass value="0.44089"/>
-				<inertia
-						ixx="0.00038"
-						ixy="0.00000"
-						ixz="0.00000"
-						iyy="0.00028"
-						iyz="0.00000"
-						izz="0.00050"/>
-			</inertial>
-			<visual>
-				<geometry>
-					<mesh filename="file://$(find arx5_description)/meshes/r5/link6.glb"/>
-				</geometry>
-			</visual>
-			<xacro:if value="${collider == 'convex'}">
-				<collision>
-					<geometry>
-						<mesh filename="file://$(find arx5_description)/meshes/r5/link6.glb"/>
-					</geometry>
-				</collision>
-			</xacro:if>
-			<xacro:if value="${collider == 'simple'}">
-				<collision name="simple_link6">
-					<origin xyz="0.038 0 0.0002" rpy="0 ${PI/2} 0"/>
-					<geometry>
-						<cylinder length="0.064" radius="0.03015"/>
-					</geometry>
-				</collision>
-			</xacro:if>
-		</link>
+		<link name="${prefix}ee"/>
 		<joint name="${prefix}joint6" type="revolute">
 			<origin xyz="0.025286 0 0.083391" rpy="3.1416 0 0"/>
 			<parent link="${prefix}link5"/>
-			<child link="${prefix}link6"/>
+			<child link="${prefix}ee"/>
 			<axis xyz="1 0 0"/>
 			<limit lower="-1.57" upper="1.57" effort="100" velocity="5"/>
 		</joint>
-		<link name="${prefix}link7">
-			<inertial>
-				<origin xyz="-0.00035522 -0.007827 -0.0029883"/>
-				<mass value="0.064798"/>
-				<inertia
-						ixx="0.00002"
-						ixy="0.00000"
-						ixz="0.00000"
-						iyy="0.00003"
-						iyz="0.00000"
-						izz="0.00003"/>
-			</inertial>
-			<visual>
-				<geometry>
-					<mesh filename="file://$(find arx5_description)/meshes/r5/link7.glb"/>
-				</geometry>
-			</visual>
-			<xacro:if value="${collider == 'convex'}">
-				<collision>
-					<geometry>
-						<mesh filename="file://$(find arx5_description)/meshes/r5/link7.glb"/>
-					</geometry>
-				</collision>
-			</xacro:if>
-			<xacro:if value="${collider == 'simple'}">
-				<collision name="simple_link7">
-					<origin xyz="0.0262 0 0.0002" rpy="0 0 0"/>
-					<geometry>
-						<box size="0.08 0.04 0.0640"/>
-					</geometry>
-				</collision>
-			</xacro:if>
-		</link>
-		<joint name="${prefix}gripper_joint" type="prismatic">
-			<origin xyz="0.08657 0.024896 -0.0002436"/>
-			<parent link="${prefix}link6"/>
-			<child link="${prefix}link7"/>
-			<axis xyz="0 1 0"/>
-			<limit lower="0" upper="0.044" effort="100" velocity="5"/>
-		</joint>
-		<link name="${prefix}link8">
-			<inertial>
-				<origin xyz="-0.000355223470270755 0.00782768751820277 0.00242005642879778"/>
-				<mass value="0.0647981725781684"/>
-				<inertia
-						ixx="0.00002"
-						ixy="0.00000"
-						ixz="0.00000"
-						iyy="0.00003"
-						iyz="0.00000"
-						izz="0.00003"/>
-			</inertial>
-			<visual>
-				<geometry>
-					<mesh filename="file://$(find arx5_description)/meshes/r5/link8.glb"/>
-				</geometry>
-			</visual>
-			<xacro:if value="${collider == 'convex'}">
-				<collision>
-					<geometry>
-						<mesh filename="file://$(find arx5_description)/meshes/r5/link8.glb"/>
-					</geometry>
-				</collision>
-			</xacro:if>
-			<xacro:if value="${collider == 'simple'}">
-				<collision name="simple_link8">
-					<origin xyz="0.0262 0 0.0002" rpy="0 0 0"/>
-					<geometry>
-						<box size="0.08 0.04 0.0640"/>
-					</geometry>
-				</collision>
-			</xacro:if>
-		</link>
-		<joint name="${prefix}joint8" type="prismatic">
-			<origin xyz="0.08657 -0.0249 -0.00024366"/>
-			<parent link="${prefix}link6"/>
-			<child link="${prefix}link8"/>
-			<axis xyz="0 -1 0"/>
-			<limit lower="0" upper="0.044" effort="100" velocity="5"/>
-			<mimic joint="${prefix}gripper_joint" multiplier="1" offset="0"/>
-		</joint>
-		<link name="${prefix}gripper_center"/>
-		<joint name="${prefix}gripper_center_fixed" type="fixed">
-			<parent link="${prefix}link6"/>
-			<child link="${prefix}gripper_center"/>
-			<origin xyz="0.08657 0 0"/>
-		</joint>
-		<link name="${prefix}left_pad"/>
-		<joint name="${prefix}left_pad_joint" type="fixed">
-			<parent link="${prefix}link7"/>
-			<child link="${prefix}left_pad"/>
-			<origin xyz="0.05843 -0.0249 0"/>
-		</joint>
-		<link name="${prefix}right_pad"/>
-		<joint name="${prefix}right_pad_joint" type="fixed">
-			<parent link="${prefix}link8"/>
-			<child link="${prefix}right_pad"/>
-			<origin xyz="0.05843 0.0249 0"/>
-		</joint>
-		<xacro:if value="${camera == 'd405'}">
-			<link name="${prefix}camera_support">
-				<visual>
-					<geometry>
-						<mesh filename="file://$(find arx5_description)/meshes/camera_stand/stand_d405.glb"/>
-					</geometry>
-				</visual>
-				<xacro:if value="${collider == 'convex'}">
-					<collision>
-						<geometry>
-							<mesh filename="file://$(find arx5_description)/meshes/camera_stand/stand_d405.glb"/>
-						</geometry>
-					</collision>
-				</xacro:if>
-				<xacro:if value="${collider == 'simple'}">
-					<collision name="simple_d405_1">
-						<origin xyz="0.0142 0 0.055" rpy="0 ${PI/6} 0"/>
-						<geometry>
-							<box size="0.01 0.05 0.06"/>
-						</geometry>
-					</collision>
-					<collision name="simple_d405_2">
-						<origin xyz="0.001 0 0.014" rpy="0 0 0"/>
-						<geometry>
-							<box size="0.01 0.05 0.03"/>
-						</geometry>
-					</collision>
-				</xacro:if>
-			</link>
-			<joint name="${prefix}camera_support_fixed" type="fixed">
-				<parent link="${prefix}link6"/>
-				<child link="${prefix}camera_support"/>
-				<origin xyz="0.045 0 0.021"/>
-			</joint>
-			<link name="${prefix}camera">
-				<visual>
-					<geometry>
-						<mesh filename="file://$(find sensor_models)/meshes/realsense/d405.glb"/>
-					</geometry>
-				</visual>
-				<xacro:if value="${collider == 'convex'}">
-					<collision>
-						<geometry>
-							<mesh filename="file://$(find sensor_models)/meshes/realsense/d405.glb"/>
-						</geometry>
-					</collision>
-				</xacro:if>
-				<xacro:if value="${collider == 'simple'}">
-					<collision name="simple_d405camera">
-						<origin xyz="-0.0115 0 0" rpy="0 0 0"/>
-						<geometry>
-							<box size="0.0231 0.0421 0.042"/>
-						</geometry>
-					</collision>
-				</xacro:if>
-			</link>
-			<joint name="${prefix}camera_fixed" type="fixed">
-				<origin xyz="0.0385 0 0.0475" rpy="-2.093 0 -1.5708"/>
-				<parent link="${prefix}camera_support"/>
-				<child link="${prefix}camera"/>
-			</joint>
-		</xacro:if>
-		<xacro:if value="${camera == 'd435'}">
-			<link name="${prefix}camera_support">
-				<visual>
-					<geometry>
-						<mesh filename="file://$(find arx5_description)/meshes/camera_stand/stand_d435.glb"/>
-					</geometry>
-				</visual>
-				<xacro:if value="${collider == 'convex'}">
-					<collision>
-						<geometry>
-							<mesh filename="file://$(find arx5_description)/meshes/camera_stand/stand_d435.glb"/>
-						</geometry>
-					</collision>
-				</xacro:if>
-				<xacro:if value="${collider == 'simple'}">
-					<collision name="simple_d435">
-						<origin xyz="0.001 0 0.014" rpy="0 0 0"/>
-						<geometry>
-							<box size="0.01 0.05 0.03"/>
-						</geometry>
-					</collision>
-				</xacro:if>
-			</link>
-			<joint name="${prefix}camera_support_fixed" type="fixed">
-				<parent link="${prefix}link6"/>
-				<child link="${prefix}camera_support"/>
-				<origin xyz="0.045 0 0.021"/>
-			</joint>
-			<link name="${prefix}camera">
-				<visual>
-					<geometry>
-						<mesh filename="file://$(find sensor_models)/meshes/d435/d435.obj"/>
-					</geometry>
-				</visual>
-				<xacro:if value="${collider == 'convex'}">
-					<collision>
-						<geometry>
-							<mesh filename="file://$(find sensor_models)/meshes/d435/d435.obj"/>
-						</geometry>
-					</collision>
-				</xacro:if>
-				<xacro:if value="${collider == 'simple'}">
-					<collision name="simple_d435camera">
-						<origin xyz="-0.0125 0 0" rpy="0 0 0"/>
-						<geometry>
-							<box size="0.0251 0.0899 0.025"/>
-						</geometry>
-					</collision>
-				</xacro:if>
-			</link>
-			<joint name="${prefix}camera_fixed" type="fixed">
-				<origin xyz="0.03 0 0.034113"/>
-				<parent link="${prefix}camera_support"/>
-				<child link="${prefix}camera"/>
-			</joint>
+		<xacro:if value="${str(with_gripper).lower() in ['1', 'true', 'yes', 'on']}">
+			<xacro:arx_gripper_2023
+				prefix="${prefix}"
+				parent_link="${prefix}ee"
+				collider="${collider}"
+				camera="${camera}"/>
 		</xacro:if>
 	</xacro:macro>

File: arx5_description/xacro/X5.xacro (robot description, xacro)
@@ -4,5 +4,6 @@
     <xacro:property name="PI" value="3.1415926535897931"/>
     <xacro:property name="collider_type" value="$(arg collider)"/>
-    <xacro:macro name="X5" params="name collider:=simple camera:=d405">
+    <xacro:include filename="$(find arx5_description)/xacro/components/gripper_2023.xacro"/>
+    <xacro:macro name="X5" params="name collider:=simple camera:=d405 with_gripper:='true'">
         <xacro:property name="prefix" value="${name + '_' if name else ''}"/>
         <link name="${prefix}base_link">
@@ -253,258 +254,18 @@
             <limit lower="-1.57" upper="1.57" effort="100" velocity="5"/>
         </joint>
-        <link name="${prefix}link6">
-            <inertial>
-                <origin xyz="0.041697 2.4368E-05 0.00014464"/>
-                <mass value="0.44089"/>
-                <inertia
-                        ixx="0.00038"
-                        ixy="0.00000"
-                        ixz="0.00000"
-                        iyy="0.00028"
-                        iyz="0.00000"
-                        izz="0.00050"/>
-            </inertial>
-            <visual>
-                <geometry>
-                    <mesh filename="file://$(find arx5_description)/meshes/r5/link6.glb"/>
-                </geometry>
-            </visual>
-            <xacro:if value="${collider == 'convex'}">
-                <collision>
-                    <geometry>
-                        <mesh filename="file://$(find arx5_description)/meshes/r5/link6.glb"/>
-                    </geometry>
-                </collision>
-            </xacro:if>
-            <xacro:if value="${collider == 'simple'}">
-                <collision name="simple_link6">
-                    <origin xyz="0.038 0 0.0002" rpy="0 ${PI/2} 0"/>
-                    <geometry>
-                        <cylinder length="0.064" radius="0.03015"/>
-                    </geometry>
-                </collision>
-            </xacro:if>
-        </link>
+        <link name="${prefix}ee"/>
         <joint name="${prefix}joint6" type="revolute">
             <origin xyz="0.02895 0 0.0865" rpy="-3.1416 0 0"/>
             <parent link="${prefix}link5"/>
-            <child link="${prefix}link6"/>
+            <child link="${prefix}ee"/>
             <axis xyz="1 0 0"/>
             <limit lower="-1.57" upper="1.57" effort="100" velocity="5"/>
         </joint>
-        <link name="${prefix}link7">
-            <inertial>
-                <origin xyz="-0.00035522 -0.007827 -0.0029883"/>
-                <mass value="0.064798"/>
-                <inertia
-                        ixx="0.00002"
-                        ixy="0.00000"
-                        ixz="0.00000"
-                        iyy="0.00003"
-                        iyz="0.00000"
-                        izz="0.00003"/>
-            </inertial>
-            <visual>
-                <geometry>
-                    <mesh filename="file://$(find arx5_description)/meshes/r5/link7.glb"/>
-                </geometry>
-            </visual>
-            <xacro:if value="${collider == 'convex'}">
-                <collision>
-                    <geometry>
-                        <mesh filename="file://$(find arx5_description)/meshes/r5/link7.glb"/>
-                    </geometry>
-                </collision>
-            </xacro:if>
-            <xacro:if value="${collider == 'simple'}">
-                <collision name="simple_link7">
-                    <origin xyz="0.0262 0 0.0002" />
-                    <geometry>
-                        <box size="0.08 0.04 0.0640"/>
-                    </geometry>
-                </collision>
-            </xacro:if>
-        </link>
-        <joint name="${prefix}gripper_joint" type="prismatic">
-            <origin xyz="0.08657 0.024896 -0.0002436"/>
-            <parent link="${prefix}link6"/>
-            <child link="${prefix}link7"/>
-            <axis xyz="0 1 0"/>
-            <limit lower="0" upper="0.044" effort="100" velocity="5"/>
-        </joint>
-        <link name="${prefix}link8">
-            <inertial>
-                <origin xyz="-0.00035522 0.0078277 0.0024201"/>
-                <mass value="0.064798"/>
-                <inertia
-                        ixx="0.00002"
-                        ixy="0.00000"
-                        ixz="0.00000"
-                        iyy="0.00003"
-                        iyz="0.00000"
-                        izz="0.00003"/>
-            </inertial>
-            <visual>
-                <geometry>
-                    <mesh filename="file://$(find arx5_description)/meshes/r5/link8.glb"/>
-                </geometry>
-            </visual>
-            <xacro:if value="${collider == 'convex'}">
-                <collision>
-                    <geometry>
-                        <mesh filename="file://$(find arx5_description)/meshes/r5/link8.glb"/>
-                    </geometry>
-                </collision>
-            </xacro:if>
-            <xacro:if value="${collider == 'simple'}">
-                <collision name="simple_link8">
-                    <origin xyz="0.0262 0 0.0002" />
-                    <geometry>
-                        <box size="0.08 0.04 0.0640"/>
-                    </geometry>
-                </collision>
-            </xacro:if>
-        </link>
-        <joint name="${prefix}joint8" type="prismatic">
-            <origin xyz="0.08657 -0.0249 -0.00024366"/>
-            <parent link="${prefix}link6"/>
-            <child link="${prefix}link8"/>
-            <axis xyz="0 -1 0"/>
-            <limit lower="0" upper="0.044" effort="100" velocity="5"/>
-            <mimic joint="${prefix}gripper_joint" multiplier="1" offset="0"/>
-        </joint>
-        <link name="${prefix}gripper_center"/>
-        <joint name="${prefix}gripper_center_fixed" type="fixed">
-            <parent link="${prefix}link6"/>
-            <child link="${prefix}gripper_center"/>
-            <origin xyz="0.145 0 0"/>
-        </joint>
-        <link name="${prefix}left_pad"/>
-        <joint name="${prefix}left_pad_joint" type="fixed">
-            <parent link="${prefix}link7"/>
-            <child link="${prefix}left_pad"/>
-            <origin xyz="0.05843 -0.0249 0"/>
-        </joint>
-        <link name="${prefix}right_pad"/>
-        <joint name="${prefix}right_pad_joint" type="fixed">
-            <parent link="${prefix}link8"/>
-            <child link="${prefix}right_pad"/>
-            <origin xyz="0.05843 0.0249 0"/>
-        </joint>
-        <xacro:if value="${camera == 'd405'}">
-            <link name="${prefix}camera_support">
-                <visual>
-                    <geometry>
-                        <mesh filename="file://$(find arx5_description)/meshes/camera_stand/stand_d405.glb"/>
-                    </geometry>
-                </visual>
-                <xacro:if value="${collider == 'convex'}">
-                    <collision>
-                        <geometry>
-                            <mesh filename="file://$(find arx5_description)/meshes/camera_stand/stand_d405.glb"/>
-                        </geometry>
-                    </collision>
-                </xacro:if>
-                <xacro:if value="${collider == 'simple'}">
-                    <collision name="simple_d405_1">
-                        <origin xyz="0.0142 0 0.055" rpy="0 ${PI/6} 0"/>
-                        <geometry>
-                            <box size="0.01 0.05 0.06"/>
-                        </geometry>
-                    </collision>
-                    <collision name="simple_d405_2">
-                        <origin xyz="0.001 0 0.014" />
-                        <geometry>
-                            <box size="0.01 0.05 0.03"/>
-                        </geometry>
-                    </collision>
-                </xacro:if>
-            </link>
-            <joint name="${prefix}camera_support_fixed" type="fixed">
-                <parent link="${prefix}link6"/>
-                <child link="${prefix}camera_support"/>
-                <origin xyz="0.045 0 0.021"/>
-            </joint>
-            <link name="${prefix}camera">
-                <visual>
-                    <geometry>
-                        <mesh filename="file://$(find sensor_models)/meshes/realsense/d405.glb"/>
-                    </geometry>
-                </visual>
-                <xacro:if value="${collider == 'convex'}">
-                    <collision>
-                        <geometry>
-                            <mesh filename="file://$(find sensor_models)/meshes/realsense/d405.glb"/>
-                        </geometry>
-                    </collision>
-                </xacro:if>
-                <xacro:if value="${collider == 'simple'}">
-                    <collision name="simple_d405camera">
-                        <origin xyz="-0.0115 0 0" />
-                        <geometry>
-                            <box size="0.0231 0.0421 0.042"/>
-                        </geometry>
-                    </collision>
-                </xacro:if>
-            </link>
-            <joint name="${prefix}camera_fixed" type="fixed">
-                <origin xyz="0.0385 0 0.0475" rpy="-2.093 0 -1.5708"/>
-                <parent link="${prefix}camera_support"/>
-                <child link="${prefix}camera"/>
-            </joint>
-        </xacro:if>
-        <xacro:if value="${camera == 'd435'}">
-            <link name="${prefix}camera_support">
-                <visual>
-                    <geometry>
-                        <mesh filename="file://$(find arx5_description)/meshes/camera_stand/stand_d435.glb"/>
-                    </geometry>
-                </visual>
-                <xacro:if value="${collider == 'convex'}">
-                    <collision>
-                        <geometry>
-                            <mesh filename="file://$(find arx5_description)/meshes/camera_stand/stand_d435.glb"/>
-                        </geometry>
-                    </collision>
-                </xacro:if>
-                <xacro:if value="${collider == 'simple'}">
-                    <collision name="simple_d435">
-                        <origin xyz="0.001 0 0.014" />
-                        <geometry>
-                            <box size="0.01 0.05 0.03"/>
-                        </geometry>
-                    </collision>
-                </xacro:if>
-            </link>
-            <joint name="${prefix}camera_support_fixed" type="fixed">
-                <parent link="${prefix}link6"/>
-                <child link="${prefix}camera_support"/>
-                <origin xyz="0.045 0 0.021"/>
-            </joint>
-            <link name="${prefix}camera">
-                <visual>
-                    <geometry>
-                        <mesh filename="file://$(find sensor_models)/meshes/d435/d435.obj"/>
-                    </geometry>
-                </visual>
-                <xacro:if value="${collider == 'convex'}">
-                    <geometry>
-                        <mesh filename="file://$(find sensor_models)/meshes/d435/d435.obj"/>
-                    </geometry>
-                </xacro:if>
-                <xacro:if value="${collider == 'simple'}">
-                    <collision name="simple_d435camera">
-                        <origin xyz="-0.0125 0 0" />
-                        <geometry>
-                            <box size="0.0251 0.0899 0.025"/>
-                        </geometry>
-                    </collision>
-                </xacro:if>
-            </link>
-            <joint name="${prefix}camera_fixed" type="fixed">
-                <origin xyz="0.03 0 0.034113"/>
-                <parent link="${prefix}camera_support"/>
-                <child link="${prefix}camera"/>
-            </joint>
+        <xacro:if value="${str(with_gripper).lower() in ['1', 'true', 'yes', 'on']}">
+            <xacro:arx_gripper_2023
+                prefix="${prefix}"
+                parent_link="${prefix}ee"
+                collider="${collider}"
+                camera="${camera}"/>
         </xacro:if>
     </xacro:macro>
