Commit message: 添加了X5的一部分简单碰撞体

File: arx5_description/xacro/X5.xacro (robot description, xacro)
@@ -1,341 +1,426 @@
 <?xml version="1.0"?>
 <robot xmlns:xacro="http://www.ros.org/wiki/xacro">
-  <xacro:macro name="X5" params="name camera:=d405">
-    <xacro:property name="prefix" value="${name + '_' if name else ''}"/>
-    <link name="${prefix}base_link">
-      <inertial>
-        <origin xyz="-3.0001E-05 3.0589E-05 0.027324"/>
-        <mass value="0.43995"/>
-        <inertia
-            ixx="0.00017"
-            ixy="0.00000"
-            ixz="0.00000"
-            iyy="0.00017"
-            iyz="0.00000"
-            izz="0.00016"/>
-      </inertial>
-      <visual>
-        <geometry>
-          <mesh filename="file://$(find arx5_description)/meshes/x5/base_link.obj"/>
-        </geometry>
-      </visual>
-      <collision>
-        <geometry>
-          <mesh filename="file://$(find arx5_description)/meshes/x5/base_link.obj"/>
-        </geometry>
-      </collision>
-    </link>
-    <link name="${prefix}link1">
-      <inertial>
-        <origin xyz="0.0054231 -0.0080289 0.017086"/>
-        <mass value="0.066982"/>
-        <inertia
-            ixx="0.00008"
-            ixy="0.00000"
-            ixz="0.00001"
-            iyy="0.00003"
-            iyz="0.00000"
-            izz="0.00008"/>
-      </inertial>
-      <visual>
-        <geometry>
-          <mesh filename="file://$(find arx5_description)/meshes/x5/link1.obj"/>
-        </geometry>
-      </visual>
-      <collision>
-        <geometry>
-          <mesh filename="file://$(find arx5_description)/meshes/x5/link1.obj"/>
-        </geometry>
-      </collision>
-    </link>
-    <joint name="${prefix}joint1" type="revolute">
-      <origin xyz="0 0 0.0605"/>
-      <parent link="${prefix}base_link"/>
-      <child link="${prefix}link1"/>
-      <axis xyz="0 0 1"/>
-      <limit lower="-2.87" upper="3.14" effort="100" velocity="5"/>
-    </joint>
-    <link name="${prefix}link2">
-      <inertial>
-        <origin xyz="-0.13237 0.0020852 0.00010549"/>
-        <mass value="1.0795"/>
-        <inertia
-            ixx="0.00051"
-            ixy="0.00001"
-            ixz="-0.00004"
-            iyy="0.01599"
-            iyz="0.00000"
-            izz="0.01605"/>
-      </inertial>
-      <visual>
-        <geometry>
-          <mesh filename="file://$(find arx5_description)/meshes/x5/link2.obj"/>
-        </geometry>
-      </visual>
-      <collision>
-        <geometry>
-          <mesh filename="file://$(find arx5_description)/meshes/x5/link2.obj"/>
-        </geometry>
-      </collision>
-    </link>
-    <joint name="${prefix}joint2" type="revolute">
-      <origin xyz="0.02 0 0.04"/>
-      <parent link="${prefix}link1"/>
-      <child link="${prefix}link2"/>
-      <axis xyz="0 1 0"/>
-      <limit lower="0" upper="3.66" effort="100" velocity="5"/>
-    </joint>
-    <link name="${prefix}link3">
-      <inertial>
-        <origin xyz="0.18531 0.00068376 -0.051638"/>
-        <mass value="0.54534"/>
-        <inertia
-            ixx="0.00036"
-            ixy="-0.00003"
-            ixz="-0.00039"
-            iyy="0.00423"
-            iyz="0.00001"
-            izz="0.00420"/>
-      </inertial>
-      <visual>
-        <geometry>
-          <mesh filename="file://$(find arx5_description)/meshes/x5/link3.obj"/>
-        </geometry>
-      </visual>
-      <collision>
-        <geometry>
-          <mesh filename="file://$(find arx5_description)/meshes/x5/link3.obj"/>
-        </geometry>
-      </collision>
-    </link>
-    <joint name="${prefix}joint3" type="revolute">
-      <origin xyz="-0.264 0 0" rpy="3.1416 0 0"/>
-      <parent link="${prefix}link2"/>
-      <child link="${prefix}link3"/>
-      <axis xyz="0 1 0"/>
-      <limit lower="0" upper="3.14" effort="100" velocity="5"/>
-    </joint>
-    <link name="${prefix}link4">
-      <inertial>
-        <origin xyz="0.040231 0.0044807 -0.035335"/>
-        <mass value="0.11714"/>
-        <inertia
-            ixx="0.00019"
-            ixy="-0.00002"
-            ixz="-0.00009"
-            iyy="0.00023"
-            iyz="0.00002"
-            izz="0.00014"/>
-      </inertial>
-      <visual>
-        <geometry>
-          <mesh filename="file://$(find arx5_description)/meshes/x5/link4.obj"/>
-        </geometry>
-      </visual>
-      <collision>
-        <geometry>
-          <mesh filename="file://$(find arx5_description)/meshes/x5/link4.obj"/>
-        </geometry>
-      </collision>
-    </link>
-    <joint name="${prefix}joint4" type="revolute">
-      <origin xyz="0.245 0 -0.056"/>
-      <parent link="${prefix}link3"/>
-      <child link="${prefix}link4"/>
-      <axis xyz="0 1 0"/>
-      <limit lower="-1.57" upper="1.57" effort="100" velocity="5"/>
-    </joint>
-    <link name="${prefix}link5">
-      <inertial>
-        <origin xyz="0.003612 -1.5455E-05 0.055214"/>
-        <mass value="0.63488"/>
-        <inertia
-            ixx="0.00083"
-            ixy="0.00000"
-            ixz="0.00007"
-            iyy="0.00082"
-            iyz="0.00000"
-            izz="0.00026"/>
-      </inertial>
-      <visual>
-        <origin xyz="0.0037 0 0"/>
-        <geometry>
-          <mesh filename="file://$(find arx5_description)/meshes/x5/link5.obj"/>
-        </geometry>
-      </visual>
-      <collision>
-        <geometry>
-          <mesh filename="file://$(find arx5_description)/meshes/x5/link5.obj"/>
-        </geometry>
-      </collision>
-    </link>
-    <joint name="${prefix}joint5" type="revolute">
-      <origin xyz="0.06775 0.0005 -0.0865"/>
-      <parent link="${prefix}link4"/>
-      <child link="${prefix}link5"/>
-      <axis xyz="0 0 1"/>
-      <limit lower="-1.57" upper="1.57" effort="100" velocity="5"/>
-    </joint>
-    <link name="${prefix}link6">
-      <inertial>
-        <origin xyz="0.041697 2.4368E-05 0.00014464"/>
-        <mass value="0.44089"/>
-        <inertia
-            ixx="0.00038"
-            ixy="0.00000"
-            ixz="0.00000"
-            iyy="0.00028"
-            iyz="0.00000"
-            izz="0.00050"/>
-      </inertial>
-      <visual>
-        <geometry>
-          <mesh filename="file://$(find arx5_description)/meshes/x5/link6.obj"/>
-        </geometry>
-      </visual>
-      <collision>
-        <geometry>
-          <mesh filename="file://$(find arx5_description)/meshes/x5/link6.obj"/>
-        </geometry>
-      </collision>
-    </link>
-    <joint name="${prefix}joint6" type="revolute">
-      <origin xyz="0.02895 0 0.0865" rpy="-3.1416 0 0"/>
-      <parent link="${prefix}link5"/>
-      <child link="${prefix}link6"/>
-      <axis xyz="1 0 0"/>
-      <limit lower="-1.57" upper="1.57" effort="100" velocity="5"/>
-    </joint>
-    <link name="${prefix}link7">
-      <inertial>
-        <origin xyz="-0.00035522 -0.007827 -0.0029883"/>
-        <mass value="0.064798"/>
-        <inertia
-            ixx="0.00002"
-            ixy="0.00000"
-            ixz="0.00000"
-            iyy="0.00003"
-            iyz="0.00000"
-            izz="0.00003"/>
-      </inertial>
-      <visual>
-        <geometry>
-          <mesh filename="file://$(find arx5_description)/meshes/x5/link7.obj"/>
-        </geometry>
-      </visual>
-      <collision>
-        <geometry>
-          <mesh filename="file://$(find arx5_description)/meshes/x5/link7.obj"/>
-        </geometry>
-      </collision>
-    </link>
-    <joint name="${prefix}gripper_joint" type="prismatic">
-      <origin xyz="0.08657 0.024896 -0.0002436"/>
-      <parent link="${prefix}link6"/>
-      <child link="${prefix}link7"/>
-      <axis xyz="0 1 0"/>
-      <limit lower="0" upper="0.044" effort="100" velocity="5"/>
-    </joint>
-    <link name="${prefix}link8">
-      <inertial>
-        <origin xyz="-0.00035522 0.0078277 0.0024201"/>
-        <mass value="0.064798"/>
-        <inertia
-            ixx="0.00002"
-            ixy="0.00000"
-            ixz="0.00000"
-            iyy="0.00003"
-            iyz="0.00000"
-            izz="0.00003"/>
-      </inertial>
-      <visual>
-        <geometry>
-          <mesh filename="file://$(find arx5_description)/meshes/x5/link8.obj"/>
-        </geometry>
-      </visual>
-      <collision>
-        <geometry>
-          <mesh filename="file://$(find arx5_description)/meshes/x5/link8.obj"/>
-        </geometry>
-      </collision>
-    </link>
-    <joint name="${prefix}joint8" type="prismatic">
-      <origin xyz="0.08657 -0.0249 -0.00024366"/>
-      <parent link="${prefix}link6"/>
-      <child link="${prefix}link8"/>
-      <axis xyz="0 -1 0"/>
-      <limit lower="0" upper="0.044" effort="100" velocity="5"/>
-      <mimic joint="${prefix}gripper_joint" multiplier="1" offset="0"/>
-    </joint>
-    <link name="${prefix}gripper_center"/>
-    <joint name="${prefix}gripper_center_fixed" type="fixed">
-      <parent link="${prefix}link6"/>
-      <child link="${prefix}gripper_center"/>
-      <origin xyz="0.145 0 0" />
-    </joint>
-    <link name="${prefix}left_pad"/>
-    <joint name="${prefix}left_pad_joint" type="fixed">
-      <parent link="${prefix}link7"/>
-      <child link="${prefix}left_pad"/>
-      <origin xyz="0.05843 -0.0249 0" />
-    </joint>
-    <link name="${prefix}right_pad"/>
-    <joint name="${prefix}right_pad_joint" type="fixed">
-      <parent link="${prefix}link8"/>
-      <child link="${prefix}right_pad"/>
-      <origin xyz="0.05843 0.0249 0" />
-    </joint>
-    <xacro:if value="${camera == 'd405'}">
-      <link name="${prefix}camera_support">
-        <visual>
-          <geometry>
-            <mesh filename="file://$(find arx5_description)/meshes/camera_stand/stand_d405.obj"/>
-          </geometry>
-        </visual>
-      </link>
-      <joint name="${prefix}camera_support_fixed" type="fixed">
-        <parent link="${prefix}link6"/>
-        <child link="${prefix}camera_support"/>
-        <origin xyz="0.045 0 0.021"/>
-      </joint>
-      <link name="${prefix}camera">
-        <visual>
-          <geometry>
-            <mesh filename="file://$(find sensor_models)/meshes/d405/d405.obj"/>
-          </geometry>
-        </visual>
-      </link>
-      <joint name="${prefix}camera_fixed" type="fixed">
-        <origin xyz="0.0385 0 0.0475" rpy="0 0.523 0"/>
-        <parent link="${prefix}camera_support"/>
-        <child link="${prefix}camera"/>
-      </joint>
-    </xacro:if>
-    <xacro:if value="${camera == 'd435'}">
-      <link name="${prefix}camera_support">
-        <visual>
-          <geometry>
-            <mesh filename="file://$(find arx5_description)/meshes/camera_stand/stand_d435.obj"/>
-          </geometry>
-        </visual>
-      </link>
-      <joint name="${prefix}camera_support_fixed" type="fixed">
-        <parent link="${prefix}link6"/>
-        <child link="${prefix}camera_support"/>
-        <origin xyz="0.045 0 0.021"/>
-      </joint>
-      <link name="${prefix}camera">
-        <visual>
-          <geometry>
-            <mesh filename="file://$(find sensor_models)/meshes/d435/d435.obj"/>
-          </geometry>
-        </visual>
-      </link>
-      <joint name="${prefix}camera_fixed" type="fixed">
-        <origin xyz="0.03 0 0.034113" />
-        <parent link="${prefix}camera_support"/>
-        <child link="${prefix}camera"/>
-      </joint>
-    </xacro:if>
-  </xacro:macro>
+    <xacro:property name="PI" value="3.1415926535897931"/>
+    <xacro:macro name="X5" params="name camera:=d405">
+        <xacro:property name="prefix" value="${name + '_' if name else ''}"/>
+        <link name="${prefix}base_link">
+            <inertial>
+                <origin xyz="-3.0001E-05 3.0589E-05 0.027324"/>
+                <mass value="0.43995"/>
+                <inertia
+                        ixx="0.00017"
+                        ixy="0.00000"
+                        ixz="0.00000"
+                        iyy="0.00017"
+                        iyz="0.00000"
+                        izz="0.00016"/>
+            </inertial>
+            <visual>
+                <geometry>
+                    <mesh filename="file://$(find arx5_description)/meshes/x5/base_link.obj"/>
+                </geometry>
+            </visual>
+            <xacro:if value="${collider == 'convex'}">
+                <collision>
+                    <geometry>
+                        <mesh filename="file://$(find arx5_description)/meshes/x5/base_link.obj"/>
+                    </geometry>
+                </collision>
+            </xacro:if>
+            <xacro:if value="${collider == 'simple'}">
+                <collision>
+                    <origin xyz="0 0 0.0312"/>
+                    <geometry>
+                        <cylinder length="0.03125" radius="0.031"/>
+                    </geometry>
+                </collision>
+            </xacro:if>
+        </link>
+        <link name="${prefix}link1">
+            <inertial>
+                <origin xyz="0.0054231 -0.0080289 0.017086"/>
+                <mass value="0.066982"/>
+                <inertia
+                        ixx="0.00008"
+                        ixy="0.00000"
+                        ixz="0.00001"
+                        iyy="0.00003"
+                        iyz="0.00000"
+                        izz="0.00008"/>
+            </inertial>
+            <visual>
+                <geometry>
+                    <mesh filename="file://$(find arx5_description)/meshes/x5/link1.obj"/>
+                </geometry>
+            </visual>
+            <collision>
+                <geometry>
+                    <mesh filename="file://$(find arx5_description)/meshes/x5/link1.obj"/>
+                </geometry>
+            </collision>
+        </link>
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
File: arx5_description/xacro/robot.xacro (robot description, xacro)
@@ -1,4 +1,5 @@
 <?xml version="1.0"?>
 <robot name="ARX 5" xmlns:xacro="http://www.ros.org/wiki/xacro">
+  <xacro:arg name="collider" default="convex"/>
   <xacro:arg name="type" default="x5"/>
   <xacro:if value="${'$(arg type)' == 'r5'}">

File: arx_lift2s_description/xacro/components/ac_one.xacro (robot description, xacro)
@@ -1,5 +1,6 @@
 <?xml version="1.0" encoding="utf-8"?>
 <robot xmlns:xacro="http://www.ros.org/wiki/xacro">
-	<xacro:macro name="ac_one">
+	<xacro:property name="PI" value="3.1415926535897931"/>
+	<xacro:macro name="ac_one" params="name:='' direction:=1 collider:=convex">
 		<link name="body_link">
 			<inertial>
@@ -19,9 +20,31 @@
 				</geometry>
 			</visual>
-			<collision>
+<!--			<xacro:if value="${collider == 'convex'}">-->
+<!--				<collision>-->
+<!--					<geometry>-->
+<!--						<mesh filename="file://$(find arx_lift2s_description)/meshes/ac_one/base.glb"/>-->
+<!--					</geometry>-->
+<!--				</collision>-->
+<!--			</xacro:if>-->
+<!--			<xacro:if value="${collider == 'simple'}">-->
+			<collision name="simple_base1">
+				<origin xyz="0.002 0 -0.05" rpy="0 0 0"/>
 				<geometry>
-					<mesh filename="file://$(find arx_lift2s_description)/meshes/ac_one/base.glb"/>
+					<box size="0.14 0.6  0.1"/>
 				</geometry>
 			</collision>
+			<collision name="simple_base2">
+				<origin xyz="0.03 0 0.15" rpy="0 0 0"/>
+				<geometry>
+					<box size="0.04 0.06  0.3"/>
+				</geometry>
+			</collision>
+			<collision name="simple_base3">
+				<origin xyz="0.08 0 0.25" rpy="0 ${-PI/6} 0"/>
+				<geometry>
+					<box size="0.04 0.06  0.1"/>
+				</geometry>
+			</collision>
+<!--			</xacro:if>-->
 		</link>
 		<link name="head_camera">

File: arx_lift2s_description/xacro/robot.xacro (robot description, xacro)
@@ -3,4 +3,5 @@
 	<xacro:arg name="enable_wheel_joints" default="false"/>
 	<xacro:arg name="ros2_control_hardware_type" default="mock_components"/>
+<!--	<xacro:arg name="collider" defa ="convex"/>-->
 	<xacro:property name="type_arg" value="$(arg type)"/>
 	<xacro:property name="selected_arm_type" value="x5"/>

Commit message: AC One部分简单碰撞体已添加

File: arx5_description/xacro/X5.xacro (robot description, xacro)
@@ -2,5 +2,5 @@
 <robot xmlns:xacro="http://www.ros.org/wiki/xacro">
     <xacro:property name="PI" value="3.1415926535897931"/>
-    <xacro:macro name="X5" params="name camera:=d405">
+    <xacro:macro name="X5" params="name camera:=d405 collider:=convex">
         <xacro:property name="prefix" value="${name + '_' if name else ''}"/>
         <link name="${prefix}base_link">

File: arx5_description/xacro/robot.xacro (robot description, xacro)
@@ -9,5 +9,5 @@
   <xacro:if value="${'$(arg type)' == 'x5'}">
     <xacro:include filename="$(find arx5_description)/xacro/X5.xacro"/>
-    <xacro:X5 name=""/>
+    <xacro:X5 name="" collider="$(arg collider)"/>
   </xacro:if>
   <xacro:if value="${'$(arg type)' == 'agilex'}">

File: arx_lift2s_description/xacro/components/ac_one.xacro (robot description, xacro)
@@ -20,31 +20,31 @@
 				</geometry>
 			</visual>
-<!--			<xacro:if value="${collider == 'convex'}">-->
-<!--				<collision>-->
-<!--					<geometry>-->
-<!--						<mesh filename="file://$(find arx_lift2s_description)/meshes/ac_one/base.glb"/>-->
-<!--					</geometry>-->
-<!--				</collision>-->
-<!--			</xacro:if>-->
-<!--			<xacro:if value="${collider == 'simple'}">-->
-			<collision name="simple_base1">
-				<origin xyz="0.002 0 -0.05" rpy="0 0 0"/>
-				<geometry>
-					<box size="0.14 0.6  0.1"/>
-				</geometry>
-			</collision>
-			<collision name="simple_base2">
-				<origin xyz="0.03 0 0.15" rpy="0 0 0"/>
-				<geometry>
-					<box size="0.04 0.06  0.3"/>
-				</geometry>
-			</collision>
-			<collision name="simple_base3">
-				<origin xyz="0.08 0 0.25" rpy="0 ${-PI/6} 0"/>
-				<geometry>
-					<box size="0.04 0.06  0.1"/>
-				</geometry>
-			</collision>
-<!--			</xacro:if>-->
+			<xacro:if value="${collider == 'convex'}">
+				<collision>
+					<geometry>
+						<mesh filename="file://$(find arx_lift2s_description)/meshes/ac_one/base.glb"/>
+					</geometry>
+				</collision>
+			</xacro:if>
+			<xacro:if value="${collider == 'simple'}">
+				<collision name="simple_base1">
+					<origin xyz="0.002 0 -0.05" rpy="0 0 0"/>
+					<geometry>
+						<box size="0.14 0.6  0.1"/>
+					</geometry>
+				</collision>
+				<collision name="simple_base2">
+					<origin xyz="0.03 0 0.15" rpy="0 0 0"/>
+					<geometry>
+						<box size="0.04 0.06  0.3"/>
+					</geometry>
+				</collision>
+				<collision name="simple_base3">
+					<origin xyz="0.08 0 0.25" rpy="0 ${-PI/6} 0"/>
+					<geometry>
+						<box size="0.04 0.06  0.1"/>
+					</geometry>
+				</collision>
+			</xacro:if>
 		</link>
 		<link name="head_camera">

File: arx_lift2s_description/xacro/robot.xacro (robot description, xacro)
@@ -3,5 +3,5 @@
 	<xacro:arg name="enable_wheel_joints" default="false"/>
 	<xacro:arg name="ros2_control_hardware_type" default="mock_components"/>
-<!--	<xacro:arg name="collider" defa ="convex"/>-->
+	<xacro:arg name="collider" default ="convex"/>
 	<xacro:property name="type_arg" value="$(arg type)"/>
 	<xacro:property name="selected_arm_type" value="x5"/>
@@ -35,9 +35,9 @@
 	</xacro:unless>
 	<xacro:include filename="$(find arx_lift2s_description)/xacro/components/ac_one.xacro"/>
-	<xacro:ac_one/>
+	<xacro:ac_one collider="$(arg collider)"/>
 	<xacro:if value="${selected_arm_type == 'x5'}">
 		<xacro:include filename="$(find arx5_description)/xacro/X5.xacro"/>
-		<xacro:X5 name="left"/>
-		<xacro:X5 name="right"/>
+		<xacro:X5 name="left" collider="$(arg collider)"/>
+		<xacro:X5 name="right" collider="$(arg collider)"/>
 	</xacro:if>
 	<xacro:if value="${selected_arm_type == 'r5'}">

Commit message: AC_One简单碰撞体已添加

File: arx5_description/xacro/X5.xacro (robot description, xacro)
@@ -309,9 +309,12 @@
                 </geometry>
             </visual>
-            <collision>
-                <geometry>
-                    <mesh filename="file://$(find arx5_description)/meshes/x5/link7.obj"/>
-                </geometry>
-            </collision>
+            <xacro:if value="${collider == 'convex'}">
+                <collision>
+                    <geometry>
+                        <mesh filename="file://$(find arx5_description)/meshes/x5/link7.obj"/>
+                    </geometry>
+                </collision>
+            </xacro:if>
+            <xacro:if value="${collider == 'simple'}">
         </link>
         <joint name="${prefix}gripper_joint" type="prismatic">
