Commit message: fix camera config

File: arx5_description/xacro/X5.xacro (robot description, xacro)
@@ -193,5 +193,5 @@
             <xacro:if value="${collider == 'simple'}">
                 <collision name="simple_link4">
-                    <origin xyz="0.0685 0.0001 -0.065" rpy="0 0 0"/>
+                    <origin xyz="0.0685 0.0001 -0.065" />
                     <geometry>
                         <cylinder length="0.04" radius="0.0315"/>
@@ -220,5 +220,4 @@
             </inertial>
             <visual>
-                <origin xyz="0.0037 0 0"/>
                 <geometry>
                     <mesh filename="file://$(find arx5_description)/meshes/x5/link5.glb"/>
@@ -240,5 +239,5 @@
                 </collision>
                 <collision name="simple_link5_2">
-                    <origin xyz="0.0035 0 0.05" rpy="0 0 0"/>
+                    <origin xyz="0.0035 0 0.05" />
                     <geometry>
                         <cylinder length="0.013" radius="0.03145"/>
@@ -320,5 +319,5 @@
             <xacro:if value="${collider == 'simple'}">
                 <collision name="simple_link7">
-                    <origin xyz="0.0262 0 0.0002" rpy="0 0 0"/>
+                    <origin xyz="0.0262 0 0.0002" />
                     <geometry>
                         <box size="0.08 0.04 0.0640"/>
@@ -360,5 +359,5 @@
             <xacro:if value="${collider == 'simple'}">
                 <collision name="simple_link8">
-                    <origin xyz="0.0262 0 0.0002" rpy="0 0 0"/>
+                    <origin xyz="0.0262 0 0.0002" />
                     <geometry>
                         <box size="0.08 0.04 0.0640"/>
@@ -415,5 +414,5 @@
                     </collision>
                     <collision name="simple_d405_2">
-                        <origin xyz="0.001 0 0.014" rpy="0 0 0"/>
+                        <origin xyz="0.001 0 0.014" />
                         <geometry>
                             <box size="0.01 0.05 0.03"/>
@@ -442,5 +441,5 @@
                 <xacro:if value="${collider == 'simple'}">
                     <collision name="simple_d405camera">
-                        <origin xyz="-0.0115 0 0" rpy="0 0 0"/>
+                        <origin xyz="-0.0115 0 0" />
                         <geometry>
                             <box size="0.0231 0.0421 0.042"/>
@@ -471,5 +470,5 @@
                 <xacro:if value="${collider == 'simple'}">
                     <collision name="simple_d435">
-                        <origin xyz="0.001 0 0.014" rpy="0 0 0"/>
+                        <origin xyz="0.001 0 0.014" />
                         <geometry>
                             <box size="0.01 0.05 0.03"/>
@@ -496,5 +495,5 @@
                 <xacro:if value="${collider == 'simple'}">
                     <collision name="simple_d435camera">
-                        <origin xyz="-0.0125 0 0" rpy="0 0 0"/>
+                        <origin xyz="-0.0125 0 0" />
                         <geometry>
                             <box size="0.0251 0.0899 0.025"/>

File: arx5_description/xacro/X5_ac1.xacro (robot description, xacro)
@@ -124,5 +124,5 @@
 			<inertial>
 				<origin xyz="0.18544 -0.00071369 0.051628"/>
-				<mass value="0.54316" />
+				<mass value="0.54316"/>
 				<inertia
 						ixx="0.00036398"
@@ -131,5 +131,5 @@
 						iyy="0.00422770"
 						iyz="-0.00001179"
-						izz="0.00419421" />
+						izz="0.00419421"/>
 			</inertial>
 			<visual>
@@ -163,5 +163,5 @@
 		</link>
 		<joint name="${prefix}joint3" type="revolute">
-			<origin xyz="-0.264 0 0" rpy="0 0 0"/>
+			<origin xyz="-0.264 0 0"/>
 			<parent link="${prefix}link2"/>
 			<child link="${prefix}link3"/>
@@ -197,5 +197,5 @@
 			<xacro:if value="${collider == 'simple'}">
 				<collision name="simple_link4">
-					<origin xyz="0.0685 0.0001 0.065" rpy="0 0 0"/>
+					<origin xyz="0.0685 0.0001 0.065"/>
 					<geometry>
 						<cylinder length="0.04" radius="0.0315"/>
@@ -214,5 +214,5 @@
 			<inertial>
 				<origin xyz="0.0029491 8.4086E-05 -0.054795"/>
-				<mass value="0.67398" />
+				<mass value="0.67398"/>
 				<inertia
 						ixx="0.00092704"
@@ -221,5 +221,5 @@
 						iyy="0.00091568"
 						iyz="0.00000053"
-						izz="0.00028327" />
+						izz="0.00028327"/>
 			</inertial>
 			<visual>
@@ -243,5 +243,5 @@
 				</collision>
 				<collision name="simple_link5_2">
-					<origin xyz="0.0035 0 -0.05" rpy="0 0 0"/>
+					<origin xyz="0.0035 0 -0.05"/>
 					<geometry>
 						<cylinder length="0.013" radius="0.03145"/>
@@ -255,10 +255,10 @@
 			<child link="${prefix}link5"/>
 			<axis xyz="0 0 -1"/>
-			<limit lower="-1.671" upper="1.671" effort="7" velocity="20" />
+			<limit lower="-1.671" upper="1.671" effort="7" velocity="20"/>
 		</joint>
 		<link name="${prefix}link6">
 			<inertial>
 				<origin xyz="0.040212 3.4542E-05 -0.010225"/>
-				<mass value="0.34667" />
+				<mass value="0.34667"/>
 				<inertia
 						ixx="0.00047210"
@@ -267,5 +267,5 @@
 						iyy="0.00049011"
 						iyz="-0.00003393"
-						izz="0.00018496" />
+						izz="0.00018496"/>
 			</inertial>
 			<visual>
@@ -291,14 +291,14 @@
 		</link>
 		<joint name="${prefix}joint6" type="revolute">
-			<origin xyz="0.02895 0 -0.0845" />
+			<origin xyz="0.02895 0 -0.0845"/>
 			<parent link="${prefix}link5"/>
 			<child link="${prefix}link6"/>
 			<axis xyz="1 0 0"/>
-			<limit lower="-2.094" upper="2.094" effort="7" velocity="20" />
+			<limit lower="-2.094" upper="2.094" effort="7" velocity="20"/>
 		</joint>
 		<link name="${prefix}link7">
 			<inertial>
 				<origin xyz="-0.0060354 -0.015602 0.013499"/>
-				<mass value="0.08924" />
+				<mass value="0.08924"/>
 				<inertia
 						ixx="0.00009869"
@@ -307,5 +307,5 @@
 						iyy="0.00009021"
 						iyz="0.00001113"
-						izz="0.00006849" />
+						izz="0.00006849"/>
 			</inertial>
 			<visual>
@@ -323,5 +323,5 @@
 			<xacro:if value="${collider == 'simple'}">
 				<collision name="simple_link7">
-					<origin xyz="0.0262 0 0.0002" rpy="0 0 0"/>
+					<origin xyz="0.0262 0 0.0002"/>
 					<geometry>
 						<box size="0.08 0.04 0.0640"/>
@@ -340,5 +340,5 @@
 			<inertial>
 				<origin xyz="-0.00581 0.015593 -0.012255"/>
-				<mass value="0.089402" />
+				<mass value="0.089402"/>
 				<inertia
 						ixx="0.00007306"
@@ -347,5 +347,5 @@
 						iyy="0.00006428"
 						iyz="0.00000327"
-						izz="0.00006822" />
+						izz="0.00006822"/>
 			</inertial>
 			<visual>
@@ -363,5 +363,5 @@
 			<xacro:if value="${collider == 'simple'}">
 				<collision name="simple_link8">
-					<origin xyz="0.0262 0 0.0002" rpy="0 0 0"/>
+					<origin xyz="0.0262 0 0.0002"/>
 					<geometry>
 						<box size="0.08 0.04 0.0640"/>
@@ -418,5 +418,5 @@
 					</collision>
 					<collision name="simple_d405_2">
-						<origin xyz="0.001 0 0.014" rpy="0 0 0"/>
+						<origin xyz="0.001 0 0.014"/>
 						<geometry>
 							<box size="0.01 0.05 0.03"/>
@@ -428,5 +428,5 @@
 				<parent link="${prefix}link6"/>
 				<child link="${prefix}camera_support"/>
-				<origin xyz="0.045 0 0.021"/>
+				<origin xyz="0.0344 0 0.0208"/>
 			</joint>
 			<link name="${prefix}camera">
@@ -445,5 +445,5 @@
 				<xacro:if value="${collider == 'simple'}">
 					<collision name="simple_d405camera">
-						<origin xyz="-0.0115 0 0" rpy="0 0 0"/>
+						<origin xyz="-0.0115 0 0"/>
 						<geometry>
 							<box size="0.0231 0.0421 0.042"/>
@@ -474,5 +474,5 @@
 				<xacro:if value="${collider == 'simple'}">
 					<collision name="simple_d435">
-						<origin xyz="0.001 0 0.014" rpy="0 0 0"/>
+						<origin xyz="0.001 0 0.014"/>
 						<geometry>
 							<box size="0.01 0.05 0.03"/>
@@ -499,5 +499,5 @@
 				<xacro:if value="${collider == 'simple'}">
 					<collision name="simple_d435camera">
-						<origin xyz="-0.0125 0 0" rpy="0 0 0"/>
+						<origin xyz="-0.0125 0 0"/>
 						<geometry>
 							<box size="0.0251 0.0899 0.025"/>

Commit message: colliders fixed

File: arx5_description/xacro/X5.xacro (robot description, xacro)
@@ -194,5 +194,5 @@
             <xacro:if value="${collider == 'simple'}">
                 <collision name="simple_link4">
-                    <origin xyz="0.0685 0.0001 -0.065" />
+                    <origin xyz="0.068 0.00022 -0.067" />
                     <geometry>
                         <cylinder length="0.04" radius="0.0315"/>
@@ -234,13 +234,13 @@
             <xacro:if value="${collider == 'simple'}">
                 <collision name="simple_link5_1">
-                    <origin xyz="0.01 0 0.086" rpy="${PI/2} 0 ${PI/2}"/>
-                    <geometry>
-                        <cylinder length="0.045" radius="0.03145"/>
+                    <origin xyz="0.006 0 0.086" rpy="${PI/2} 0 ${PI/2}"/>
+                    <geometry>
+                        <cylinder length="0.047" radius="0.03145"/>
                     </geometry>
                 </collision>
                 <collision name="simple_link5_2">
-                    <origin xyz="0.0035 0 0.05" />
-                    <geometry>
-                        <cylinder length="0.013" radius="0.03145"/>
+                    <origin xyz="0.00038 -0.0003 0.048" />
+                    <geometry>
+                        <cylinder length="0.014" radius="0.03145"/>
                     </geometry>
                 </collision>

File: arx5_description/xacro/X5_ac1.xacro (robot description, xacro)
@@ -198,5 +198,5 @@
 			<xacro:if value="${collider == 'simple'}">
 				<collision name="simple_link4">
-					<origin xyz="0.0685 0.0001 0.065"/>
+					<origin xyz="0.0679 -0.00045 0.067"/>
 					<geometry>
 						<cylinder length="0.04" radius="0.0315"/>
@@ -238,5 +238,5 @@
 			<xacro:if value="${collider == 'simple'}">
 				<collision name="simple_link5_1">
-					<origin xyz="0.01 0 -0.086" rpy="${PI/2} 0 ${PI/2}"/>
+					<origin xyz="0.006 0 -0.0845" rpy="${PI/2} 0 ${PI/2}"/>
 					<geometry>
 						<cylinder length="0.045" radius="0.03145"/>
@@ -244,7 +244,7 @@
 				</collision>
 				<collision name="simple_link5_2">
-					<origin xyz="0.0035 0 -0.05"/>
-					<geometry>
-						<cylinder length="0.013" radius="0.03145"/>
+					<origin xyz="0.000375 -0.000265 -0.047"/>
+					<geometry>
+						<cylinder length="0.014" radius="0.0315"/>
 					</geometry>
 				</collision>

File: arx5_description/xacro/components/camera.xacro (robot description, xacro)
@@ -29,5 +29,5 @@
                         <origin xyz="0.001 0 0.014" rpy="0 0 0"/>
                         <geometry>
-                            <box size="0.01 0.05 0.03"/>
+                            <box size="0.01 0.057 0.03"/>
                         </geometry>
                     </collision>
@@ -49,5 +49,5 @@
                 <xacro:if value="${collider == 'simple'}">
                     <collision name="simple_d405camera">
-                        <origin xyz="-0.0115 0 0" rpy="0 0 0"/>
+                        <origin xyz="0 0 -0.0115" rpy="0 ${PI/2} 0"/>
                         <geometry>
                             <box size="0.0231 0.0421 0.042"/>

File: arx5_description/xacro/components/gripper_2023.xacro (robot description, xacro)
@@ -22,8 +22,14 @@
             </xacro:if>
             <xacro:if value="${collider == 'simple'}">
-                <collision name="simple_link6">
+                <collision name="simple_link6_1">
                     <origin xyz="0.038 0 0.0002" rpy="0 ${PI/2} 0"/>
                     <geometry>
                         <cylinder length="0.064" radius="0.03015"/>
+                    </geometry>
+                </collision>
+                <collision name="simple_link6_2">
+                    <origin xyz="0.0705 0 -0.0012" rpy="0 0 0"/>
+                    <geometry>
+                        <box size="0.01 0.178 0.015"/>
                     </geometry>
                 </collision>
@@ -52,4 +58,12 @@
                 </collision>
             </xacro:if>
+            <xacro:if value="${collider == 'simple'}">
+                <collision name="simple_link7">
+                    <origin xyz="0.038 -0.0125 0.0002" rpy="0 0 ${PI/2}"/>
+                    <geometry>
+                        <box size="0.0231 0.07 0.042"/>
+                    </geometry>
+                </collision>
+            </xacro:if>
         </link>
         <joint name="${prefix}gripper_joint" type="prismatic">
@@ -75,4 +89,12 @@
                     <geometry>
                         <mesh filename="file://$(find arx5_description)/meshes/r5/link8.glb"/>
+                    </geometry>
+                </collision>
+            </xacro:if>
+            <xacro:if value="${collider == 'simple'}">
+                <collision name="simple_link8">
+                    <origin xyz="0.038 0.0125 0.0002" rpy="0 0 ${PI/2}"/>
+                    <geometry>
+                        <box size="0.0231 0.07 0.042"/>
                     </geometry>
                 </collision>

File: arx5_description/xacro/components/gripper_2025.xacro (robot description, xacro)
@@ -18,4 +18,18 @@
                     <geometry>
                         <mesh filename="file://$(find arx5_description)/meshes/ac1/link6.glb"/>
+                    </geometry>
+                </collision>
+            </xacro:if>
+            <xacro:if value="${collider == 'simple'}">
+                <collision name="simple_link6_1">
+                    <origin xyz="0.038 0 0.0002" rpy="0 ${PI/2} 0"/>
+                    <geometry>
+                        <cylinder length="0.064" radius="0.025"/>
+                    </geometry>
+                </collision>
+                <collision name="simple_link6_2">
+                    <origin xyz="0.063 0 -0.0012" rpy="0 0 0"/>
+                    <geometry>
+                        <box size="0.007 0.07 0.07"/>
                     </geometry>
                 </collision>
@@ -44,4 +58,12 @@
                 </collision>
             </xacro:if>
+            <xacro:if value="${collider == 'simple'}">
+                <collision name="simple_link7">
+                    <origin xyz="0.038 -0.0125 0.00025" rpy="0 0 ${PI/2}"/>
+                    <geometry>
+                        <box size="0.0231 0.07 0.042"/>
+                    </geometry>
+                </collision>
+            </xacro:if>
         </link>
         <joint name="${prefix}gripper_joint" type="prismatic">
@@ -67,4 +89,12 @@
                     <geometry>
                         <mesh filename="file://$(find arx5_description)/meshes/ac1/link8.glb"/>
+                    </geometry>
+                </collision>
+            </xacro:if>
+            <xacro:if value="${collider == 'simple'}">
+                <collision name="simple_link8">
+                    <origin xyz="0.038 0.0125 0.00025" rpy="0 0 ${PI/2}"/>
+                    <geometry>
+                        <box size="0.0231 0.07 0.042"/>
                     </geometry>
                 </collision>
