Commit message: fix arx lift fullbody control

File: arx_acone_description/xacro/arm_mount.xacro (robot description, xacro)
@@ -10,19 +10,31 @@
 		</joint>
 	</xacro:macro>
-	<!-- Mount dual arms onto an existing parent link (typically arm_base). -->
-	<xacro:macro name="DualArmMount" params="parent:=arm_base">
+	<!-- Mount dual arms onto parent (typically arm_base). Defaults = AC One 原厂安装位姿。 -->
+	<xacro:macro name="DualArmMount" params="
+		parent:=arm_base
+		left_xyz:='-0.01602 0.25 -0.035'
+		right_xyz:='-0.01602 -0.25 -0.035'
+		left_rpy:='0 0 0'
+		right_rpy:='0 0 0'
+	">
 		<joint name="arm_left_fixed" type="fixed">
 			<parent link="${parent}"/>
 			<child link="left_base_link"/>
-			<origin xyz="-0.01602 0.25 -0.035"/>
+			<origin xyz="${left_xyz}" rpy="${left_rpy}"/>
 		</joint>
 		<joint name="arm_right_fixed" type="fixed">
 			<parent link="${parent}"/>
 			<child link="right_base_link"/>
-			<origin xyz="-0.01602 -0.25 -0.035"/>
+			<origin xyz="${right_xyz}" rpy="${right_rpy}"/>
 		</joint>
 	</xacro:macro>
-	<!-- Standalone base + torso + arm_base for component visualization. -->
-	<xacro:macro name="DualArmBase" params="collider:=simple">
+	<!-- Standalone base + torso + arm_base（带 AC One 底座）。 -->
+	<xacro:macro name="DualArmBase" params="
+		collider:=simple
+		left_xyz:='-0.01602 0.25 -0.035'
+		right_xyz:='-0.01602 -0.25 -0.035'
+		left_rpy:='0 0 0'
+		right_rpy:='0 0 0'
+	">
 		<link name="base_link"/>
 		<joint name="base_joint" type="fixed">
@@ -33,5 +45,46 @@
 		<xacro:ac_one collider="${collider}"/>
 		<xacro:ArmBase parent="body_link"/>
-		<xacro:DualArmMount parent="arm_base"/>
+		<xacro:DualArmMount parent="arm_base"
+			left_xyz="${left_xyz}" right_xyz="${right_xyz}"
+			left_rpy="${left_rpy}" right_rpy="${right_rpy}"/>
+	</xacro:macro>
+	<!-- 展台 / 无 AC One 躯干：base_link + arm_base（同 m6_ccs variant:=desktop）。 -->
+	<xacro:macro name="DesktopArmBase" params="
+		left_xyz:='-0.01602 0.25 0.0'
+		right_xyz:='-0.01602 -0.25 0.0'
+		left_rpy:='0 0 0'
+		right_rpy:='0 0 0'
+		arm_base_xyz:='0 0 0.35'
+	">
+		<link name="base_link"/>
+		<link name="arm_base">
+			<visual>
+				<origin xyz="0 0 -0.175"/>
+				<geometry>
+					<box size="0.20 0.55 0.35"/>
+				</geometry>
+			</visual>
+			<collision>
+				<origin xyz="0 0 -0.175"/>
+				<geometry>
+					<box size="0.20 0.55 0.35"/>
+				</geometry>
+			</collision>
+		</link>
+		<joint name="arm_base_joint" type="fixed">
+			<parent link="base_link"/>
+			<child link="arm_base"/>
+			<origin xyz="${arm_base_xyz}"/>
+		</joint>
+		<!-- 规划 / 碰撞参考（无 AC One mesh） -->
+		<link name="body_link"/>
+		<joint name="arm_base_body" type="fixed">
+			<parent link="arm_base"/>
+			<child link="body_link"/>
+			<origin xyz="0 0 0"/>
+		</joint>
+		<xacro:DualArmMount parent="arm_base"
+			left_xyz="${left_xyz}" right_xyz="${right_xyz}"
+			left_rpy="${left_rpy}" right_rpy="${right_rpy}"/>
 	</xacro:macro>
 </robot>

File: arx_acone_description/xacro/component.xacro (robot description, xacro)
@@ -19,3 +19,10 @@
 		<xacro:X5 name="right" collider="$(arg collider)"/>
 	</xacro:if>
+	<xacro:if value="${'$(arg type)' == 'desktop'}">
+		<xacro:include filename="$(find arx_acone_description)/xacro/arm_mount.xacro"/>
+		<xacro:DesktopArmBase/>
+		<xacro:include filename="$(find arx5_description)/xacro/X5_ac1.xacro"/>
+		<xacro:X5 name="left" collider="$(arg collider)"/>
+		<xacro:X5 name="right" collider="$(arg collider)"/>
+	</xacro:if>
 </robot>

File: arx_acone_description/xacro/robot.xacro (robot description, xacro)
@@ -1,20 +1,61 @@
 <?xml version="1.0"?>
 <robot name="arx_acone" xmlns:xacro="http://www.ros.org/wiki/xacro">
+	<!-- type: 臂型 x5|r5（与末端无关） -->
 	<xacro:arg name="type" default="x5"/>
+	<!-- variant: acone=带 AC One 躯干（默认）；desktop=展台底座（无 AC One mesh） -->
+	<xacro:arg name="variant" default="acone"/>
 	<xacro:arg name="collider" default="simple"/>
 	<xacro:arg name="ros2_control_hardware_type" default="mock_components"/>
+	<!-- 双臂安装位姿（空=按 variant 默认；可覆盖间距，同 m6 left_xyz/right_xyz） -->
+	<xacro:arg name="left_xyz" default=""/>
+	<xacro:arg name="right_xyz" default=""/>
+	<xacro:arg name="left_rpy" default="0 0 0"/>
+	<xacro:arg name="right_rpy" default="0 0 0"/>
+	<!-- desktop 时 arm_base 相对 base_link 高度 -->
+	<xacro:arg name="arm_base_xyz" default="0 0 0.35"/>
 	<xacro:property name="type_arg" value="$(arg type)"/>
+	<xacro:property name="variant_raw" value="$(arg variant)"/>
+	<!-- 空字符串兼容旧 launch，视为 acone -->
+	<xacro:property name="variant_arg" value="${'acone' if variant_raw == '' else variant_raw}"/>
 	<xacro:property name="selected_arm_type" value="x5"/>
 	<xacro:if value="${type_arg == 'r5'}">
 		<xacro:property name="selected_arm_type" value="r5"/>
 	</xacro:if>
-	<!-- Fixed-base dual-arm torso (no lift chassis) -->
-	<link name="base_link"/>
-	<joint name="base_joint" type="fixed">
-		<parent link="base_link"/>
-		<child link="body_link"/>
-	</joint>
-	<xacro:include filename="$(find arx_acone_description)/xacro/components/ac_one.xacro"/>
-	<xacro:ac_one collider="$(arg collider)"/>
+	<!-- 默认安装：AC One 原厂；desktop 默认 z=0（相对 arm_base） -->
+	<xacro:property name="default_left_xyz" value="-0.01602 0.25 -0.035"/>
+	<xacro:property name="default_right_xyz" value="-0.01602 -0.25 -0.035"/>
+	<xacro:if value="${variant_arg == 'desktop'}">
+		<xacro:property name="default_left_xyz" value="-0.01602 0.25 0.0"/>
+		<xacro:property name="default_right_xyz" value="-0.01602 -0.25 0.0"/>
+	</xacro:if>
+	<xacro:property name="left_xyz_arg" value="$(arg left_xyz)"/>
+	<xacro:property name="right_xyz_arg" value="$(arg right_xyz)"/>
+	<xacro:property name="effective_left_xyz"
+		value="${left_xyz_arg if left_xyz_arg != '' else default_left_xyz}"/>
+	<xacro:property name="effective_right_xyz"
+		value="${right_xyz_arg if right_xyz_arg != '' else default_right_xyz}"/>
+	<xacro:include filename="$(find arx_acone_description)/xacro/arm_mount.xacro"/>
+	<!-- ===== desktop：展台底座，无 AC One ===== -->
+	<xacro:if value="${variant_arg == 'desktop'}">
+		<xacro:DesktopArmBase
+			left_xyz="${effective_left_xyz}" right_xyz="${effective_right_xyz}"
+			left_rpy="$(arg left_rpy)" right_rpy="$(arg right_rpy)"
+			arm_base_xyz="$(arg arm_base_xyz)"/>
+	</xacro:if>
+	<!-- ===== acone：带 AC One 躯干 ===== -->
+	<xacro:if value="${variant_arg == 'acone'}">
+		<link name="base_link"/>
+		<joint name="base_joint" type="fixed">
+			<parent link="base_link"/>
+			<child link="body_link"/>
+		</joint>
+		<xacro:include filename="$(find arx_acone_description)/xacro/components/ac_one.xacro"/>
+		<xacro:ac_one collider="$(arg collider)"/>
+		<xacro:ArmBase parent="body_link"/>
+		<xacro:DualArmMount parent="arm_base"
+			left_xyz="${effective_left_xyz}" right_xyz="${effective_right_xyz}"
+			left_rpy="$(arg left_rpy)" right_rpy="$(arg right_rpy)"/>
+	</xacro:if>
+	<!-- 双臂 -->
 	<xacro:if value="${selected_arm_type == 'x5'}">
 		<xacro:include filename="$(find arx5_description)/xacro/X5_ac1.xacro"/>
@@ -27,6 +68,3 @@
 		<xacro:R5 name="right" collider="$(arg collider)"/>
 	</xacro:if>
-	<xacro:include filename="$(find arx_acone_description)/xacro/arm_mount.xacro"/>
-	<xacro:ArmBase parent="body_link"/>
-	<xacro:DualArmMount parent="arm_base"/>
 </robot>

File: arx_lift_description/xacro/components/body.xacro (robot description, xacro)
@@ -1,6 +1,6 @@
 <?xml version="1.0" encoding="utf-8"?>
 <robot xmlns:xacro="http://www.ros.org/wiki/xacro">
+    <!-- 仅升降柱；头见 head.xacro（须在双臂之后展开，以匹配 WBC 关节序 lift|L|R|head） -->
     <xacro:macro name="Body">
-        <xacro:property name="PI" value="3.1415926535897931"/>
         <link name="lift_link">
             <inertial>
@@ -27,98 +27,4 @@
             <limit effort="1000" lower="0.0" upper="0.86" velocity="100"/>
         </joint>
-        <link name="h_base_link">
-            <inertial>
-                <origin xyz="-0.0020743076738515215 0 0.024619861716967787"/>
-                <mass value="0.9930933606993821"/>
-                <inertia ixx="0.000391" ixy="-0.0" ixz="1.7e-05" iyy="0.000452" iyz="0.0" izz="0.000532"/>
-            </inertial>
-            <visual>
-                <geometry>
-                    <mesh filename="file://$(find arx_lift_description)/meshes/body/h_base.obj"/>
-                </geometry>
-            </visual>
-            <collision>
-                <geometry>
-                    <mesh filename="file://$(find arx_lift_description)/meshes/body/h_base.obj"/>
-                </geometry>
-            </collision>
-        </link>
-        <link name="head_link1">
-            <inertial>
-                <origin xyz="-1.2166451790474E-08 0.000155101086835956 0.0414775143344981"/>
-                <mass value="0.429406588376073"/>
-                <inertia
-                        ixx="0.00027"
-                        ixy="0.00000"
-                        ixz="0.00000"
-                        iyy="0.00026"
-                        iyz="-0.00001"
-                        izz="0.00018"/>
-            </inertial>
-            <visual>
-                <geometry>
-                    <mesh filename="file://$(find arx_lift_description)/meshes/body/neck.obj"/>
-                </geometry>
-            </visual>
-            <collision>
-                <geometry>
-                    <mesh filename="file://$(find arx_lift_description)/meshes/body/neck.obj"/>
-                </geometry>
-            </collision>
-        </link>
-        <link name="head_link2">
-            <inertial>
-                <origin xyz="0.0145474612596931 0.0229595215513494 0.0787914285814235"/>
-                <mass value="1.54420437039843"/>
-                <inertia
-                        ixx="0.00576"
-                        ixy="-0.00007"
-                        ixz="0.00018"
-                        iyy="0.00477"
-                        iyz="0.00015"
-                        izz="0.00768"/>
-            </inertial>
-            <visual>
-                <geometry>
-                    <mesh filename="file://$(find arx_lift_description)/meshes/body/head.obj"/>
-                </geometry>
-            </visual>
-            <collision>
-                <geometry>
-                    <mesh filename="file://$(find arx_lift_description)/meshes/body/head.obj"/>
-                </geometry>
-            </collision>
-        </link>
-        <joint name="head_joint1" type="continuous">
-            <origin xyz="0.0 0.0 0.046"/>
-            <parent link="h_base_link"/>
-            <child link="head_link1"/>
-            <axis xyz="0.0 0.0 1.0"/>
-            <limit effort="100" lower="${-PI/2}" upper="${PI/2}" velocity="100"/>
-        </joint>
-        <joint name="head_joint2" type="continuous">
-            <origin xyz="0.0 -0.025 0.049"/>
-            <parent link="head_link1"/>
-            <child link="head_link2"/>
-            <axis xyz="0.0 -1.0 0.0"/>
-            <limit effort="100" lower="${-PI/4}" upper="${PI/4}" velocity="100"/>
-        </joint>
-        <joint name="h_fixed" type="fixed">
-            <parent link="lift_link"/>
-            <child link="h_base_link"/>
-            <origin xyz="0.258786 0 0.220008"/>
-        </joint>
-        <link name="head_camera">
-            <visual>
-                <geometry>
-                    <mesh filename="file://$(find sensor_models)/meshes/realsense/d405.glb"/>
-                </geometry>
-            </visual>
-        </link>
-        <joint name="head_camera_joint" type="fixed">
-            <origin xyz="0.095 0.025 0.06" rpy="-1.5708 0 -1.5708"/>
-            <parent link="head_link2"/>
-            <child link="head_camera"/>
-        </joint>
     </xacro:macro>
 </robot>

File: arx_lift_description/xacro/robot.xacro (robot description, xacro)
@@ -1,32 +1,89 @@
 <?xml version="1.0" ?>
 <robot name="arx_lift" xmlns:xacro="http://www.ros.org/wiki/xacro">
+  <!-- topology:
+       full (default) = 底盘 + 升降 + 双臂 + 头（全身 / 真机 / 可视化）
+       dual           = 仅双臂，根在 arm_base（分体 OCS2 规划，同 m6_ccs）
+       全身 Pinocchio / WBC 关节序须为：lift | left×6 | right×6 | head×2 -->
+  <xacro:arg name="topology" default="full"/>
   <xacro:arg name="type" default="x5"/>
   <xacro:arg name="enable_wheel_joints" default="false"/>
-  <!-- 根据type参数包含不同的机械臂描述文件 -->
-  <xacro:if value="${'$(arg type)' == 'x5'}">
-    <xacro:include filename="$(find arx5_description)/xacro/X5.xacro"/>
-    <!-- 使用R5宏来创建两个机械臂 -->
-    <xacro:X5 name="left"/>
-    <xacro:X5 name="right"/>
+  <xacro:property name="topology_arg" value="$(arg topology)"/>
+  <xacro:property name="type_arg" value="$(arg type)"/>
+  <xacro:property name="selected_arm_type" value="x5"/>
+  <xacro:if value="${type_arg == 'r5'}">
+    <xacro:property name="selected_arm_type" value="r5"/>
   </xacro:if>
-  <xacro:if value="${'$(arg type)' == 'r5'}">
-    <xacro:include filename="$(find arx5_description)/xacro/R5.xacro"/>
-    <!-- 使用R5宏来创建两个机械臂 -->
-    <xacro:R5 name="left"/>
-    <xacro:R5 name="right"/>
+  <!-- ===== dual：仅双臂（分体规划，根 = arm_base，同 m6_ccs） ===== -->
+  <xacro:if value="${topology_arg == 'dual'}">
+    <link name="arm_base"/>
+    <link name="body_link"/>
+    <joint name="arm_base_body" type="fixed">
+      <parent link="arm_base"/>
+      <child link="body_link"/>
+      <origin xyz="0 0 0"/>
+    </joint>
+    <xacro:if value="${selected_arm_type == 'x5'}">
+      <xacro:include filename="$(find arx5_description)/xacro/X5.xacro"/>
+      <xacro:X5 name="left"/>
+      <xacro:X5 name="right"/>
+    </xacro:if>
+    <xacro:if value="${selected_arm_type == 'r5'}">
+      <xacro:include filename="$(find arx5_description)/xacro/R5.xacro"/>
+      <xacro:R5 name="left"/>
+      <xacro:R5 name="right"/>
+    </xacro:if>
+    <joint name="arm_left_fixed" type="fixed">
+      <parent link="arm_base"/>
+      <child link="left_base_link"/>
+      <origin xyz="0.208 0.25000 0.092"/>
+    </joint>
+    <joint name="arm_right_fixed" type="fixed">
+      <parent link="arm_base"/>
+      <child link="right_base_link"/>
+      <origin xyz="0.208 -0.25000 0.092"/>
+    </joint>
   </xacro:if>
-  <xacro:include filename="$(find arx_lift_description)/xacro/components/mobile_base.xacro"/>
-  <xacro:include filename="$(find arx_lift_description)/xacro/components/body.xacro"/>
-  <xacro:MobileBase enable_wheel_joints="$(arg enable_wheel_joints)"/>
-  <xacro:Body/>
-  <joint name="arm_left_fixed" type="fixed">
-    <parent link="lift_link"/>
-    <child link="left_base_link"/>
-    <origin  xyz="0.208 0.25000 0.092"/>
-  </joint>
-  <joint name="arm_right_fixed" type="fixed">
-    <parent link="lift_link"/>
-    <child link="right_base_link"/>
-    <origin xyz="0.208 -0.25000 0.092"/>
-  </joint>
+  <!-- ===== full：整机（升降 → 双臂 → 头，匹配 WBC 布局） ===== -->
+  <xacro:unless value="${topology_arg == 'dual'}">
+    <xacro:include filename="$(find arx_lift_description)/xacro/components/mobile_base.xacro"/>
+    <xacro:include filename="$(find arx_lift_description)/xacro/components/body.xacro"/>
+    <xacro:include filename="$(find arx_lift_description)/xacro/components/head.xacro"/>
+    <xacro:MobileBase enable_wheel_joints="$(arg enable_wheel_joints)"/>
+    <xacro:Body/>
+    <!-- 臂座：与 lift_link 固连 -->
+    <link name="body_link"/>
+    <joint name="body_fixed" type="fixed">
+      <parent link="lift_link"/>
+      <child link="body_link"/>
+      <origin xyz="0 0 0"/>
+    </joint>
+    <link name="arm_base"/>
+    <joint name="arm_base_joint" type="fixed">
+      <parent link="lift_link"/>
+      <child link="arm_base"/>
+      <origin xyz="0 0 0"/>
+    </joint>
+    <xacro:if value="${selected_arm_type == 'x5'}">
+      <xacro:include filename="$(find arx5_description)/xacro/X5.xacro"/>
+      <xacro:X5 name="left"/>
+      <xacro:X5 name="right"/>
+    </xacro:if>
+    <xacro:if value="${selected_arm_type == 'r5'}">
+      <xacro:include filename="$(find arx5_description)/xacro/R5.xacro"/>
+      <xacro:R5 name="left"/>
+      <xacro:R5 name="right"/>
+    </xacro:if>
+    <joint name="arm_left_fixed" type="fixed">
+      <parent link="arm_base"/>
+      <child link="left_base_link"/>
+      <origin xyz="0.208 0.25000 0.092"/>
+    </joint>
+    <joint name="arm_right_fixed" type="fixed">
+      <parent link="arm_base"/>
+      <child link="right_base_link"/>
+      <origin xyz="0.208 -0.25000 0.092"/>
+    </joint>
+    <!-- 头放在双臂之后，Pinocchio 序 = lift | L6 | R6 | head×2 -->
+    <xacro:Head/>
+  </xacro:unless>
 </robot>

File: arx_lift_description/xacro/ros2_control/interfaces.xacro (robot description, xacro)
@@ -1,15 +1,21 @@
 <?xml version="1.0"?>
 <robot xmlns:xacro="http://www.ros.org/wiki/xacro">
-	<xacro:macro name="lift_interfaces">
-		<!-- 升降机构关节 -->
+	<!-- iface_mode: mix = pos/vel/effort（mock/gz）；position = 仅 position（Isaac） -->
+	<xacro:macro name="lift_interfaces" params="iface_mode:=mix">
 		<joint name="lift_joint">
 			<command_interface name="position"/>
+			<xacro:if value="${iface_mode == 'mix'}">
+				<command_interface name="velocity"/>
+				<command_interface name="effort"/>
+			</xacro:if>
 			<state_interface name="position">
 				<param name="initial_value">0.3</param>
 			</state_interface>
-			<state_interface name="velocity"/>
-			<state_interface name="effort"/>
+			<xacro:if value="${iface_mode == 'mix'}">
+				<state_interface name="velocity"/>
+				<state_interface name="effort"/>
+			</xacro:if>
 		</joint>
-		<!-- 头部关节1 -->
+		<!-- 头：仅 position；当前不进 WBC / body 控制器 -->
 		<joint name="head_joint1">
 			<command_interface name="position"/>
@@ -18,5 +24,4 @@
 			<state_interface name="effort"/>
 		</joint>
-		<!-- 头部关节2 -->
 		<joint name="head_joint2">
 			<command_interface name="position"/>

File: arx_lift_description/xacro/ros2_control/robot.xacro (robot description, xacro)
@@ -1,7 +1,12 @@
 <?xml version="1.0"?>
 <robot xmlns:xacro="http://www.ros.org/wiki/xacro" name="arx_lift">
+  <xacro:arg name="ros2_control_hardware_type" default="mock_components"/>
+  <xacro:arg name="gazebo" default="false"/>
   <xacro:include filename="$(find arx_lift_description)/xacro/robot.xacro"/>
   <xacro:include filename="$(find arx5_description)/xacro/ros2_control/interfaces.xacro"/>
   <xacro:include filename="$(find arx_lift_description)/xacro/ros2_control/interfaces.xacro"/>
+  <!-- 硬件描述始终用 full 拓扑（分体规划 dual 只影响 planning URDF） -->
+  <xacro:property name="sim_iface_mode"
+    value="${'position' if '$(arg ros2_control_hardware_type)' == 'isaac' else 'mix'}"/>
   <ros2_control name="arx_lift_unified_system" type="system">
     <hardware>
@@ -18,10 +23,8 @@
       </xacro:if>
     </hardware>
-    <xacro:lift_interfaces/>
-    <xacro:arx5_interfaces name="left"/>
-    <xacro:arx5_interfaces name="right"/>
+    <xacro:lift_interfaces iface_mode="${sim_iface_mode}"/>
+    <xacro:arx5_interfaces name="left" iface_mode="${sim_iface_mode}"/>
+    <xacro:arx5_interfaces name="right" iface_mode="${sim_iface_mode}"/>
   </ros2_control>
-  <!-- Gazebo插件配置 -->
-  <xacro:arg name="gazebo" default="false" />
   <xacro:if value="$(arg gazebo)">
     <gazebo>
