Commit message: fix arx camera direction

File: arx5_description/xacro/components/camera.xacro (robot description, xacro)
@@ -88,5 +88,5 @@
                 <visual>
                     <geometry>
-                        <mesh filename="file://$(find sensor_models)/meshes/d435/d435.obj"/>
+                        <mesh filename="file://$(find sensor_models)/meshes/realsense/d435.glb"/>
                     </geometry>
                 </visual>
@@ -94,5 +94,5 @@
                     <collision>
                         <geometry>
-                            <mesh filename="file://$(find sensor_models)/meshes/d435/d435.obj"/>
+                            <mesh filename="file://$(find sensor_models)/meshes/realsense/d435.glb"/>
                         </geometry>
                     </collision>
@@ -100,7 +100,7 @@
                 <xacro:if value="${collider == 'simple'}">
                     <collision name="simple_d435camera">
-                        <origin xyz="-0.0125 0 0" rpy="0 0 0"/>
+                        <origin xyz="0 0 -0.0125" rpy="0 0 0"/>
                         <geometry>
-                            <box size="0.0251 0.0899 0.025"/>
+                            <box size="0.0899 0.025 0.0251"/>
                         </geometry>
                     </collision>
@@ -108,5 +108,5 @@
             </link>
             <joint name="${prefix}camera_fixed" type="fixed">
-                <origin xyz="0.03 0 0.034113"/>
+                <origin xyz="0.03 0 0.034113" rpy="-1.5708 0 -1.5708"/>
                 <parent link="${prefix}camera_support"/>
                 <child link="${prefix}camera"/>
