Commit message: add sepetate acone package

File: arx_acone_description/xacro/components/ac_one.xacro (robot description, xacro)
@@ -17,5 +17,5 @@
 			<visual>
 				<geometry>
-					<mesh filename="file://$(find arx_lift2s_description)/meshes/ac_one/base.glb"/>
+					<mesh filename="file://$(find arx_acone_description)/meshes/ac_one/base.glb"/>
 				</geometry>
 			</visual>
@@ -23,5 +23,5 @@
 				<collision>
 					<geometry>
-						<mesh filename="file://$(find arx_lift2s_description)/meshes/ac_one/base.glb"/>
+						<mesh filename="file://$(find arx_acone_description)/meshes/ac_one/base.glb"/>
 					</geometry>
 				</collision>
@@ -56,5 +56,4 @@
 		</link>
 		<joint name="head_camera_joint" type="fixed">
-<!--			<origin xyz="0.090415 0.002 0.2285" rpy="0 1.0472 0"/>-->
 			<origin xyz="0.090415 0.002 0.2285" rpy="-2.618 0 -1.5708"/>
 			<parent link="body_link"/>

File: arx_acone_description/xacro/robot.xacro (robot description, xacro)
@@ -1,7 +1,7 @@
-<robot name="arx_lift2s" xmlns:xacro="http://www.ros.org/wiki/xacro">
+<?xml version="1.0"?>
+<robot name="arx_acone" xmlns:xacro="http://www.ros.org/wiki/xacro">
 	<xacro:arg name="type" default="x5"/>
-	<xacro:arg name="enable_wheel_joints" default="false"/>
+	<xacro:arg name="collider" default="simple"/>
 	<xacro:arg name="ros2_control_hardware_type" default="mock_components"/>
-	<xacro:arg name="collider" default="simple"/>
 	<xacro:property name="type_arg" value="$(arg type)"/>
 	<xacro:property name="selected_arm_type" value="x5"/>
@@ -9,13 +9,10 @@
 		<xacro:property name="selected_arm_type" value="r5"/>
 	</xacro:if>
-	<!-- Lift chassis + prismatic lift_joint -->
-	<xacro:include filename="$(find arx_lift2s_description)/xacro/components/chassis.xacro"/>
-	<xacro:chassis enable_wheel_joints="$(arg enable_wheel_joints)"/>
-	<joint name="body_joint" type="fixed">
-		<origin xyz="0.13 0.001801 0.0529"/>
-		<parent link="lift_link"/>
+	<!-- Fixed-base dual-arm torso (no lift chassis) -->
+	<link name="base_link"/>
+	<joint name="base_joint" type="fixed">
+		<parent link="base_link"/>
 		<child link="body_link"/>
 	</joint>
-	<!-- AC One torso + dual arms from arx_acone_description -->
 	<xacro:include filename="$(find arx_acone_description)/xacro/components/ac_one.xacro"/>
 	<xacro:ac_one collider="$(arg collider)"/>

File: arx_acone_description/xacro/ros2_control/robot.xacro (robot description, xacro)
@@ -1,12 +1,10 @@
 <?xml version="1.0"?>
-<robot xmlns:xacro="http://www.ros.org/wiki/xacro" name="arx_lift2s">
+<robot xmlns:xacro="http://www.ros.org/wiki/xacro" name="arx_acone">
 	<xacro:arg name="ros2_control_hardware_type" default="mock_components"/>
 	<xacro:arg name="gazebo" default="false"/>
-	<xacro:include filename="$(find arx_lift2s_description)/xacro/robot.xacro"/>
+	<xacro:include filename="$(find arx_acone_description)/xacro/robot.xacro"/>
 	<xacro:include filename="$(find arx5_description)/xacro/ros2_control/interfaces.xacro"/>
-	<xacro:include filename="$(find arx_lift2s_description)/xacro/ros2_control/interfaces.xacro"/>
 	<xacro:if value="${'$(arg ros2_control_hardware_type)' == 'real'}">
-		<!-- Dual arms: official LIFT2S X5 HW (can1 / can3) -->
-		<ros2_control name="arx_lift2s_left_system" type="system">
+		<ros2_control name="arx_acone_left_system" type="system">
 			<hardware>
 				<plugin>arxlift2s_ros2_control/ArxX5Hardware</plugin>
@@ -18,5 +16,5 @@
 			<xacro:arx5_interfaces name="left"/>
 		</ros2_control>
-		<ros2_control name="arx_lift2s_right_system" type="system">
+		<ros2_control name="arx_acone_right_system" type="system">
 			<hardware>
 				<plugin>arxlift2s_ros2_control/ArxX5Hardware</plugin>
@@ -28,15 +26,7 @@
 			<xacro:arx5_interfaces name="right"/>
 		</ros2_control>
-		<!-- Lift column: official LIFT2S lift HW (can5) -->
-		<ros2_control name="arx_lift2s_lift_system" type="system">
-			<hardware>
-				<plugin>arxlift2s_ros2_control/ArxLiftHardware</plugin>
-				<param name="can_name">can5</param>
-			</hardware>
-			<xacro:arx_lift2s_base_interfaces/>
-		</ros2_control>
 	</xacro:if>
 	<xacro:unless value="${'$(arg ros2_control_hardware_type)' == 'real'}">
-		<ros2_control name="arx_lift2s_system" type="system">
+		<ros2_control name="arx_acone_system" type="system">
 			<hardware>
 				<xacro:if value="${'$(arg ros2_control_hardware_type)' == 'gz'}">
@@ -52,5 +42,4 @@
 				</xacro:if>
 			</hardware>
-			<xacro:arx_lift2s_base_interfaces/>
 			<xacro:arx5_interfaces name="left"/>
 			<xacro:arx5_interfaces name="right"/>
@@ -60,5 +49,5 @@
 		<gazebo>
 			<plugin filename="gz_ros2_control-system" name="gz_ros2_control::GazeboSimROS2ControlPlugin">
-				<parameters>$(find arx_lift2s_description)/config/ros2_control/ros2_controllers.yaml</parameters>
+				<parameters>$(find arx_acone_description)/config/ros2_control/ros2_controllers.yaml</parameters>
 			</plugin>
 		</gazebo>

File: arx_lift2s_description/xacro/component.xacro (robot description, xacro)
@@ -1,23 +1,13 @@
 <?xml version="1.0" ?>
 <!-- =================================================================================== -->
-<!-- |    Complete Robot Description for ARX LIFT2S                                     | -->
-<!-- |    This file includes the base robot structure and both arms                    | -->
+<!-- |    Component visualization for ARX LIFT2S                                         | -->
 <!-- =================================================================================== -->
-<robot name="AC One" xmlns:xacro="http://www.ros.org/wiki/xacro">
+<robot name="ARX Lift2S" xmlns:xacro="http://www.ros.org/wiki/xacro">
 	<xacro:property name="PI" value="3.1415926535897931"/>
 	<xacro:arg name="type" default="chassis"/>
+	<xacro:arg name="collider" default="simple"/>
 	<xacro:if value="${'$(arg type)' == 'chassis'}">
-		<!-- Include Chassis -->
 		<xacro:include filename="$(find arx_lift2s_description)/xacro/components/chassis.xacro"/>
 		<xacro:chassis enable_wheel_joints="true"/>
-	</xacro:if>
-	<xacro:if value="${'$(arg type)' == 'ac_one'}">
-		<link name="base_link"/>
-		<joint name="base_joint" type="fixed">
-			<parent link="base_link"/>
-			<child link="body_link"/>
-		</joint>
-		<xacro:include filename="$(find arx_lift2s_description)/xacro/components/ac_one.xacro"/>
-		<xacro:ac_one />
 	</xacro:if>
 	<xacro:if value="${'$(arg type)' == 'wheel'}">

File: arx_lift2s_description/xacro/ros2_control/interfaces.xacro (robot description, xacro)
@@ -1,15 +1,12 @@
 <?xml version="1.0"?>
 <robot xmlns:xacro="http://www.ros.org/wiki/xacro">
-    <!-- ARX LIFT 2S 基座关节接口宏定义 -->
-    <xacro:macro name="arx_lift2s_base_interfaces">
-        <!-- 升降关节接口定义 (仅 lift2s 底盘需要) -->
-        <xacro:if value="${selected_base_type == 'lift2s'}">
-            <joint name="lift_joint">
-                <command_interface name="position"/>
-                <state_interface name="position"/>
-                <state_interface name="velocity"/>
-                <state_interface name="effort"/>
-            </joint>
-        </xacro:if>
-    </xacro:macro>
+	<!-- ARX LIFT 2S 基座关节接口宏定义 -->
+	<xacro:macro name="arx_lift2s_base_interfaces">
+		<joint name="lift_joint">
+			<command_interface name="position"/>
+			<state_interface name="position"/>
+			<state_interface name="velocity"/>
+			<state_interface name="effort"/>
+		</joint>
+	</xacro:macro>
 </robot>

Commit message: fix arx rviz

File: arx_acone_description/xacro/components/ac_one.xacro (robot description, xacro)
@@ -28,4 +28,5 @@
 			</xacro:if>
 			<xacro:if value="${collider == 'simple'}">
+				<!-- ACone 底座横梁：不参与 OCS2 自碰对 -->
 				<collision name="simple_base1">
 					<origin xyz="0.002 0 -0.05" rpy="0 0 0"/>
@@ -34,5 +35,10 @@
 					</geometry>
 				</collision>
-				<collision name="simple_base2">
+			</xacro:if>
+		</link>
+		<!-- 短相机立柱：独立 link，供 OCS2 只配臂↔立柱，避开底座 simple_base1 -->
+		<link name="camera_pillar_link">
+			<xacro:if value="${collider == 'simple'}">
+				<collision name="simple_camera_pillar">
 					<origin xyz="0.03 0 0.15" rpy="0 0 0"/>
 					<geometry>
@@ -40,5 +46,5 @@
 					</geometry>
 				</collision>
-				<collision name="simple_base3">
+				<collision name="simple_camera_pillar_top">
 					<origin xyz="0.08 0 0.25" rpy="0 ${-PI/6} 0"/>
 					<geometry>
@@ -48,4 +54,9 @@
 			</xacro:if>
 		</link>
+		<joint name="camera_pillar_joint" type="fixed">
+			<origin xyz="0 0 0" rpy="0 0 0"/>
+			<parent link="body_link"/>
+			<child link="camera_pillar_link"/>
+		</joint>
 		<link name="head_camera">
 			<visual>

File: arx_lift_description/xacro/components/head.xacro (robot description, xacro)
@@ -72,5 +72,6 @@
             <origin xyz="0.258786 0 0.220008"/>
         </joint>
-        <joint name="head_joint1" type="continuous">
+        <!-- revolute: continuous → Pinocchio nq=2, breaks OCS2 armDim vs joints (15). -->
+        <joint name="head_joint1" type="revolute">
             <origin xyz="0.0 0.0 0.046"/>
             <parent link="h_base_link"/>
@@ -79,5 +80,5 @@
             <limit effort="100" lower="${-PI/2}" upper="${PI/2}" velocity="100"/>
         </joint>
-        <joint name="head_joint2" type="continuous">
+        <joint name="head_joint2" type="revolute">
             <origin xyz="0.0 -0.025 0.049"/>
             <parent link="head_link1"/>

File: arx_lift_description/xacro/robot.xacro (robot description, xacro)
@@ -2,8 +2,9 @@
 <robot name="arx_lift" xmlns:xacro="http://www.ros.org/wiki/xacro">
   <!-- topology:
-       full (default) = 底盘 + 升降 + 双臂 + 头（全身 / 真机 / 可视化）
-       dual           = 仅双臂，根在 arm_base（分体 OCS2 规划，同 m6_ccs）
+       dual (default) = 仅双臂，根在 arm_base（分体 OCS2 规划 URDF 默认）
+       full           = 底盘 + 升降 + 双臂 + 头（真机 / 可视化 / 全身规划须显式传入）
+       硬件与 ros2_control 在 xacro/ros2_control/robot.xacro 里强制 topology:=full。
        全身 Pinocchio / WBC 关节序须为：lift | left×6 | right×6 | head×2 -->
-  <xacro:arg name="topology" default="full"/>
+  <xacro:arg name="topology" default="dual"/>
   <xacro:arg name="type" default="x5"/>
   <xacro:arg name="enable_wheel_joints" default="false"/>

File: arx_lift_description/xacro/ros2_control/robot.xacro (robot description, xacro)
@@ -3,4 +3,7 @@
   <xacro:arg name="ros2_control_hardware_type" default="mock_components"/>
   <xacro:arg name="gazebo" default="false"/>
+  <!-- Force full tree for hardware / robot_state_publisher. Planning URDF uses
+       xacro/robot.xacro alone (default topology:=dual) so split markers stay correct. -->
+  <xacro:arg name="topology" default="full"/>
   <xacro:include filename="$(find arx_lift_description)/xacro/robot.xacro"/>
   <xacro:include filename="$(find arx5_description)/xacro/ros2_control/interfaces.xacro"/>
