Commit message: fix lift and x7s rviz bug

File: arx_lift_description/xacro/robot.xacro (robot description, xacro)
@@ -1,13 +1,8 @@
 <?xml version="1.0" ?>
 <robot name="arx_lift" xmlns:xacro="http://www.ros.org/wiki/xacro">
-  <!-- topology:
-       dual (default) = 仅双臂，根在 arm_base（分体 OCS2 规划 URDF 默认）
-       full           = 底盘 + 升降 + 双臂 + 头（真机 / 可视化 / 全身规划须显式传入）
-       硬件与 ros2_control 在 xacro/ros2_control/robot.xacro 里强制 topology:=full。
-       全身 Pinocchio / WBC 关节序须为：lift | left×6 | right×6 | head×2 -->
-  <xacro:arg name="topology" default="dual"/>
+  <!-- Full robot only. Split-body OCS2 planning uses arx_acone_description
+       (robot_name override + Lift mount xyz), same pattern as Lift2S. -->
   <xacro:arg name="type" default="x5"/>
   <xacro:arg name="enable_wheel_joints" default="false"/>
-  <xacro:property name="topology_arg" value="$(arg topology)"/>
   <xacro:property name="type_arg" value="$(arg type)"/>
   <xacro:property name="selected_arm_type" value="x5"/>
@@ -15,76 +10,44 @@
     <xacro:property name="selected_arm_type" value="r5"/>
   </xacro:if>
-  <!-- ===== dual：仅双臂（分体规划，根 = arm_base，同 m6_ccs） ===== -->
-  <xacro:if value="${topology_arg == 'dual'}">
-    <link name="arm_base"/>
-    <link name="body_link"/>
-    <joint name="arm_base_body" type="fixed">
-      <parent link="arm_base"/>
-      <child link="body_link"/>
-      <origin xyz="0 0 0"/>
-    </joint>
-    <xacro:if value="${selected_arm_type == 'x5'}">
-      <xacro:include filename="$(find arx5_description)/xacro/X5.xacro"/>
-      <xacro:X5 name="left"/>
-      <xacro:X5 name="right"/>
-    </xacro:if>
-    <xacro:if value="${selected_arm_type == 'r5'}">
-      <xacro:include filename="$(find arx5_description)/xacro/R5.xacro"/>
-      <xacro:R5 name="left"/>
-      <xacro:R5 name="right"/>
-    </xacro:if>
-    <joint name="arm_left_fixed" type="fixed">
-      <parent link="arm_base"/>
-      <child link="left_base_link"/>
-      <origin xyz="0.208 0.25000 0.092"/>
-    </joint>
-    <joint name="arm_right_fixed" type="fixed">
-      <parent link="arm_base"/>
-      <child link="right_base_link"/>
-      <origin xyz="0.208 -0.25000 0.092"/>
-    </joint>
+  <xacro:include filename="$(find arx_lift_description)/xacro/components/mobile_base.xacro"/>
+  <xacro:include filename="$(find arx_lift_description)/xacro/components/body.xacro"/>
+  <xacro:include filename="$(find arx_lift_description)/xacro/components/head.xacro"/>
+  <xacro:MobileBase enable_wheel_joints="$(arg enable_wheel_joints)"/>
+  <xacro:Body/>
+  <!-- 臂座：与 lift_link 固连 -->
+  <link name="body_link"/>
+  <joint name="body_fixed" type="fixed">
+    <parent link="lift_link"/>
+    <child link="body_link"/>
+    <origin xyz="0 0 0"/>
+  </joint>
+  <link name="arm_base"/>
+  <joint name="arm_base_joint" type="fixed">
+    <parent link="lift_link"/>
+    <child link="arm_base"/>
+    <origin xyz="0 0 0"/>
+  </joint>
+  <xacro:if value="${selected_arm_type == 'x5'}">
+    <xacro:include filename="$(find arx5_description)/xacro/X5.xacro"/>
+    <xacro:X5 name="left"/>
+    <xacro:X5 name="right"/>
   </xacro:if>
-  <!-- ===== full：整机（升降 → 双臂 → 头，匹配 WBC 布局） ===== -->
-  <xacro:unless value="${topology_arg == 'dual'}">
-    <xacro:include filename="$(find arx_lift_description)/xacro/components/mobile_base.xacro"/>
-    <xacro:include filename="$(find arx_lift_description)/xacro/components/body.xacro"/>
-    <xacro:include filename="$(find arx_lift_description)/xacro/components/head.xacro"/>
-    <xacro:MobileBase enable_wheel_joints="$(arg enable_wheel_joints)"/>
-    <xacro:Body/>
-    <!-- 臂座：与 lift_link 固连 -->
-    <link name="body_link"/>
-    <joint name="body_fixed" type="fixed">
-      <parent link="lift_link"/>
-      <child link="body_link"/>
-      <origin xyz="0 0 0"/>
-    </joint>
-    <link name="arm_base"/>
-    <joint name="arm_base_joint" type="fixed">
-      <parent link="lift_link"/>
-      <child link="arm_base"/>
-      <origin xyz="0 0 0"/>
-    </joint>
-    <xacro:if value="${selected_arm_type == 'x5'}">
-      <xacro:include filename="$(find arx5_description)/xacro/X5.xacro"/>
-      <xacro:X5 name="left"/>
-      <xacro:X5 name="right"/>
-    </xacro:if>
-    <xacro:if value="${selected_arm_type == 'r5'}">
-      <xacro:include filename="$(find arx5_description)/xacro/R5.xacro"/>
-      <xacro:R5 name="left"/>
-      <xacro:R5 name="right"/>
-    </xacro:if>
-    <joint name="arm_left_fixed" type="fixed">
-      <parent link="arm_base"/>
-      <child link="left_base_link"/>
-      <origin xyz="0.208 0.25000 0.092"/>
-    </joint>
-    <joint name="arm_right_fixed" type="fixed">
-      <parent link="arm_base"/>
-      <child link="right_base_link"/>
-      <origin xyz="0.208 -0.25000 0.092"/>
-    </joint>
-    <!-- 头放在双臂之后，Pinocchio 序 = lift | L6 | R6 | head×2 -->
-    <xacro:Head/>
-  </xacro:unless>
+  <xacro:if value="${selected_arm_type == 'r5'}">
+    <xacro:include filename="$(find arx5_description)/xacro/R5.xacro"/>
+    <xacro:R5 name="left"/>
+    <xacro:R5 name="right"/>
+  </xacro:if>
+  <!-- Classic Lift mount (≠ acone default); split planning must pass same xyz to acone. -->
+  <joint name="arm_left_fixed" type="fixed">
+    <parent link="arm_base"/>
+    <child link="left_base_link"/>
+    <origin xyz="0.208 0.25000 0.092"/>
+  </joint>
+  <joint name="arm_right_fixed" type="fixed">
+    <parent link="arm_base"/>
+    <child link="right_base_link"/>
+    <origin xyz="0.208 -0.25000 0.092"/>
+  </joint>
+  <!-- 头放在双臂之后，Pinocchio 序 = lift | L6 | R6 | head×2 -->
+  <xacro:Head/>
 </robot>

File: arx_lift_description/xacro/ros2_control/robot.xacro (robot description, xacro)
@@ -3,11 +3,9 @@
   <xacro:arg name="ros2_control_hardware_type" default="mock_components"/>
   <xacro:arg name="gazebo" default="false"/>
-  <!-- Force full tree for hardware / robot_state_publisher. Planning URDF uses
-       xacro/robot.xacro alone (default topology:=dual) so split markers stay correct. -->
-  <xacro:arg name="topology" default="full"/>
+  <!-- Hardware / RSP always use full arx_lift xacro/robot.xacro.
+       Split planning uses arx_acone (robot_name override), not this file. -->
   <xacro:include filename="$(find arx_lift_description)/xacro/robot.xacro"/>
   <xacro:include filename="$(find arx5_description)/xacro/ros2_control/interfaces.xacro"/>
   <xacro:include filename="$(find arx_lift_description)/xacro/ros2_control/interfaces.xacro"/>
-  <!-- 硬件描述始终用 full 拓扑（分体规划 dual 只影响 planning URDF） -->
   <xacro:property name="sim_iface_mode"
     value="${'position' if '$(arg ros2_control_hardware_type)' == 'isaac' else 'mix'}"/>

File: arx_x7s_description/xacro/robot.xacro (robot description, xacro)
@@ -1,17 +1,14 @@
 <robot name="ARX X7S" xmlns:xacro="http://www.ros.org/wiki/xacro">
+  <!-- Full robot only. Split-body OCS2 planning uses arx_x7s_arms_description
+       (robot_name override), same pattern as Lift2S→acone / fa_w2→m6_ccs. -->
   <xacro:arg name="enable_wheel_joints" default="false"/>
-  <!-- Include component files -->
   <xacro:include filename="$(find arx_x7s_description)/xacro/components/base.xacro"/>
   <xacro:include filename="$(find arx_x7s_description)/xacro/components/body.xacro"/>
   <xacro:include filename="$(find arx_x7s_description)/xacro/components/arm.xacro"/>
   <xacro:include filename="$(find arx_x7s_description)/xacro/components/gripper.xacro"/>
-  <!-- Base and lift -->
   <xacro:Base enable_wheel_joints="$(arg enable_wheel_joints)"/>
-  <!-- Body, neck, and head -->
   <xacro:Body/>
-  <!-- Left arm -->
   <xacro:Arm name="left" direction="1"/>
   <xacro:Gripper name="left" direction="1"/>
-  <!-- Right arm -->
   <xacro:Arm name="right" direction="-1"/>
   <xacro:Gripper name="right" direction="-1"/>

File: arx_x7s_description/xacro/ros2_control/robot.xacro (robot description, xacro)
@@ -2,15 +2,11 @@
 <!-- =================================================================================== -->
 <!-- |    Complete Robot Description for ARX X7S with ROS2 Control                    | -->
-<!-- |    This file includes the base robot structure and both arms                   | -->
 <!-- =================================================================================== -->
 <robot name="arx_x7s_whole_body" xmlns:xacro="http://www.ros.org/wiki/xacro">
   <xacro:arg name="ros2_control_hardware_type" default="mock_components"/>
-  <!-- Include the base robot structure -->
   <xacro:include filename="$(find arx_x7s_description)/xacro/robot.xacro"/>
-  <!-- Import modular interface components -->
   <xacro:include filename="$(find arx_x7s_description)/xacro/ros2_control/arx_x7s_base_interfaces.xacro"/>
   <xacro:include filename="$(find arx_x7s_description)/xacro/ros2_control/arx_x7s_arm_interfaces.xacro"/>
   <xacro:include filename="$(find arx_x7s_description)/xacro/ros2_control/arx_x7s_gripper_interfaces.xacro"/>
-  <!-- Unified ros2_control system -->
   <ros2_control name="arx_x7s_unified_system" type="system">
     <hardware>
@@ -27,11 +23,7 @@
       </xacro:if>
     </hardware>
-    <!-- 基座接口 (包含升降、腰部、头部) -->
     <xacro:arx_x7s_base_interfaces/>
-    <!-- 左臂接口 -->
     <xacro:arx_x7s_arm_interfaces name="left"/>
-    <!-- 右臂接口 -->
     <xacro:arx_x7s_arm_interfaces name="right"/>
-    <!-- 夹爪接口 -->
     <xacro:arx_x7s_gripper_interfaces name="left"/>
     <xacro:arx_x7s_gripper_interfaces name="right"/>
