Commit message: fix x7s rviz ,split body and full body

File: arx_x7s_description/urdf/arx_x7s.urdf (robot description, URDF)
Before this commit: robot ARX X7S, 30 links, 29 joints
Joints:
- removed joint waist_joint
- added joint body_joint: type revolute, parent lift, child body, origin xyz=0.066 -0.0546 -0.06, axis 0 1 0, limit lower=0 upper=1.57 effort=100 velocity=5

File: arx_x7s_description/xacro/components/body.xacro (robot description, xacro)
@@ -26,5 +26,6 @@
       </collision>
     </link>
-    <joint name="waist_joint" type="revolute">
+    <!-- Named body_joint (not waist_joint) so MOVEJ Body group matches arms/fa-py rules. -->
+    <joint name="body_joint" type="revolute">
       <origin xyz="0.066 -0.0546 -0.06"/>
       <parent link="lift"/>

File: arx_x7s_description/xacro/robot.xacro (robot description, xacro)
@@ -1,15 +1,29 @@
+<?xml version="1.0"?>
+<!-- Planning / visualization entry.
+     topology:=full (default) — whole robot (WBC).
+     topology:=dual — root=body, arms only (split-body OCS2 planning).
+     Hardware always uses ros2_control/robot.xacro → robot_full.xacro (ignores dual). -->
 <robot name="ARX X7S" xmlns:xacro="http://www.ros.org/wiki/xacro">
-  <!-- Full robot only. Split-body OCS2 planning uses arx_x7s_arms_description
-       (robot_name override), same pattern as Lift2S→acone / fa_w2→m6_ccs. -->
+  <xacro:arg name="topology" default="full"/>
   <xacro:arg name="enable_wheel_joints" default="false"/>
-  <xacro:include filename="$(find arx_x7s_description)/xacro/components/base.xacro"/>
-  <xacro:include filename="$(find arx_x7s_description)/xacro/components/body.xacro"/>
+  <xacro:property name="topo" value="$(arg topology)"/>
   <xacro:include filename="$(find arx_x7s_description)/xacro/components/arm.xacro"/>
   <xacro:include filename="$(find arx_x7s_description)/xacro/components/gripper.xacro"/>
-  <xacro:Base enable_wheel_joints="$(arg enable_wheel_joints)"/>
-  <xacro:Body/>
-  <xacro:Arm name="left" direction="1"/>
-  <xacro:Gripper name="left" direction="1"/>
-  <xacro:Arm name="right" direction="-1"/>
-  <xacro:Gripper name="right" direction="-1"/>
+  <xacro:if value="${topo == 'dual'}">
+    <link name="body"/>
+    <xacro:Arm name="left" direction="1"/>
+    <xacro:Gripper name="left" direction="1"/>
+    <xacro:Arm name="right" direction="-1"/>
+    <xacro:Gripper name="right" direction="-1"/>
+  </xacro:if>
+  <xacro:unless value="${topo == 'dual'}">
+    <xacro:include filename="$(find arx_x7s_description)/xacro/components/base.xacro"/>
+    <xacro:include filename="$(find arx_x7s_description)/xacro/components/body.xacro"/>
+    <xacro:Base enable_wheel_joints="$(arg enable_wheel_joints)"/>
+    <xacro:Body/>
+    <xacro:Arm name="left" direction="1"/>
+    <xacro:Gripper name="left" direction="1"/>
+    <xacro:Arm name="right" direction="-1"/>
+    <xacro:Gripper name="right" direction="-1"/>
+  </xacro:unless>
 </robot>

File: arx_x7s_description/xacro/ros2_control/arx_x7s_base_interfaces.xacro (robot description, xacro)
@@ -10,6 +10,6 @@
       <state_interface name="effort"/>
     </joint>
-    <!-- 腰部关节接口定义 -->
-    <joint name="waist_joint">
+    <!-- 腰俯仰（body_joint；MOVEJ Body 前缀需 body*） -->
+    <joint name="body_joint">
       <command_interface name="position"/>
       <state_interface name="position"/>

File: arx_x7s_description/xacro/ros2_control/robot.xacro (robot description, xacro)
@@ -1,9 +1,8 @@
 <?xml version="1.0" ?>
-<!-- =================================================================================== -->
-<!-- |    Complete Robot Description for ARX X7S with ROS2 Control                    | -->
-<!-- =================================================================================== -->
+<!-- Hardware / RSP: always full kinematics (never honor planning topology:=dual). -->
 <robot name="arx_x7s_whole_body" xmlns:xacro="http://www.ros.org/wiki/xacro">
   <xacro:arg name="ros2_control_hardware_type" default="mock_components"/>
-  <xacro:include filename="$(find arx_x7s_description)/xacro/robot.xacro"/>
+  <xacro:arg name="enable_wheel_joints" default="false"/>
+  <xacro:include filename="$(find arx_x7s_description)/xacro/robot_full.xacro"/>
   <xacro:include filename="$(find arx_x7s_description)/xacro/ros2_control/arx_x7s_base_interfaces.xacro"/>
   <xacro:include filename="$(find arx_x7s_description)/xacro/ros2_control/arx_x7s_arm_interfaces.xacro"/>
