Commit message: Feature/lift2s mit：MIT arms, lift hybrid modes, and full-body WBC (#5)
* add sepetate acone package

* add self-collision for lift body

* add feedforward for arm

* fix the arm marker Vanished bug in rviz

* add mit control

* MIT ok for arms

* add mit control

* change ocs2 info,fix marker bug

* add hybrid control for lift

* add soft_p control for lift_joint

* add position control for arm

* :sparkles: add wbc for lift2s

* add shutdown to home

* :sparkles: add friction compensation

* remove HI ramp

* set default param

* update the descritpionf

* update new readme

* close debug info

* stash default config

* modify planning urdf

* Improve the comments

* delete .idea

* modify readme

* change default  param

* add scale param

* update yaml for vr

* update config

* update yaml

* fix fullbody mode

* fix arx lift fullbody control

* add chassis move param

* fix arx camera direction

* fix arx rviz

* update arx rviz ,expect x7s

* fix lift and x7s rviz bug

* fix x7s rviz ,split body and full body

* fix lift ,close collision

* update readme

---------

Co-authored-by: Huang Zhenbiao <biao876990970@hotmail.com>

File: arx_lift2s_description/xacro/ros2_control/robot.xacro (robot description, xacro)
@@ -4,6 +4,8 @@
 	<xacro:arg name="gazebo" default="false"/>
 	<!-- Arms: full_control only (MIT MIX). -->
-	<!-- Lift: soft_p|position | hybrid. hybrid 直跟 pos+vel，HI 重力+摩擦（忽略 effort） -->
+	<!-- Lift: soft_p|position | hybrid. 两种模式升降/底盘分开发；hybrid 跟 pos+vel，soft_p 只跟 position -->
 	<xacro:arg name="lift_motor_mode" default="hybrid"/>
+	<!-- Lift HI：可选订阅 /cmd_vel → setChassisCmd（默认开；若与 WBC 底盘规划抢指令可显式关） -->
+	<xacro:arg name="enable_chassis_cmd_vel" default="true"/>
 	<xacro:include filename="$(find arx_lift2s_description)/xacro/robot.xacro"/>
 	<xacro:include filename="$(find arx5_description)/xacro/ros2_control/interfaces.xacro"/>
@@ -53,5 +55,5 @@
 				<param name="can_name">can5</param>
 				<param name="robot_type">2</param>
-				<!-- soft_p|position: 仅跟踪 position；hybrid: 直跟 pos+vel + HI 重力/摩擦（忽略 effort） -->
+				<!-- soft_p|position: 仅跟踪 position + 常值重力；hybrid: 直跟 pos+vel + 重力/摩擦（忽略 effort） -->
 				<param name="lift_motor_mode">$(arg lift_motor_mode)</param>
 				<!-- Soft-P (setHeight/loop); live: arx_lift.soft_p_kp -->
@@ -66,5 +68,5 @@
 				<param name="friction_vel_eps_mps">0.01</param>
 				<param name="lift_max_torque">15.0</param>
-				<!-- cmd_ramp_vel: soft_p 跟踪与关机插值；hybrid 跟踪不用 -->
+				<!-- cmd_ramp_vel: 仅关机回零插值；Soft-P/hybrid 跟踪都不用 -->
 				<param name="cmd_ramp_vel">0.12</param>
 				<param name="max_height_m">0.48</param>
@@ -78,8 +80,21 @@
 				<param name="shutdown_home_velocity">0.10</param>
 				<param name="shutdown_home_timeout">2.0</param>
+				<!-- 可选：/cmd_vel → 底盘 setChassisCmd；默认关 -->
+				<param name="enable_chassis_cmd_vel">$(arg enable_chassis_cmd_vel)</param>
+				<param name="chassis_cmd_vel_topic">/cmd_vel</param>
+				<param name="chassis_cmd_timeout">0.3</param>
+				<!-- LIFTS SDK 未初始化 max_vel；供 setChassisCmd 量化：
+				     CAN ≈ (v/max_vel)*±660。同 cmd_vel 下 max 越小 → 比例越大 → 越“快”；
+				     同时 v 会被 clamp 到 ±max。单位与 Twist 一致（m/s、rad/s）。 -->
+				<param name="chassis_max_vel_x">1.0</param>
+				<param name="chassis_max_vel_y">1.0</param>
+				<param name="chassis_max_vel_z">2.0</param>
 			</hardware>
 			<xacro:arx_lift2s_base_interfaces/>
 		</ros2_control>
 	</xacro:if>
+	<!-- Isaac: position-only（TopicBasedSystem / 仿真对 effort、velocity 支持差）；mock/gz 仍 MIX -->
+	<xacro:property name="sim_iface_mode"
+		value="${'position' if '$(arg ros2_control_hardware_type)' == 'isaac' else 'mix'}"/>
 	<xacro:unless value="${'$(arg ros2_control_hardware_type)' == 'real'}">
 		<ros2_control name="arx_lift2s_system" type="system">
@@ -97,8 +112,7 @@
 				</xacro:if>
 			</hardware>
-			<xacro:arx_lift2s_base_interfaces/>
-			<!-- Sim: MIX arm IFs to match real Stanford HI / full_control -->
-			<xacro:arx5_interfaces name="left"/>
-			<xacro:arx5_interfaces name="right"/>
+			<xacro:arx_lift2s_base_interfaces iface_mode="${sim_iface_mode}"/>
+			<xacro:arx5_interfaces name="left" iface_mode="${sim_iface_mode}"/>
+			<xacro:arx5_interfaces name="right" iface_mode="${sim_iface_mode}"/>
 		</ros2_control>
 	</xacro:unless>

File: arx_lift_description/xacro/robot.xacro (robot description, xacro)
@@ -1,32 +1,53 @@
 <?xml version="1.0" ?>
 <robot name="arx_lift" xmlns:xacro="http://www.ros.org/wiki/xacro">
+  <!-- Full robot only. Split-body OCS2 planning uses arx_acone_description
+       (robot_name override + Lift mount xyz), same pattern as Lift2S. -->
   <xacro:arg name="type" default="x5"/>
   <xacro:arg name="enable_wheel_joints" default="false"/>
-  <!-- 根据type参数包含不同的机械臂描述文件 -->
-  <xacro:if value="${'$(arg type)' == 'x5'}">
+  <xacro:property name="type_arg" value="$(arg type)"/>
+  <xacro:property name="selected_arm_type" value="x5"/>
+  <xacro:if value="${type_arg == 'r5'}">
+    <xacro:property name="selected_arm_type" value="r5"/>
+  </xacro:if>
+  <xacro:include filename="$(find arx_lift_description)/xacro/components/mobile_base.xacro"/>
+  <xacro:include filename="$(find arx_lift_description)/xacro/components/body.xacro"/>
+  <xacro:include filename="$(find arx_lift_description)/xacro/components/head.xacro"/>
+  <xacro:MobileBase enable_wheel_joints="$(arg enable_wheel_joints)"/>
+  <xacro:Body/>
+  <!-- 臂座：与 lift_link 固连 -->
+  <link name="body_link"/>
+  <joint name="body_fixed" type="fixed">
+    <parent link="lift_link"/>
+    <child link="body_link"/>
+    <origin xyz="0 0 0"/>
+  </joint>
+  <link name="arm_base"/>
+  <joint name="arm_base_joint" type="fixed">
+    <parent link="lift_link"/>
+    <child link="arm_base"/>
+    <origin xyz="0 0 0"/>
+  </joint>
+  <xacro:if value="${selected_arm_type == 'x5'}">
     <xacro:include filename="$(find arx5_description)/xacro/X5.xacro"/>
-    <!-- 使用R5宏来创建两个机械臂 -->
     <xacro:X5 name="left"/>
     <xacro:X5 name="right"/>
   </xacro:if>
-  <xacro:if value="${'$(arg type)' == 'r5'}">
+  <xacro:if value="${selected_arm_type == 'r5'}">
     <xacro:include filename="$(find arx5_description)/xacro/R5.xacro"/>
-    <!-- 使用R5宏来创建两个机械臂 -->
     <xacro:R5 name="left"/>
     <xacro:R5 name="right"/>
   </xacro:if>
-  <xacro:include filename="$(find arx_lift_description)/xacro/components/mobile_base.xacro"/>
-  <xacro:include filename="$(find arx_lift_description)/xacro/components/body.xacro"/>
-  <xacro:MobileBase enable_wheel_joints="$(arg enable_wheel_joints)"/>
-  <xacro:Body/>
+  <!-- Classic Lift mount (≠ acone default); split planning must pass same xyz to acone. -->
   <joint name="arm_left_fixed" type="fixed">
-    <parent link="lift_link"/>
+    <parent link="arm_base"/>
     <child link="left_base_link"/>
-    <origin  xyz="0.208 0.25000 0.092"/>
+    <origin xyz="0.208 0.25000 0.092"/>
   </joint>
   <joint name="arm_right_fixed" type="fixed">
-    <parent link="lift_link"/>
+    <parent link="arm_base"/>
     <child link="right_base_link"/>
     <origin xyz="0.208 -0.25000 0.092"/>
   </joint>
+  <!-- 头放在双臂之后，Pinocchio 序 = lift | L6 | R6 | head×2 -->
+  <xacro:Head/>
 </robot>

File: arx_lift_description/xacro/ros2_control/interfaces.xacro (robot description, xacro)
@@ -1,24 +1,37 @@
 <?xml version="1.0"?>
 <robot xmlns:xacro="http://www.ros.org/wiki/xacro">
-	<xacro:macro name="lift_interfaces">
-		<!-- 升降机构关节 -->
+	<!-- iface_mode: mix = pos/vel/effort（mock/gz）；position = 仅 position（Isaac） -->
+	<xacro:macro name="lift_interfaces" params="iface_mode:=mix">
 		<joint name="lift_joint">
 			<command_interface name="position"/>
+			<xacro:if value="${iface_mode == 'mix'}">
+				<command_interface name="velocity"/>
+				<command_interface name="effort"/>
+			</xacro:if>
 			<state_interface name="position">
 				<param name="initial_value">0.3</param>
 			</state_interface>
-			<state_interface name="velocity"/>
-			<state_interface name="effort"/>
+			<xacro:if value="${iface_mode == 'mix'}">
+				<state_interface name="velocity"/>
+				<state_interface name="effort"/>
+			</xacro:if>
 		</joint>
-		<!-- 头部关节1 -->
+		<!-- 头：mock/gz 与 WBC MIX 一致（pos/vel/effort）；Isaac 仅 position -->
 		<joint name="head_joint1">
 			<command_interface name="position"/>
+			<xacro:if value="${iface_mode == 'mix'}">
+				<command_interface name="velocity"/>
+				<command_interface name="effort"/>
+			</xacro:if>
 			<state_interface name="position"/>
 			<state_interface name="velocity"/>
 			<state_interface name="effort"/>
 		</joint>
-		<!-- 头部关节2 -->
 		<joint name="head_joint2">
 			<command_interface name="position"/>
+			<xacro:if value="${iface_mode == 'mix'}">
+				<command_interface name="velocity"/>
+				<command_interface name="effort"/>
+			</xacro:if>
 			<state_interface name="position"/>
 			<state_interface name="velocity"/>

File: arx_lift_description/xacro/ros2_control/robot.xacro (robot description, xacro)
@@ -1,7 +1,13 @@
 <?xml version="1.0"?>
 <robot xmlns:xacro="http://www.ros.org/wiki/xacro" name="arx_lift">
+  <xacro:arg name="ros2_control_hardware_type" default="mock_components"/>
+  <xacro:arg name="gazebo" default="false"/>
+  <!-- Hardware / RSP always use full arx_lift xacro/robot.xacro.
+       Split planning uses arx_acone (robot_name override), not this file. -->
   <xacro:include filename="$(find arx_lift_description)/xacro/robot.xacro"/>
   <xacro:include filename="$(find arx5_description)/xacro/ros2_control/interfaces.xacro"/>
   <xacro:include filename="$(find arx_lift_description)/xacro/ros2_control/interfaces.xacro"/>
+  <xacro:property name="sim_iface_mode"
+    value="${'position' if '$(arg ros2_control_hardware_type)' == 'isaac' else 'mix'}"/>
   <ros2_control name="arx_lift_unified_system" type="system">
     <hardware>
@@ -18,10 +24,8 @@
       </xacro:if>
     </hardware>
-    <xacro:lift_interfaces/>
-    <xacro:arx5_interfaces name="left"/>
-    <xacro:arx5_interfaces name="right"/>
+    <xacro:lift_interfaces iface_mode="${sim_iface_mode}"/>
+    <xacro:arx5_interfaces name="left" iface_mode="${sim_iface_mode}"/>
+    <xacro:arx5_interfaces name="right" iface_mode="${sim_iface_mode}"/>
   </ros2_control>
-  <!-- Gazebo插件配置 -->
-  <xacro:arg name="gazebo" default="false" />
   <xacro:if value="$(arg gazebo)">
     <gazebo>

File: arx_x7s_description/xacro/robot.xacro (robot description, xacro)
@@ -1,18 +1,29 @@
+<?xml version="1.0"?>
+<!-- Planning / visualization entry.
+     topology:=full (default) — whole robot (WBC).
+     topology:=dual — root=body, arms only (split-body OCS2 planning).
+     Hardware always uses ros2_control/robot.xacro → robot_full.xacro (ignores dual). -->
 <robot name="ARX X7S" xmlns:xacro="http://www.ros.org/wiki/xacro">
+  <xacro:arg name="topology" default="full"/>
   <xacro:arg name="enable_wheel_joints" default="false"/>
-  <!-- Include component files -->
-  <xacro:include filename="$(find arx_x7s_description)/xacro/components/base.xacro"/>
-  <xacro:include filename="$(find arx_x7s_description)/xacro/components/body.xacro"/>
+  <xacro:property name="topo" value="$(arg topology)"/>
   <xacro:include filename="$(find arx_x7s_description)/xacro/components/arm.xacro"/>
   <xacro:include filename="$(find arx_x7s_description)/xacro/components/gripper.xacro"/>
-  <!-- Base and lift -->
-  <xacro:Base enable_wheel_joints="$(arg enable_wheel_joints)"/>
-  <!-- Body, neck, and head -->
-  <xacro:Body/>
-  <!-- Left arm -->
-  <xacro:Arm name="left" direction="1"/>
-  <xacro:Gripper name="left" direction="1"/>
-  <!-- Right arm -->
-  <xacro:Arm name="right" direction="-1"/>
-  <xacro:Gripper name="right" direction="-1"/>
+  <xacro:if value="${topo == 'dual'}">
+    <link name="body"/>
+    <xacro:Arm name="left" direction="1"/>
+    <xacro:Gripper name="left" direction="1"/>
+    <xacro:Arm name="right" direction="-1"/>
+    <xacro:Gripper name="right" direction="-1"/>
+  </xacro:if>
+  <xacro:unless value="${topo == 'dual'}">
+    <xacro:include filename="$(find arx_x7s_description)/xacro/components/base.xacro"/>
+    <xacro:include filename="$(find arx_x7s_description)/xacro/components/body.xacro"/>
+    <xacro:Base enable_wheel_joints="$(arg enable_wheel_joints)"/>
+    <xacro:Body/>
+    <xacro:Arm name="left" direction="1"/>
+    <xacro:Gripper name="left" direction="1"/>
+    <xacro:Arm name="right" direction="-1"/>
+    <xacro:Gripper name="right" direction="-1"/>
+  </xacro:unless>
 </robot>

File: arx_x7s_description/xacro/ros2_control/robot.xacro (robot description, xacro)
@@ -1,16 +1,11 @@
 <?xml version="1.0" ?>
-<!-- =================================================================================== -->
-<!-- |    Complete Robot Description for ARX X7S with ROS2 Control                    | -->
-<!-- |    This file includes the base robot structure and both arms                   | -->
-<!-- =================================================================================== -->
+<!-- Hardware / RSP: always full kinematics (never honor planning topology:=dual). -->
 <robot name="arx_x7s_whole_body" xmlns:xacro="http://www.ros.org/wiki/xacro">
   <xacro:arg name="ros2_control_hardware_type" default="mock_components"/>
-  <!-- Include the base robot structure -->
-  <xacro:include filename="$(find arx_x7s_description)/xacro/robot.xacro"/>
-  <!-- Import modular interface components -->
+  <xacro:arg name="enable_wheel_joints" default="false"/>
+  <xacro:include filename="$(find arx_x7s_description)/xacro/robot_full.xacro"/>
   <xacro:include filename="$(find arx_x7s_description)/xacro/ros2_control/arx_x7s_base_interfaces.xacro"/>
   <xacro:include filename="$(find arx_x7s_description)/xacro/ros2_control/arx_x7s_arm_interfaces.xacro"/>
   <xacro:include filename="$(find arx_x7s_description)/xacro/ros2_control/arx_x7s_gripper_interfaces.xacro"/>
-  <!-- Unified ros2_control system -->
   <ros2_control name="arx_x7s_unified_system" type="system">
     <hardware>
@@ -27,11 +22,7 @@
       </xacro:if>
     </hardware>
-    <!-- 基座接口 (包含升降、腰部、头部) -->
     <xacro:arx_x7s_base_interfaces/>
-    <!-- 左臂接口 -->
     <xacro:arx_x7s_arm_interfaces name="left"/>
-    <!-- 右臂接口 -->
     <xacro:arx_x7s_arm_interfaces name="right"/>
-    <!-- 夹爪接口 -->
     <xacro:arx_x7s_gripper_interfaces name="left"/>
     <xacro:arx_x7s_gripper_interfaces name="right"/>
